File: Boards/GateDriver/GateDriver.kicad_pcb (KiCad board)
At the start: 6 copper layers, 75 x 60 mm, 69 parts, among them IC1 ADUM4136BRWZ, IC2 ADUM4136BRWZ, J1 Conn_02x08_Counter_Clockwise

Commit message: board changes and switchingcontroller
Parts:
- H1, H3: footprint MountingHole:MountingHole_5.3mm_M5 -> MountingHole:MountingHole_3.2mm_M3
Changed lines of the file:
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@@
 		)
 	)
-	(footprint "MountingHole:MountingHole_5.3mm_M5"
+	(footprint "MountingHole:MountingHole_3.2mm_M3"
 		(layer "F.Cu")
 		(at 6 54)
-		(descr "Mounting Hole 5.3mm, no annular, M5")
-		(tags "mounting hole 5.3mm no annular m5")
+		(descr "Mounting Hole 3.2mm, M3, no annular, generated by kicad-footprint-generator mountinghole.py")
+		(tags "mountinghole M3")
 		(property "Reference" "H1"
-			(at -4 5 0)
+			(at 0 -4.15 0)
 			(layer "F.SilkS")
 			(effects
@@
 		)
 		(property "Value" "MountingHole"
-			(at 0 6.3 0)
+			(at 0 4.15 0)
 			(layer "F.Fab")
 			(effects
@@
 		(property "Datasheet" ""
 			(at 0 0 0)
-			(unlocked yes)
 			(layer "F.Fab")
 			(hide yes)
@@
 		(property "Description" "Mounting Hole without connection"
 			(at 0 0 0)
-			(unlocked yes)
 			(layer "F.Fab")
 			(hide yes)
@@
 		(fp_circle
 			(center 0 0)
-			(end 5.3 0)
+			(end 3.2 0)
 			(stroke
 				(width 0.15)
@@
 		(fp_circle
 			(center 0 0)
-			(end 5.55 0)
+			(end 3.45 0)
 			(stroke
 				(width 0.05)
@@
 		(pad "" np_thru_hole circle
 			(at 0 0)
-			(size 5.3 5.3)
-			(drill 5.3)
+			(size 3.2 3.2)
+			(drill 3.2)
 			(layers "*.Cu" "*.Mask")
 		)
@@
 		)
 	)
-	(footprint "MountingHole:MountingHole_5.3mm_M5"
+	(footprint "MountingHole:MountingHole_3.2mm_M3"
 		(layer "F.Cu")
 		(at 69 54)
-		(descr "Mounting Hole 5.3mm, no annular, M5")
-		(tags "mounting hole 5.3mm no annular m5")
+		(descr "Mounting Hole 3.2mm, M3, no annular, generated by kicad-footprint-generator mountinghole.py")
+		(tags "mountinghole M3")
 		(property "Reference" "H3"
-			(at 4 5 0)
+			(at 0 -4.15 0)
 			(layer "F.SilkS")
 			(effects
@@
 		)
 		(property "Value" "MountingHole"
-			(at 0 6.3 0)
+			(at 0 4.15 0)
 			(layer "F.Fab")
 			(effects
@@
 		(property "Datasheet" ""
 			(at 0 0 0)
-			(unlocked yes)
 			(layer "F.Fab")
 			(hide yes)
@@
 		(property "Description" "Mounting Hole without connection"
 			(at 0 0 0)
-			(unlocked yes)
 			(layer "F.Fab")
 			(hide yes)
@@
 		(fp_circle
 			(center 0 0)
-			(end 5.3 0)
+			(end 3.2 0)
 			(stroke
 				(width 0.15)
@@
 		(fp_circle
 			(center 0 0)
-			(end 5.55 0)
+			(end 3.45 0)
 			(stroke
 				(width 0.05)
@@
 		(pad "" np_thru_hole circle
 			(at 0 0)
-			(size 5.3 5.3)
-			(drill 5.3)
+			(size 3.2 3.2)
+			(drill 3.2)
 			(layers "*.Cu" "*.Mask")
 		)
