File: Boards/GateDriver/GateDriver.kicad_sch (KiCad schematic)
At the start: 23 parts, among them J1 Conn_02x08_Counter_Clockwise

Commit message: board changes and switchingcontroller
Parts:
- H1, H3: footprint MountingHole:MountingHole_5.3mm_M5 -> MountingHole:MountingHole_3.2mm_M3
Changed lines of the file:
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@@
 			)
 		)
-		(property "Footprint" "MountingHole:MountingHole_5.3mm_M5"
+		(property "Footprint" "MountingHole:MountingHole_3.2mm_M3"
 			(at 25.4 25.4 0)
 			(effects
@@
 			)
 		)
-		(property "Footprint" "MountingHole:MountingHole_5.3mm_M5"
+		(property "Footprint" "MountingHole:MountingHole_3.2mm_M3"
 			(at 25.4 50.8 0)
 			(effects
