File: Boards/MainBoard/MainBoard.kicad_pcb (KiCad board)
At the start: 6 copper layers, 297.5 x 60 mm, 140 parts, among them IC1 MAX22530AWE+, IC13 DRDNB21D-7, IC14 DRDNB21D-7, IC2 MAX22530AWE+, IC5 MCP2515-e_ST, IC6 ISO1042BDWVR, J1 Conn_02x08_Counter_Clockwise, J11 Conn_02x10_Counter_Clockwise, J12 Conn_02x10_Counter_Clockwise, J13 Conn_02x10_Counter_Clockwise, J14 Conn_02x10_Counter_Clockwise, J2 Conn_02x08_Counter_Clockwise, J3 Conn_02x08_Counter_Clockwise, J4 TBP01R1-508-06BE, J5 Conn_02x10_Counter_Clockwise, J6 TBP01R2-508-06BE, K1 AWHSH105D00G, K2 AWHSH105D00G, K3 AWHSH105D00G, Y1 8MHz

Commit message: add board part numbers
Other:
- board text added: "C2-MCB-GEN REVISION A"
- board text added: "SERIAL NUMBER"
- board text removed: "TRACTION INVERTER, GEN 5, MAIN INTERFACE BOARD, REVISION 1, 1200VMAX, 800V WORKING"
Changed lines of the file:
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@@
 			(outputformat 1)
 			(mirror no)
-			(drillshape 1)
+			(drillshape 0)
 			(scaleselection 1)
-			(outputdirectory "")
+			(outputdirectory "Fab/")
 		)
 	)
@@
 	)
 	(gr_rect
-		(start 75 47.5)
-		(end 85 57.5)
+		(start 17 1)
+		(end 27 11)
 		(stroke
 			(width 0.1)
@@
 		)
 	)
-	(gr_text "TRACTION INVERTER, GEN 5,\nMAIN INTERFACE BOARD,\nREVISION 1,\n1200VMAX, 800V WORKING"
-		(at 13.5 11.5 0)
+	(gr_text "C2-MCB-GEN\nREVISION A"
+		(at 31 6 0)
 		(layer "F.SilkS")
 		(effects
@@
 		)
 	)
+	(gr_text "SERIAL NUMBER"
+		(at 22 13 0)
+		(layer "F.SilkS")
+		(effects
+			(font
+				(size 1.25 1.25)
+				(thickness 0.3)
+				(bold yes)
+			)
+			(justify bottom)
+		)
+	)
 	(gr_text "CONN. TO PH U GATE DRIVER"
 		(at 235 58 0)
@@
 	)
 	(gr_text "ISOLATED VOLTAGE SENSE"
-		(at 6 17 0)
+		(at 7 43 0)
 		(layer "F.SilkS")
 		(effects
