File: Boards/ControlBoard/ControlBoard.kicad_pcb (KiCad board)
At the start: 6 copper layers, 297.5 x 60 mm, 138 parts, among them IC3 MAX22530AWE+, IC4 MAX22530AWE+, J1 TBP02R2W-381-06BE, J11 Conn_02x10_Counter_Clockwise, J12 Conn_02x10_Counter_Clockwise, J13 Conn_02x10_Counter_Clockwise, J14 Conn_02x10_Counter_Clockwise, J2 TBP02R2W-381-06BE, J29 Conn_01x02_Pin, J3 TBP01R2W-508-02BE, J4 TBP01R1-508-04BE, J5 Conn_02x10_Counter_Clockwise, J7 TBP02R2W-381-08BE, J8 TBP02R2W-381-08BE

Commit message: add shell wip
Other:
- board text added: "C2-CTRL-XX12 REVISION A"
- board text added: "SERIAL NUMBER"
- board text added: "[ ] 12VIN NOM [ ] 15VIN NOM [ ] 24VIN NOM [ ] 48VIN NOM"
- board text removed: "TRACTION INVERTER, GEN 5, CONTROL BOARD, REVISION 1, 1200VMAX, 800V WORKING"
Changed lines of the file:
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@@
 			(fill no)
 			(layer "Cmts.User")
-			(net 103194064)
 		)
 		(fp_circle
@@
 			(fill no)
 			(layer "F.CrtYd")
-			(net 103194064)
 		)
 		(fp_text user "${REFERENCE}"
@@
 			(fill no)
 			(layer "Cmts.User")
-			(net 103194064)
 		)
 		(fp_circle
@@
 			(fill no)
 			(layer "F.CrtYd")
-			(net 103194064)
 		)
 		(fp_text user "${REFERENCE}"
@@
 	)
 	(gr_rect
-		(start 219 37)
-		(end 229 47)
+		(start 221 31)
+		(end 231 41)
 		(stroke
 			(width 0.1)
@@
 		)
 	)
+	(gr_text "SERIAL NUMBER"
+		(at 217 44 0)
+		(layer "F.SilkS")
+		(effects
+			(font
+				(size 1.5 1.5)
+				(thickness 0.3)
+				(bold yes)
+			)
+			(justify left bottom)
+		)
+	)
 	(gr_text "DANGER!\nHAZARDOUS VOLTAGES PRESENT\nREMOVE POWER AND VERIFY\nCAPACITORS DISCHARGED BEFORE SERVICING"
 		(at 124 54 0)
@@
 		)
 	)
-	(gr_text "TRACTION INVERTER, GEN 5,\nCONTROL BOARD,\nREVISION 1,\n1200VMAX, 800V WORKING"
-		(at 197 58 0)
+	(gr_text "C2-CTRL-XX12\nREVISION A"
+		(at 197 53 0)
 		(layer "F.SilkS")
 		(effects
@@
 				(bold yes)
 			)
+			(justify left bottom)
+		)
+	)
+	(gr_text "[ ] 12VIN NOM\n[ ] 15VIN NOM\n[ ] 24VIN NOM\n[ ] 48VIN NOM"
+		(at 216 58 0)
+		(layer "F.SilkS")
+		(effects
+			(font
+				(size 1.5 1.5)
+				(thickness 0.3)
+				(bold yes)
+			)
