File: Hardware/Chassis0/Boards/GateDriverBoard/GateDriver.kicad_sch (KiCad schematic)
At the start: 32 parts, among them IC7 ADUM4136BRWZ

Commit message: Update chassis 0 gate driver board, remove old files
Parts:
- removed C126, C46, C48: 10uF, Capacitor_SMD:C_1210_3225Metric_Pad1.33x2.70mm_HandSolder, symbol Device:C
- removed C183: UCM1H101MCL1GS, InverterCom:CAPAE660X800N, symbol InverterCom:UCM1H101MCL1GS
- removed D1: BAT54WS-7-F, InverterCom:SOD2513X120N, symbol InverterCom:BAT54WS-7-F
- removed FB1: FBMJ1608HS220NTR, InverterCom:BEADC1608X100N, symbol InverterCom:FBMJ1608HS220NTR
- removed LED10, LED7: LTST-C230GKT, InverterCom:LEDC3216X120N, symbol InverterCom:LTST-C230GKT
- removed LED8, LED9: LTST-C230CKT, InverterCom:LEDC3216X120N, symbol InverterCom:LTST-C230CKT
- removed R14, R22, R23: 4.7k, Resistor_SMD:R_1210_3225Metric_Pad1.30x2.65mm_HandSolder, symbol Device:R
- removed R15: 220, Resistor_SMD:R_1210_3225Metric_Pad1.30x2.65mm_HandSolder, symbol Device:R
- removed R16, R21: 0, Resistor_SMD:R_1210_3225Metric_Pad1.30x2.65mm_HandSolder, symbol Device:R
- removed R17: 9.1, Resistor_SMD:R_1210_3225Metric_Pad1.30x2.65mm_HandSolder, symbol Device:R
- removed R18: 6.8, Resistor_SMD:R_1210_3225Metric_Pad1.30x2.65mm_HandSolder, symbol Device:R
- added C3, C9: UCM1H101MCL1GS, CAPAE660X800N, symbol InverterCom:UCM1H101MCL1GS
Connections:
- net +12V_A: now also C3.1 (+), C9.1 (+)
- net GATE_B: now also IC7.11 (VOUT)
- net GND_A: now also C3.2 (-), C9.2 (-)
Other:
- note removed: "DESAT DISABLE RESISTOR"
- note removed: "GREEN LED FOR +12V_A DC/DC INPUT"
- note removed: "GREEN LED FOR +15V_B GATE DRIVE RAIL"
- note removed: "RED LED FOR -9V_B GATE DRIVER RAIL"
- note removed: "RED POWER LED FOR GATE DRIVER +5V_A"
- note removed: "When tuning this driver for other power stages make sure to adjust the gate drive resistors."
