File: Hardware/Chassis0/Boards/GateDriverBoard/GateDriverBoard.kicad_pcb (KiCad board)
At the start: 6 copper layers, 180 x 52.5 mm, 22 parts, among them IC10 ADUM4136BRWZ, IC11 ADUM4136BRWZ, IC12 ADUM4136BRWZ, IC7 ADUM4136BRWZ, IC8 ADUM4136BRWZ, IC9 ADUM4136BRWZ, J5 Conn_02x08_Counter_Clockwise, J6 Conn_02x08_Counter_Clockwise, J7 Conn_02x08_Counter_Clockwise, J8 Conn_02x08_Counter_Clockwise, J9 Conn_02x08_Counter_Clockwise

Commit message: Update chassis 0 gate driver board, remove old files
Parts:
- added C10: UCM1H101MCL1GS, InverterCom:CAPAE660X800N, F.Cu at (162.5, 84.5)
- added C100: 100nF, Capacitor_SMD:C_1210_3225Metric_Pad1.33x2.70mm_HandSolder, F.Cu at (125.5, 90.7)
- added C101: 10uF, Capacitor_SMD:C_1210_3225Metric_Pad1.33x2.70mm_HandSolder, F.Cu at (114.0, 97.0)
- added C102: 10uF, Capacitor_SMD:C_1210_3225Metric_Pad1.33x2.70mm_HandSolder, F.Cu at (126.5, 95.0)
- added C103: 100nF, Capacitor_SMD:C_1210_3225Metric_Pad1.33x2.70mm_HandSolder, F.Cu at (118.6, 89.7)
- added C104: 10uF, Capacitor_SMD:C_1210_3225Metric_Pad1.33x2.70mm_HandSolder, B.Cu at (126.5, 95.0)
- added C106: 100nF, Capacitor_SMD:C_1210_3225Metric_Pad1.33x2.70mm_HandSolder, B.Cu at (117.0, 101.0)
- added C11: UCM1H101MCL1GS, InverterCom:CAPAE660X800N, F.Cu at (162.5, 93.5)
- added C12: UCM1H101MCL1GS, InverterCom:CAPAE660X800N, F.Cu at (29.4, 73.5)
- added C13: UCM1H101MCL1GS, InverterCom:CAPAE660X800N, F.Cu at (58.9, 73.0)
- added C14: UCM1H101MCL1GS, InverterCom:CAPAE660X800N, F.Cu at (131.0, 63.0)
- added C3: UCM1H101MCL1GS, InverterCom:CAPAE660X800N, F.Cu at (140.8, 63.0)
- added C38: 100nF, Capacitor_SMD:C_1210_3225Metric_Pad1.33x2.70mm_HandSolder, F.Cu at (17.4, 74.0)
- added C39: 10uF, Capacitor_SMD:C_1210_3225Metric_Pad1.33x2.70mm_HandSolder, F.Cu at (17.4, 70.5)
- added C4: UCM1H101MCL1GS, InverterCom:CAPAE660X800N, F.Cu at (150.8, 63.0)
- added C40: 100nF, Capacitor_SMD:C_1210_3225Metric_Pad1.33x2.70mm_HandSolder, F.Cu at (33.0, 88.0)
- added C41: 100nF, Capacitor_SMD:C_1210_3225Metric_Pad1.33x2.70mm_HandSolder, F.Cu at (45.0, 90.5)
- added C42: 10uF, Capacitor_SMD:C_1210_3225Metric_Pad1.33x2.70mm_HandSolder, F.Cu at (40.0, 96.0)
- added C43: 10uF, Capacitor_SMD:C_1210_3225Metric_Pad1.33x2.70mm_HandSolder, B.Cu at (45.5, 95.0)
- added C44: 100nF, Capacitor_SMD:C_1210_3225Metric_Pad1.33x2.70mm_HandSolder, F.Cu at (38.0, 89.5)
- added C45: 10uF, Capacitor_SMD:C_1210_3225Metric_Pad1.33x2.70mm_HandSolder, F.Cu at (45.5, 95.0)
- added C47: 100nF, Capacitor_SMD:C_1210_3225Metric_Pad1.33x2.70mm_HandSolder, B.Cu at (37.0, 100.0)
- added C5: UCM1H101MCL1GS, InverterCom:CAPAE660X800N, F.Cu at (159.0, 74.5)
- added C53: 100nF, Capacitor_SMD:C_1210_3225Metric_Pad1.33x2.70mm_HandSolder, F.Cu at (40.4, 74.0)
- added C54: 10uF, Capacitor_SMD:C_1210_3225Metric_Pad1.33x2.70mm_HandSolder, F.Cu at (40.4, 70.5)
- added C55: 100nF, Capacitor_SMD:C_1210_3225Metric_Pad1.33x2.70mm_HandSolder, F.Cu at (10.0, 88.0)
- added C56: 100nF, Capacitor_SMD:C_1210_3225Metric_Pad1.33x2.70mm_HandSolder, F.Cu at (22.0, 90.5)
- added C57: 10uF, Capacitor_SMD:C_1210_3225Metric_Pad1.33x2.70mm_HandSolder, F.Cu at (11.0, 96.0)
- added C58: 10uF, Capacitor_SMD:C_1210_3225Metric_Pad1.33x2.70mm_HandSolder, F.Cu at (23.0, 95.0)
- added C59: 100nF, Capacitor_SMD:C_1210_3225Metric_Pad1.33x2.70mm_HandSolder, F.Cu at (15.0, 90.0)
- added C6: UCM1H101MCL1GS, InverterCom:CAPAE660X800N, F.Cu at (6.35, 73.0)
- added C60: 10uF, Capacitor_SMD:C_1210_3225Metric_Pad1.33x2.70mm_HandSolder, B.Cu at (23.0, 94.5)
- added C62: 100nF, Capacitor_SMD:C_1210_3225Metric_Pad1.33x2.70mm_HandSolder, B.Cu at (14.0, 100.0)
- added C64: 100nF, Capacitor_SMD:C_1210_3225Metric_Pad1.33x2.70mm_HandSolder, F.Cu at (142.9, 70.7)
- added C65: 10uF, Capacitor_SMD:C_1210_3225Metric_Pad1.33x2.70mm_HandSolder, F.Cu at (142.9, 74.2)
- added C66: 100nF, Capacitor_SMD:C_1210_3225Metric_Pad1.33x2.70mm_HandSolder, F.Cu at (85.5, 88.2)
- added C67: 100nF, Capacitor_SMD:C_1210_3225Metric_Pad1.33x2.70mm_HandSolder, F.Cu at (97.0, 90.7)
- added C68: 10uF, Capacitor_SMD:C_1210_3225Metric_Pad1.33x2.70mm_HandSolder, F.Cu at (99.0, 96.0)
- added C69: 10uF, Capacitor_SMD:C_1210_3225Metric_Pad1.33x2.70mm_HandSolder, F.Cu at (85.9, 94.5)
- added C7: UCM1H101MCL1GS, InverterCom:CAPAE660X800N, F.Cu at (82.3, 73.9)
- added C70: 100nF, Capacitor_SMD:C_1210_3225Metric_Pad1.33x2.70mm_HandSolder, F.Cu at (90.5, 89.7)
- added C71: 10uF, Capacitor_SMD:C_1210_3225Metric_Pad1.33x2.70mm_HandSolder, B.Cu at (85.9, 94.5)
- added C73: 100nF, Capacitor_SMD:C_1210_3225Metric_Pad1.33x2.70mm_HandSolder, B.Cu at (96.0, 100.0)
- added C75: 100nF, Capacitor_SMD:C_1210_3225Metric_Pad1.33x2.70mm_HandSolder, F.Cu at (69.9, 70.4)
- added C76: 10uF, Capacitor_SMD:C_1210_3225Metric_Pad1.33x2.70mm_HandSolder, F.Cu at (69.9, 73.9)
- added C77: 100nF, Capacitor_SMD:C_1210_3225Metric_Pad1.33x2.70mm_HandSolder, F.Cu at (62.5, 88.2)
- added C78: 100nF, Capacitor_SMD:C_1210_3225Metric_Pad1.33x2.70mm_HandSolder, F.Cu at (74.5, 90.7)
- added C79: 10uF, Capacitor_SMD:C_1210_3225Metric_Pad1.33x2.70mm_HandSolder, F.Cu at (70.0, 96.0)
- added C8: UCM1H101MCL1GS, InverterCom:CAPAE660X800N, F.Cu at (132.8, 73.0)
- added C80: 10uF, Capacitor_SMD:C_1210_3225Metric_Pad1.33x2.70mm_HandSolder, F.Cu at (63.6, 95.5)
- added C81: 100nF, Capacitor_SMD:C_1210_3225Metric_Pad1.33x2.70mm_HandSolder, F.Cu at (67.5, 89.7)
- added C82: 10uF, Capacitor_SMD:C_1210_3225Metric_Pad1.33x2.70mm_HandSolder, B.Cu at (63.5, 95.5)
- added C84: 100nF, Capacitor_SMD:C_1210_3225Metric_Pad1.33x2.70mm_HandSolder, B.Cu at (73.0, 100.0)
- added C86: 100nF, Capacitor_SMD:C_1210_3225Metric_Pad1.33x2.70mm_HandSolder, F.Cu at (92.9, 73.9)
- added C87: 10uF, Capacitor_SMD:C_1210_3225Metric_Pad1.33x2.70mm_HandSolder, F.Cu at (92.9, 70.4)
- added C88: 100nF, Capacitor_SMD:C_1210_3225Metric_Pad1.33x2.70mm_HandSolder, F.Cu at (135.5, 88.2)
- added C89: 100nF, Capacitor_SMD:C_1210_3225Metric_Pad1.33x2.70mm_HandSolder, F.Cu at (147.5, 90.7)
- added C9: UCM1H101MCL1GS, InverterCom:CAPAE660X800N, F.Cu at (110.2, 73.5)
- added C90: 10uF, Capacitor_SMD:C_1210_3225Metric_Pad1.33x2.70mm_HandSolder, F.Cu at (143.0, 97.0)
- added C91: 10uF, Capacitor_SMD:C_1210_3225Metric_Pad1.33x2.70mm_HandSolder, F.Cu at (148.5, 95.5)
- added C92: 100nF, Capacitor_SMD:C_1210_3225Metric_Pad1.33x2.70mm_HandSolder, F.Cu at (140.5, 89.7)
- added C93: 10uF, Capacitor_SMD:C_1210_3225Metric_Pad1.33x2.70mm_HandSolder, B.Cu at (148.5, 95.5)
- added C95: 100nF, Capacitor_SMD:C_1210_3225Metric_Pad1.33x2.70mm_HandSolder, B.Cu at (139.5, 101.0)
- added C97: 100nF, Capacitor_SMD:C_1210_3225Metric_Pad1.33x2.70mm_HandSolder, F.Cu at (120.9, 70.7)
- added C98: 10uF, Capacitor_SMD:C_1210_3225Metric_Pad1.33x2.70mm_HandSolder, F.Cu at (120.9, 74.2)
- added C99: 100nF, Capacitor_SMD:C_1210_3225Metric_Pad1.33x2.70mm_HandSolder, F.Cu at (113.5, 88.2)
- added D11: FM2000GP-TP, InverterCom:DIOM5226X244N, F.Cu at (135.0, 99.0)
- added D13: FM2000GP-TP, InverterCom:DIOM5226X244N, F.Cu at (122.0, 99.2)
- added D14: FM2000GP-TP, InverterCom:DIOM5226X244N, F.Cu at (19.0, 99.0)
- added D2: FM2000GP-TP, InverterCom:DIOM5226X244N, F.Cu at (32.0, 99.0)
- added D7: FM2000GP-TP, InverterCom:DIOM5226X244N, F.Cu at (91.0, 99.0)
- added D9: FM2000GP-TP, InverterCom:DIOM5226X244N, F.Cu at (78.0, 99.2)
- added R1: 4.7k, Resistor_SMD:R_1210_3225Metric_Pad1.30x2.65mm_HandSolder, F.Cu at (83.5, 59.5)
- added R19: 1k, Resistor_SMD:R_1210_3225Metric_Pad1.30x2.65mm_HandSolder, B.Cu at (37.0, 96.0)
- added R2: 4.7k, Resistor_SMD:R_1210_3225Metric_Pad1.30x2.65mm_HandSolder, F.Cu at (90.5, 59.5)
- added R20: 1k, Resistor_SMD:R_1210_3225Metric_Pad1.30x2.65mm_HandSolder, B.Cu at (32.0, 99.0)
- added R3: 4.7k, Resistor_SMD:R_1210_3225Metric_Pad1.30x2.65mm_HandSolder, F.Cu at (75.5, 59.5)
- added R30: 1k, Resistor_SMD:R_1210_3225Metric_Pad1.30x2.65mm_HandSolder, B.Cu at (14.0, 96.0)
- added R31: 1k, Resistor_SMD:R_1210_3225Metric_Pad1.30x2.65mm_HandSolder, B.Cu at (19.0, 99.0)
- added R40: 1k, Resistor_SMD:R_1210_3225Metric_Pad1.30x2.65mm_HandSolder, B.Cu at (96.0, 96.0)
- added R41: 1k, Resistor_SMD:R_1210_3225Metric_Pad1.30x2.65mm_HandSolder, B.Cu at (91.0, 99.0)
- added R50: 1k, Resistor_SMD:R_1210_3225Metric_Pad1.30x2.65mm_HandSolder, B.Cu at (73.0, 96.0)
- added R51: 1k, Resistor_SMD:R_1210_3225Metric_Pad1.30x2.65mm_HandSolder, B.Cu at (78.0, 99.0)
- added R60: 1k, Resistor_SMD:R_1210_3225Metric_Pad1.30x2.65mm_HandSolder, B.Cu at (139.5, 97.0)
- added R61: 1k, Resistor_SMD:R_1210_3225Metric_Pad1.30x2.65mm_HandSolder, B.Cu at (135.0, 99.0)
- added R70: 1k, Resistor_SMD:R_1210_3225Metric_Pad1.30x2.65mm_HandSolder, B.Cu at (117.0, 97.0)
- added R71: 1k, Resistor_SMD:R_1210_3225Metric_Pad1.30x2.65mm_HandSolder, B.Cu at (122.0, 99.0)
- added TP36: TestPoint, TestPoint:TestPoint_Loop_D2.54mm_Drill1.5mm_Beaded, F.Cu at (77.5, 63.5)
- added TP37: TestPoint, TestPoint:TestPoint_Loop_D2.54mm_Drill1.5mm_Beaded, F.Cu at (85.0, 63.5)
- added TP38: TestPoint, TestPoint:TestPoint_Loop_D2.54mm_Drill1.5mm_Beaded, F.Cu at (92.0, 63.5)
- added TP39: TestPoint, TestPoint:TestPoint_Loop_D2.54mm_Drill1.5mm_Beaded, F.Cu at (68.5, 63.0)
- moved IC7 30.1 mm to (40.0, 82.0), turned to -90 degrees
- moved IC8 18.1 mm to (17.0, 82.5), turned to -90 degrees
- moved IC12 10.8 mm to (120.4, 82.0), turned to -90 degrees
- moved PS12 10.8 mm to (120.4, 82.0)
- moved IC10 10.0 mm to (69.5, 81.7), turned to -90 degrees
- moved PS10 10.0 mm to (69.5, 82.0)
- moved IC11 8.20 mm to (142.6, 82.0), turned to -90 degrees
- moved PS11 8.20 mm to (142.6, 82.0)
- moved IC9 7.95 mm to (92.4, 82.0), turned to -90 degrees
- moved PS9 7.95 mm to (92.4, 82.0)
- moved PS8 7.62 mm to (17.0, 82.0)
- moved PS5 5.83 mm to (40.0, 82.0)
- moved J7 1.25 mm to (7.42, 62.5)
Connections:
- IC10 pad 11: Net-(D8-K) -> /PH_V_L_G
- IC11 pad 11: Net-(D10-K) -> /PH_W_H_G
- IC12 pad 11: Net-(D12-K) -> /PH_W_L_G
- IC7 pad 11: Net-(D1-K) -> /PH_U_H_G
- IC8 pad 11: Net-(D5-K) -> /PH_U_L_G
- IC9 pad 11: Net-(D6-K) -> /PH_V_H_G
Routing:
- net /RESET: track 0.00 -> 195.4 mm, vias 0 -> 18
- net /FAULT: track 0.00 -> 190.2 mm, vias 0 -> 8
- net /READY: track 0.00 -> 185.8 mm, vias 0 -> 9
- net /PH_W_L: track 0.00 -> 161.2 mm, vias 0 -> 3
- net /PH_W_H: track 0.00 -> 157.4 mm, vias 0 -> 3
- net /PH_V_H: track 0.00 -> 115.2 mm, vias 0 -> 3
- net /PH_V_L: track 0.00 -> 113.7 mm, vias 0 -> 3
- net /PH_U_H: track 0.00 -> 66.6 mm, vias 0 -> 3
- net /PH_U_L: track 0.00 -> 57.7 mm, vias 0 -> 3
- net /GND_A: track 0.00 -> 44.2 mm, vias 0 -> 30
- net /+3.3V_A: track 0.00 -> 40.2 mm, vias 0 -> 16
- net /PH_U_H_G: track 0.00 -> 26.1 mm
- net /PH_W_H_G: track 0.00 -> 25.7 mm
- net /PH_V_L_G: track 0.00 -> 22.7 mm
- net /PH_W_H_S: track 0.00 -> 21.3 mm, vias 0 -> 4
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- added copper zone on In3.Cu, net /+12V_A
- added copper zone on In2.Cu, net /+3.3V_A
- added copper zone on B.Cu, net /GND_A
- added copper zone on F.Cu, net /GND_A
- added copper zone on In1.Cu, net /GND_A
- added copper zone on In4.Cu, net /GND_A
- added copper zone on In2.Cu, net /GateDriverAssembly/GateDriver_PH_U_H/+15V_B
- added copper zone on In3.Cu, net /GateDriverAssembly/GateDriver_PH_U_H/-9V_B
- added copper zone on In2.Cu, net /GateDriverAssembly/GateDriver_PH_U_L/+15V_B
- added copper zone on In3.Cu, net /GateDriverAssembly/GateDriver_PH_U_L/-9V_B
- added copper zone on In2.Cu, net /GateDriverAssembly/GateDriver_PH_V_H/+15V_B
- added copper zone on In3.Cu, net /GateDriverAssembly/GateDriver_PH_V_H/-9V_B
- added copper zone on In2.Cu, net /GateDriverAssembly/GateDriver_PH_V_L/+15V_B
- added copper zone on In3.Cu, net /GateDriverAssembly/GateDriver_PH_V_L/-9V_B
- added copper zone on In2.Cu, net /GateDriverAssembly/GateDriver_PH_W_H/+15V_B
- added copper zone on In3.Cu, net /GateDriverAssembly/GateDriver_PH_W_H/-9V_B
- added copper zone on In2.Cu, net /GateDriverAssembly/GateDriver_PH_W_L/+15V_B
- added copper zone on In3.Cu, net /GateDriverAssembly/GateDriver_PH_W_L/-9V_B
- added copper zone on B.Cu, net /PH_U_H_S
- added copper zone on F.Cu, net /PH_U_H_S
- added copper zone on In1.Cu, net /PH_U_H_S
- added copper zone on In4.Cu, net /PH_U_H_S
- added copper zone on B.Cu, net /PH_U_L_S
- added copper zone on F.Cu, net /PH_U_L_S
- added copper zone on In1.Cu, net /PH_U_L_S
- added copper zone on In4.Cu, net /PH_U_L_S
- added copper zone on B.Cu, net /PH_V_H_S
- added copper zone on F.Cu, net /PH_V_H_S
- added copper zone on In1.Cu, net /PH_V_H_S
- added copper zone on In4.Cu, net /PH_V_H_S
- added copper zone on B.Cu, net /PH_V_L_S
- added copper zone on F.Cu, net /PH_V_L_S
- added copper zone on In1.Cu, net /PH_V_L_S
- added copper zone on In4.Cu, net /PH_V_L_S
- added copper zone on B.Cu, net /PH_W_H_S
- added copper zone on F.Cu, net /PH_W_H_S
- added copper zone on In1.Cu, net /PH_W_H_S
- added copper zone on In4.Cu, net /PH_W_H_S
- added copper zone on B.Cu, net /PH_W_L_S
- added copper zone on F.Cu, net /PH_W_L_S
- added copper zone on In1.Cu, net /PH_W_L_S
- added copper zone on In4.Cu, net /PH_W_L_S
