File: Hardware/Chassis0/Boards/ControlBoard/ADC1.kicad_sch (KiCad schematic)
At the start: 31 parts, among them IC1 MAX22530AWE+, IC2 MAX22530AWE+

Commit message: finish chassis 0 board design v1
Parts:
- removed LED1, LED35: LTST-C230GKT, InverterCom:LEDC3216X120N, symbol InverterCom:LTST-C230GKT
- removed LED2: LTST-C230CKT, InverterCom:LEDC3216X120N, symbol InverterCom:LTST-C230CKT
- removed R125, R4: 220, Resistor_SMD:R_1210_3225Metric_Pad1.30x2.65mm_HandSolder, symbol Device:R
- removed R5: 1k, Resistor_SMD:R_1210_3225Metric_Pad1.30x2.65mm_HandSolder, symbol Device:R
- removed TP1, TP10, TP2, TP3, TP4, TP5, TP6, TP7, TP8, TP9: TestPoint, TestPoint:TestPoint_Loop_D2.54mm_Drill1.5mm_Beaded, symbol Connector:TestPoint
Other:
- note removed: "GREEN LED FOR +3.3V ADC POWER"
- note removed: "GREEN LED FOR +5V CURRENT SENSE RAIL"
