File: Hardware/Chassis0/Boards/ControlBoard/ADC2.kicad_sch (KiCad schematic)
At the start: 20 parts, among them IC3 MAX22530AWE+, IC4 MAX22530AWE+

Commit message: finish chassis 0 board design v1
Parts:
- removed LED3, LED4: LTST-C230CKT, InverterCom:LEDC3216X120N, symbol InverterCom:LTST-C230CKT
- removed R6, R7: 1k, Resistor_SMD:R_1210_3225Metric_Pad1.30x2.65mm_HandSolder, symbol Device:R
- removed TP11, TP12: TestPoint, TestPoint:TestPoint_Loop_D2.54mm_Drill1.5mm_Beaded, symbol Connector:TestPoint
Other:
- note removed: "RED LED FOR AUX +5V RAIL"
- note removed: "RED LED FOR HALL +5V RAIL"
