File: Hardware/Chassis0/Boards/ControlBoard/CAN.kicad_sch (KiCad schematic)
At the start: 24 parts, among them IC5 MCP2515-e_ST, IC6 ISO1042BDWVR, Y1 8MHz

Commit message: finish chassis 0 board design v1
Parts:
- removed LED5: LTST-C230GKT, InverterCom:LEDC3216X120N, symbol InverterCom:LTST-C230GKT
- removed LED6: LTST-C230CKT, InverterCom:LEDC3216X120N, symbol InverterCom:LTST-C230CKT
- removed R10, R11: 220, Resistor_SMD:R_1210_3225Metric_Pad1.30x2.65mm_HandSolder, symbol Device:R
Other:
- note removed: "GREEN LED FOR +3.3V CANBUS TRANSCIEVER INPUT"
- note removed: "GREEN POWER LED FOR CAN CAN_ISO_5V"
