File: Hardware/Chassis0/Boards/ControlBoard/Control.kicad_sch (KiCad schematic)
At the start: 16 parts, among them J29 Conn_01x02_Pin

Commit message: finish chassis 0 board design v1
Parts:
- removed R12: 0, Resistor_SMD:R_1210_3225Metric_Pad1.30x2.65mm_HandSolder, symbol Device:R
- removed TP21, TP22, TP23, TP24, TP29, TP30, TP31, TP32, TP33, TP34, TP35: TestPoint, TestPoint:TestPoint_Loop_D2.54mm_Drill1.5mm_Beaded, symbol Connector:TestPoint
Connections:
- net GND_A: now also A1.33 (AGND)
