File: Hardware/Chassis2/Boards/DCBusCapacitorBoard/DCBusCapacitorBoard.kicad_pcb (KiCad board)
At the start: 4 copper layers, 89 x 85 mm, 16 parts

Commit message: Add power stage wip design for size 0
Parts:
- moved C8 2.00 mm to (38.0, 23.0)
- moved C6 1.00 mm to (65.0, 22.0)
Changed lines of the file:
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@@
 	(footprint "InverterCom:CAPPRD750W80D1825H3200"
 		(layer "F.Cu")
-		(at 65 21 180)
+		(at 65 22 180)
 		(descr "18mm x 30.5mm")
 		(tags "Capacitor")
@@
 	(footprint "InverterCom:CAPPRD750W80D1825H3200"
 		(layer "F.Cu")
-		(at 38 21 180)
+		(at 38 23 180)
 		(descr "18mm x 30.5mm")
 		(tags "Capacitor")

Commit message: update dc bus board
Routing:
- added copper zone on In1.Cu, net /DC_LINK_+
- added copper zone on In2.Cu, net /DC_LINK_-
Changed lines of the file:
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@@
 		(net 1)
 		(net_name "/DC_LINK_+")
-		(layer "F.Cu")
+		(layers "F.Cu" "In1.Cu")
 		(hatch edge 0.5)
 		(connect_pads yes
@@
 		(net 2)
 		(net_name "/DC_LINK_-")
-		(layer "B.Cu")
+		(layers "B.Cu" "In2.Cu")
 		(hatch edge 0.5)
 		(connect_pads yes
