File: Hardware/Chassis2/Boards/DCBusCapacitorBoard/DCBusCapacitorBoard.kicad_pcb (KiCad board)
At the start: 4 copper layers, 89 x 85 mm, 16 parts

Commit message: Powerstage intermediate rework
Parts:
- added C13: UCS2D331MHD, InverterCom:CAPPRD750W80D1800H3700, B.Cu at (52.2, 77.0)
- added C14: UCS2D331MHD, InverterCom:CAPPRD750W80D1800H3700, B.Cu at (60.2, 18.5)
- added C15: UCS2D331MHD, InverterCom:CAPPRD750W80D1800H3700, B.Cu at (90.5, 77.0)
- added C16: UCS2D331MHD, InverterCom:CAPPRD750W80D1800H3700, B.Cu at (33.2, 77.0)
- added C17: UCS2D331MHD, InverterCom:CAPPRD750W80D1800H3700, B.Cu at (160.2, 1.00)
- added C18: UCS2D331MHD, InverterCom:CAPPRD750W80D1800H3700, B.Cu at (68.8, 0.50)
- added C19: UCS2D331MHD, InverterCom:CAPPRD750W80D1800H3700, B.Cu at (84.8, 10.5)
- added C20: UCS2D331MHD, InverterCom:CAPPRD750W80D1800H3700, B.Cu at (83.5, 60.0)
- added C21: UCS2D331MHD, InverterCom:CAPPRD750W80D1800H3700, B.Cu at (71.2, 77.0)
- added C22: UCS2D331MHD, InverterCom:CAPPRD750W80D1800H3700, B.Cu at (151.5, 18.0)
- added C23: UCS2D331MHD, InverterCom:CAPPRD750W80D1800H3700, B.Cu at (124.2, 50.0)
- added C24: UCS2D331MHD, InverterCom:CAPPRD750W80D1800H3700, B.Cu at (109.2, 77.0)
- added C25: UCS2D331MHD, InverterCom:CAPPRD750W80D1800H3700, B.Cu at (106.5, 0.50)
- added C26: UCS2D331MHD, InverterCom:CAPPRD750W80D1800H3700, B.Cu at (95.2, 26.0)
- added C27: UCS2D331MHD, InverterCom:CAPPRD750W80D1800H3700, B.Cu at (94.0, 44.5)
- added C28: UCS2D331MHD, InverterCom:CAPPRD750W80D1800H3700, B.Cu at (107.0, 58.5)
- added C29: UCS2D331MHD, InverterCom:CAPPRD750W80D1800H3700, B.Cu at (247.2, 10.0)
- added C30: UCS2D331MHD, InverterCom:CAPPRD750W80D1800H3700, B.Cu at (167.2, 28.0)
- added C31: UCS2D331MHD, InverterCom:CAPPRD750W80D1800H3700, B.Cu at (172.0, 47.0)
- added C32: UCS2D331MHD, InverterCom:CAPPRD750W80D1800H3700, B.Cu at (181.5, 64.0)
- added C33: UCS2D331MHD, InverterCom:CAPPRD750W80D1800H3700, B.Cu at (176.2, 11.0)
- added C34: UCS2D331MHD, InverterCom:CAPPRD750W80D1800H3700, B.Cu at (132.2, 16.0)
- added C35: UCS2D331MHD, InverterCom:CAPPRD750W80D1800H3700, B.Cu at (113.8, 18.0)
- added C36: UCS2D331MHD, InverterCom:CAPPRD750W80D1800H3700, B.Cu at (110.8, 36.5)
- added C37: UCS2D331MHD, InverterCom:CAPPRD750W80D1800H3700, B.Cu at (191.8, 21.5)
- added C38: UCS2D331MHD, InverterCom:CAPPRD750W80D1800H3700, B.Cu at (189.2, 40.0)
- added C39: UCS2D331MHD, InverterCom:CAPPRD750W80D1800H3700, B.Cu at (198.8, 56.5)
- added C40: UCS2D331MHD, InverterCom:CAPPRD750W80D1800H3700, B.Cu at (166.2, 77.0)
- added C41: UCS2D331MHD, InverterCom:CAPPRD750W80D1800H3700, B.Cu at (209.2, 15.0)
- added C42: UCS2D331MHD, InverterCom:CAPPRD750W80D1800H3700, B.Cu at (153.2, 41.0)
- added C43: UCS2D331MHD, InverterCom:CAPPRD750W80D1800H3700, B.Cu at (157.5, 60.0)
- added C44: UCS2D331MHD, InverterCom:CAPPRD750W80D1800H3700, B.Cu at (147.2, 77.0)
- added C45: UCS2D331MHD, InverterCom:CAPPRD750W80D1800H3700, B.Cu at (285.2, 10.0)
- added C46: UCS2D331MHD, InverterCom:CAPPRD750W80D1800H3700, B.Cu at (196.8, 0.50)
- added C47: UCS2D331MHD, InverterCom:CAPPRD750W80D1800H3700, B.Cu at (206.8, 33.5)
- added C48: UCS2D331MHD, InverterCom:CAPPRD750W80D1800H3700, B.Cu at (197.2, 78.0)
- added C49: UCS2D331MHD, InverterCom:CAPPRD750W80D1800H3700, B.Cu at (229.2, 16.0)
- added C50: UCS2D331MHD, InverterCom:CAPPRD750W80D1800H3700, B.Cu at (128.2, 77.0)
- added C51: UCS2D331MHD, InverterCom:CAPPRD750W80D1800H3700, B.Cu at (216.0, 49.5)
- added C52: UCS2D331MHD, InverterCom:CAPPRD750W80D1800H3700, B.Cu at (217.2, 77.0)
- added C53: UCS2D331MHD, InverterCom:CAPPRD750W80D1800H3700, B.Cu at (244.2, 29.0)
- added C54: UCS2D331MHD, InverterCom:CAPPRD750W80D1800H3700, B.Cu at (244.2, 48.0)
- added C55: UCS2D331MHD, InverterCom:CAPPRD750W80D1800H3700, B.Cu at (251.2, 65.0)
- added C56: UCS2D331MHD, InverterCom:CAPPRD750W80D1800H3700, B.Cu at (236.2, 77.0)
- added C57: UCS2D331MHD, InverterCom:CAPPRD750W80D1800H3700, B.Cu at (266.0, 11.0)
- added C58: UCS2D331MHD, InverterCom:CAPPRD750W80D1800H3700, B.Cu at (263.2, 30.0)
- added C59: UCS2D331MHD, InverterCom:CAPPRD750W80D1800H3700, B.Cu at (263.2, 50.0)
- added C60: UCS2D331MHD, InverterCom:CAPPRD750W80D1800H3700, B.Cu at (266.2, 77.0)
- added H10: MountingHole_Pad, MountingHole:MountingHole_6.4mm_M6_ISO14580_Pad, F.Cu at (275.0, -3.00)
- added H11: MountingHole_Pad, MountingHole:MountingHole_6.4mm_M6_ISO14580_Pad, F.Cu at (285.0, 81.0)
- added H12: MountingHole_Pad, MountingHole:MountingHole_6.4mm_M6_ISO14580_Pad, F.Cu at (185.0, 81.0)
- added H3: MountingHole_Pad, MountingHole:MountingHole_6.4mm_M6_ISO14580_Pad, F.Cu at (140.0, 63.0)
- added H6: MountingHole_Pad, MountingHole:MountingHole_6.4mm_M6_ISO14580_Pad, F.Cu at (230.0, 35.0)
- added H7: MountingHole_Pad, MountingHole:MountingHole_6.4mm_M6_ISO14580_Pad, F.Cu at (6.00, 81.0)
- added H8: MountingHole_Pad, MountingHole:MountingHole_6.4mm_M6_ISO14580_Pad, F.Cu at (95.0, -3.00)
- added H9: MountingHole_Pad, MountingHole:MountingHole_6.4mm_M6_ISO14580_Pad, F.Cu at (185.0, -3.00)
- C1, C10, C11, C12, C2, C3, C4, C5, C6, C7, C8, C9: value UCS2C331MHD -> UCS2D331MHD; footprint InverterCom:CAPPRD750W80D1825H3200 -> InverterCom:CAPPRD750W80D1800H3700; moved to B.Cu
- H4, H5: footprint MountingHole:MountingHole_3.2mm_M3_ISO14580_Pad -> MountingHole:MountingHole_6.4mm_M6_ISO14580_Pad
- moved H5 156.3 mm to (230.0, 63.0)
- moved H4 132.2 mm to (140.0, 35.0)
- moved C2 85.2 mm to (7.25, 11.0), turned to 0 degrees
- moved C3 78.9 mm to (6.25, 30.0), turned to 0 degrees
- moved C12 70.2 mm to (64.2, 59.0), turned to 0 degrees
- moved C5 63.5 mm to (23.5, 1.00), turned to 0 degrees
- moved C8 52.4 mm to (10.2, 67.5), turned to 0 degrees
- moved C11 49.0 mm to (62.5, 40.0), turned to 0 degrees
- moved C9 42.2 mm to (42.0, 14.6), turned to 0 degrees
- moved C6 41.0 mm to (24.0, 20.0), turned to 0 degrees
- moved C4 32.9 mm to (6.25, 49.0), turned to 0 degrees
- moved C10 14.1 mm to (27.2, 59.0), turned to 0 degrees
- moved C7 13.7 mm to (23.2, 40.0), turned to 0 degrees
- moved C1 7.65 mm to (76.3, 28.1), turned to 0 degrees
Connections:
- H4 pad 1: /CHASSIS_GND -> /DC_LINK_-
- H5 pad 1: /CHASSIS_GND_1 -> /DC_LINK_+
Routing:
- removed copper zone on In1.Cu, net /DC_LINK_+
- removed copper zone on In2.Cu, net /DC_LINK_-
Other:
- board size 89 x 85 mm -> 300 x 96.1 mm
- copper layers 4 -> 2
- board text added: "DC LINK CAPACITOR MODULE"
- board text added: "DURING ASSEMBLY MARK VARIANT HERE"
- board text added: "MODULE WILL RETAIN VOLTAGE WHEN DISCONNECTED. CONFIRM DISCHARGED PRIOR TO SERVICING. ENSURE MODULE IS CONNECTED THERMALLY TO HEAT SPREADER BELOW VIA NON-CONDUCTIVE THERMAL INTERFACE MATERIAL."
- board text added: "REV B | 2026-07 | THOMAS LIAO CORZINE SMART POWER LAB"
- board text removed: "BULK CAPACITOR BOARD"
- board text removed: "DANGER: HIGH VOLTAGE"
- board text removed: "DESIGNED BY THOMAS LIAO"
- board text removed: "MODEL: C2-BCB-LV"
- board text removed: "SERIAL NUMBER"
- board text removed: "VARIANT"
- board text removed: "[ ] 160VMAX, 106VNOM [ ] 200VMAX, 132VNOM [ ] 250VMAX, 165VNOM [ ] 350VMAX, 230VNOM [ ] 400VMAX, 265VNOM [ ] 450VMAX, 300VNOM"

Commit message: Update IO Board silkscreen, ExM pinout
Parts:
- added H13: 9774030592R, InverterCom:9774030592R, F.Cu at (12.0, -2.00)
- added H14: 9774030592R, InverterCom:9774030592R, F.Cu at (249.0, -3.00)
- added H15: 9774030592R, InverterCom:9774030592R, F.Cu at (103.0, 13.0)
- added H16: 9774030592R, InverterCom:9774030592R, F.Cu at (269.0, 64.0)
- moved C30 9.85 mm to (176.2, 32.0)
- moved C38 3.81 mm to (190.8, 43.5)
- moved C43 3.78 mm to (153.8, 60.5)
- moved C31 3.40 mm to (169.2, 49.0)
- moved C39 3.25 mm to (200.0, 59.5)
- moved C8 3.16 mm to (13.2, 66.5)
- moved C10 2.92 mm to (28.8, 56.5)
- moved C33 2.66 mm to (174.5, 13.0)
- moved C19 2.50 mm to (83.2, 12.5)
- moved C25 2.25 mm to (108.8, 0.50)
- moved C34 2.14 mm to (133.0, 18.0)
- moved C40 2.06 mm to (165.8, 75.0)
- moved C57 2.02 mm to (265.8, 13.0)
- moved C60 1.82 mm to (264.5, 77.5)
- moved C46 1.75 mm to (198.5, 0.50)
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Other:
- board text added: "DANGER - HIGH VOLTAGE"
- board text added: "SERIAL NUMBER"
- board text added: "TOP CASE MOUNTING HOLE M5, 1.2Nm, USE THREADLOCKER"

Commit message: Update Mechanical Model, Fix Interference Issues
Parts:
- moved C21 2.24 mm to (73.2, 76.0)
- moved C13 2.06 mm to (54.2, 77.5)
- moved C15 1.35 mm to (91.8, 77.5)
- moved C24 0.90 mm to (110.2, 76.5)
- moved C50 0.71 mm to (128.8, 77.5)
- moved C1 0.50 mm to (77.2, 30.0)
- moved C12 0.50 mm to (64.8, 59.0)
- moved C20 0.50 mm to (83.0, 60.0)
- moved C28 0.50 mm to (106.5, 58.5)
Other:
- board size 300 x 96.1 mm -> 297 x 96.1 mm
Changed lines of the file:
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@@
 		(capping no)
 		(filling no)
-		(zone_defaults)
 		(pcbplotparams
 			(layerselection 0x00000000_00000000_55555555_5755f5ff)
@@
 	(footprint "InverterCom:CAPPRD750W80D1800H3700"
 		(layer "B.Cu")
-		(at 106.5 59)
+		(at 106.5 58.5)
 		(descr "UCS2D331MHD")
 		(tags "Capacitor")
@@
 		)
 		(fp_text user "-"
-			(at 12.75 0 180)
+			(at 10 -1.5 180)
 			(unlocked yes)
 			(layer "B.SilkS")
@@
 	(footprint "InverterCom:CAPPRD750W80D1800H3700"
 		(layer "B.Cu")
-		(at 71.25 77)
+		(at 73.25 76)
 		(descr "UCS2D331MHD")
 		(tags "Capacitor")
@@
 	(footprint "InverterCom:CAPPRD750W80D1800H3700"
 		(layer "B.Cu")
-		(at 64.25 59)
+		(at 64.75 59)
 		(descr "UCS2D331MHD")
 		(tags "Capacitor")
@@
 	(footprint "InverterCom:CAPPRD750W80D1800H3700"
 		(layer "B.Cu")
-		(at 52.25 77)
+		(at 54.25 77.5)
 		(descr "UCS2D331MHD")
 		(tags "Capacitor")
@@
 	(footprint "InverterCom:CAPPRD750W80D1800H3700"
 		(layer "B.Cu")
-		(at 128.25 77)
+		(at 128.75 77.5)
 		(descr "UCS2D331MHD")
 		(tags "Capacitor")
@@
 	(footprint "InverterCom:CAPPRD750W80D1800H3700"
 		(layer "B.Cu")
-		(at 109.5 77)
+		(at 110.25 76.5)
 		(descr "UCS2D331MHD")
 		(tags "Capacitor")
@@
 	(footprint "InverterCom:CAPPRD750W80D1800H3700"
 		(layer "B.Cu")
-		(at 83.5 60)
+		(at 83 60)
 		(descr "UCS2D331MHD")
 		(tags "Capacitor")
@@
 	(footprint "InverterCom:CAPPRD750W80D1800H3700"
 		(layer "B.Cu")
-		(at 77.25 29.5)
+		(at 77.25 30)
 		(descr "UCS2D331MHD")
 		(tags "Capacitor")
@@
 	(footprint "InverterCom:CAPPRD750W80D1800H3700"
 		(layer "B.Cu")
-		(at 90.5 77)
+		(at 91.75 77.5)
 		(descr "UCS2D331MHD")
 		(tags "Capacitor")
@@
 			(xy 152.983024 5.033842) (xy 126.991997 5.017863) (xy 127.000615 -8.999999) (xy 127.000614 -9) (xy 63 -9)
 			(xy 63 5) (xy 37 5) (xy 37 -8) (xy 36 -9) (xy 9 -9) (xy 0 0) (xy 0 85) (xy 2 87) (xy 277 87) (xy 292 87)
-			(xy 292 71) (xy 277 71) (xy 277 22) (xy 278 21) (xy 300.020228 20.984632) (xy 300.010476 7.010476)
+			(xy 292 79) (xy 287 74) (xy 277 74) (xy 277 22) (xy 278 21) (xy 296.99371 20.980456) (xy 296.981852 3.988134)
 			(xy 284 -9)
 		)
@@
 	(zone
 		(net "/DC_LINK_-")
+		(locked yes)
 		(layer "B.Cu")
 		(hatch edge 0.5)

Commit message: Update documentation
Parts:
- added H17: 9774030592R, InverterCom:9774030592R, F.Cu at (82.5, 45.0)
- added H18: 9774030592R, InverterCom:9774030592R, F.Cu at (22.0, 81.0)
- added H19: 9774030592R, InverterCom:9774030592R, F.Cu at (254.0, 79.0)
- added H20: 9774030592R, InverterCom:9774030592R, F.Cu at (165.0, 29.0)
Other:
- board text added: "HEATSPREADER COMPRESSION MODULE SCREW M5 -->"

Commit message: Update DC bus capacitor board
Other:
- board text added: "HW-C2-PCB-DCBUSCAP-A"
- board text added: "REV A | 2026-07 | THOMAS LIAO CORZINE SMART POWER LAB"
- board text removed: "REV B | 2026-07 | THOMAS LIAO CORZINE SMART POWER LAB"
Changed lines of the file:
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@@
 		)
 	)
-	(gr_text "REV B | 2026-07 | THOMAS LIAO\nCORZINE SMART POWER LAB"
+	(gr_text "REV A | 2026-07 | THOMAS LIAO\nCORZINE SMART POWER LAB"
 		(at 193.5 86 0)
 		(layer "F.SilkS")
 		(effects
+			(font
+				(size 1.5 1.5)
+				(thickness 0.375)
+				(bold yes)
+			)
+			(justify left bottom)
+		)
+	)
+	(gr_text "HW-C2-PCB-DCBUSCAP-A"
+		(at 213.425 9.25 0)
+		(layer "F.SilkS")
+		(effects

Commit message: Finalize Filter board
Other:
- board text added: "P/N: HW-C2-PCB-DCBUSCAP-A"
- board text removed: "HW-C2-PCB-DCBUSCAP-A"
Changed lines of the file:
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@@
 		)
 	)
-	(gr_text "HW-C2-PCB-DCBUSCAP-A"
-		(at 213.425 9.25 0)
+	(gr_text "P/N: HW-C2-PCB-DCBUSCAP-A"
+		(at 209.75 8.75 0)
 		(layer "F.SilkS")
 		(effects
