File: Hardware/Chassis2/Boards/GateDriver/SingleChannelDriver.kicad_sch (KiCad schematic)
At the start: 23 parts, among them IC1 ADUM4136BRWZ

Commit message: New gate driver
Parts:
- removed C1: 100nF, Capacitor_SMD:C_1210_3225Metric_Pad1.33x2.70mm_HandSolder, symbol Device:C
- removed FB1: FBMJ1608HS220NTR, InverterCom:BEADC1608X100N, symbol InverterCom:FBMJ1608HS220NTR
- removed IC1: ADUM4136BRWZ, InverterCom:SOIC127P1032X265-16N, symbol InverterCom:ADUM4136BRWZ
- removed R14, R9: 0, Resistor_SMD:R_1210_3225Metric_Pad1.30x2.65mm_HandSolder, symbol Device:R
- added C3: 10uF, Capacitor_SMD:C_1210_3225Metric_Pad1.33x2.70mm_HandSolder, symbol Device:C
- added D2: BAT54WS-7-F, InverterCom:SOD2513X120N, symbol InverterCom:BAT54WS-7-F
- added IC1: NCD57100DWR2G, SOIC127P1030X265-16N, symbol InverterCom:NCD57100DWR2G
- C2: value 10uF -> 100nF
- R3: renamed from R10; value 9.1 -> 2.7
- R4: renamed from R11; value 6.8 -> 2.7
- renumbered C13 to C12, C12 to C13, D2 to D3, R12 to R5, R13 to R6
Connections:
- net +15V_B: now also D1.1 (K), IC1.5 (VDD2)
- net +3.3V_A: now also C2.2, C3.1, IC1.15 (VDD1); no longer C2.1
- net -9V_B: now also IC1.1 (VEE2A), IC1.8 (VEE2)
- net EMITTER_B: now also D2.2 (A), IC1.3 (GND2)
- net FAULT: now also IC1.13 (~{FLT})
- net GATE_B: now also R3.1, R4.1, IC1.7 (CLAMP)
- net GND_A: now also C2.1, C3.2, IC1.16 (GND1), IC1.9 (GND1A); no longer C2.2
- net INPUT_+: now also IC1.10 (IN+)
- net INPUT_-: now also IC1.11 (IN-)
- net READY: now also IC1.12 (RDY)
- net RESET: now also IC1.14 (~{RST})
- net at R3.2: now also IC1.6 (OUTL); no longer D1.1 (K)
- net at D1.2 (A): now also C13.2, R5.2, R6.2, D2.1 (K), IC1.2 (DESAT); no longer R4.2
- new net: IC1.4 (OUTH), R4.2
Other:
- note removed: "DESAT DISABLE RESISTOR"
- moved on the sheet: D3, R3, R4, R5, R6
