File: Hardware/Chassis2/Boards/GateDriver/SingleChannelDriver.kicad_sch (KiCad schematic)
At the start: 21 parts, among them IC1 NCD57100DWR2G

Commit message: update hw revision 7
Parts:
- removed D3: FM2000GP-TP, InverterCom:DIOM5226X244N, symbol InverterCom:FM2000GP-TP
- added D19, D25: UF4007, DIOAD1413W86L463D238, symbol InverterCom:UF4007
- added TP11, TP5: TestPoint, TestPoint:TestPoint_Loop_D2.54mm_Drill1.5mm_Beaded, symbol Connector:TestPoint
- C13: value 100nF -> 220pF
Connections:
- net COLLECTOR_B: now also D25.1 (K)
- net GATE_B: now also TP11.1
- net at R6.1: now also D19.2 (A)
- net at C13.2, D1.2 (A), D2.1 (K)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: now also TP5.1
- new net: D19.1 (K), D25.2 (A)
Other:
- note added: "Good for ~2kV blocking, each is 1000v, 75nS fast recovery"
- note added: "With CM600DY-24T MODULES THIS SHOULD GIVE US ~4uS (Module switches in ~1.2uS)"
- note added: "might need to increase resistance here but perhaps not Observed some ringing on power conns <---"
- company: (none) -> Corzine Lab, University of California, Santa Cruz
- title: (none) -> Open Inverter Platform - Gate Driver Board

Commit message: Update Gate Driver Board, New Connector, New Desat Diode, 1oo2 SSO Pathway
Parts:
- removed D19, D25: UF4007, DIOAD1413W86L463D238, symbol InverterCom:UF4007
- added C83: 100nF, Capacitor_SMD:C_1210_3225Metric_Pad1.33x2.70mm_HandSolder, symbol Device:C
- added C84: 10uF, Capacitor_SMD:C_1210_3225Metric_Pad1.33x2.70mm_HandSolder, symbol Device:C
- added D3: STTH112A, DIOM5126X265N, symbol InverterCom:STTH112A
- D1, D2: footprint InverterCom:SOD2513X120N -> SOD2513X120N
- PS1: footprint InverterCom:MGJ2D121509MPCR7 -> MGJ2D121509MPCR7
Connections:
- net +12V_A: now also C83.2, C84.1
- net COLLECTOR_B: now also D3.1 (K)
- net GND_A: now also C83.1, C84.2
- net at R6.1: now also D3.2 (A)
Other:
- note added: "1200v <75nS fast recovery diode"
- note removed: "Good for ~2kV blocking, each is 1000v, 75nS fast recovery"

Commit message: fix schematic to aec-q100 gate driver p/n
Parts:
- IC1: value NCD57100DWR2G -> NCV57100DWR2G
Changed lines of the file:
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@@
 			)
 		)
-		(property "Value" "NCD57100DWR2G"
+		(property "Value" "NCV57100DWR2G"
 			(at 121.92 91.44 0)
 			(show_name no)

Commit message: fix(Hardware/Chassis2): gate driver AEC-Q100 MPN and precharge <2 A note
- Update GateDriver schematic/PDF to AEC-Q100 gate driver part number
- Update IOBoard schematic/PDF precharge note to stay below 2 A input fuse limit
Parts:
- IC1: Manufacturer_Part_Number NCD57100DWR2G -> NCV57100DWR2G; Mouser Part Number 863-NCD57100DWR2G -> 863-NCV57100DWR2G; Mouser Price/Stock https://www.mouser.co.uk/ProductDetail/onsemi/NCD57100DWR2G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 -> https://www.mouser.co.uk/ProductDetail/onsemi/NCV57100DWR2G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
Changed lines of the file:
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@@
 			)
 		)
-		(property "Mouser Part Number" "863-NCD57100DWR2G"
+		(property "Mouser Part Number" "863-NCV57100DWR2G"
 			(at 110.49 -380.62 0)
 			(hide yes)
@@
 			)
 		)
-		(property "Mouser Price/Stock" "https://www.mouser.co.uk/ProductDetail/onsemi/NCD57100DWR2G?qs=vvQtp7zwQdOcYrqkXGsoBw%3D%3D"
+		(property "Mouser Price/Stock" "https://www.mouser.co.uk/ProductDetail/onsemi/NCV57100DWR2G?qs=vvQtp7zwQdOcYrqkXGsoBw%3D%3D"
 			(at 110.49 -480.62 0)
 			(hide yes)
@@
 			)
 		)
-		(property "Manufacturer_Part_Number" "NCD57100DWR2G"
+		(property "Manufacturer_Part_Number" "NCV57100DWR2G"
 			(at 110.49 -680.62 0)
 			(hide yes)

Commit message: Finalize Gate driver model, connectors, ss, pn
Parts:
- D1, D2: footprint SOD2513X120N -> InverterCom:SOD2513X120N
- D3: footprint DIOM5126X265N -> InverterCom:DIOM5126X265N
- IC1: footprint SOIC127P1030X265-16N -> InverterCom:SOIC127P1030X265-16N
- PS1: footprint MGJ2D121509MPCR7 -> InverterCom:MGJ2D121509MPCR7
Changed lines of the file:
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@@
 		(title "Open Inverter Platform - Gate Driver Board")
 		(date "2026-07-07")
-		(rev "C")
+		(rev "A")
 		(company "Corzine Lab, University of California, Santa Cruz")
 		(comment 1 "Prepared by Thomas Liao")
+		(comment 2 "HW-C2-PCB-GD")
 	)
 	(text "might need to increase resistance here but perhaps not\nObserved some ringing on power conns\n\n<---"
@@
 			)
 		)
-		(property "Footprint" "MGJ2D121509MPCR7"
+		(property "Footprint" "InverterCom:MGJ2D121509MPCR7"
 			(at 186.36 26.67 0)
 			(hide yes)
@@
 			)
 		)
-		(property "Footprint" "SOD2513X120N"
+		(property "Footprint" "InverterCom:SOD2513X120N"
 			(at 82.88 125.73 0)
 			(hide yes)
@@
 			)
 		)
-		(property "Footprint" "SOD2513X120N"
+		(property "Footprint" "InverterCom:SOD2513X120N"
 			(at 82.88 140.97 0)
 			(hide yes)
@@
 			)
 		)
-		(property "Footprint" "SOIC127P1030X265-16N"
+		(property "Footprint" "InverterCom:SOIC127P1030X265-16N"
 			(at 110.49 19.38 0)
 			(hide yes)
@@
 			)
 		)
-		(property "Footprint" "DIOM5126X265N"
+		(property "Footprint" "InverterCom:DIOM5126X265N"
 			(at 222.25 32.08 0)
 			(hide yes)

Commit message: Labels tool, composite board views, InverterGen5 C2 branding, even render resolution
- Labels.pdf: HV warning labels, chassis ID, per-assembly labels (label cmd)
- Board sections add composite front/back views (PCB-viewer look, mirrored
  back) and layer plots now carry the drawing sheet with true plot scale
- Branding standardized to InverterGen5 C2 (cover, footer, labels)
- STEP previews render at even resolution regardless of part aspect
- Fab part titles from info.txt PartName; ALL-CAPS handling fixed
Other:
- title: Open Inverter Platform - Gate Driver Board -> InverterGen5 - Gate Driver Board
Changed lines of the file:
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@@
 	(paper "USLetter")
 	(title_block
-		(title "Open Inverter Platform - Gate Driver Board")
+		(title "InverterGen5 - Gate Driver Board")
 		(date "2026-07-07")
 		(rev "A")
