File: Hardware/Chassis2/Boards/GateDriver/GateDriver.kicad_pcb (KiCad board)
At the start: 6 copper layers, 75 x 60 mm, 69 parts, among them IC1 ADUM4136BRWZ, IC2 ADUM4136BRWZ, J1 Conn_02x08_Counter_Clockwise

Commit message: New gate driver
Parts:
- removed FB1, FB2: FBMJ1608HS220NTR, InverterCom:BEADC1608X100N
- removed LED5: LTST-C230GKT, InverterCom:LEDC3216X120N
- removed Q1: ~, InverterCom:62mm_power_module
- removed TP5, TP6: TestPoint, TestPoint:TestPoint_Loop_D2.54mm_Drill1.5mm_Beaded
- added C16: 10uF, Capacitor_SMD:C_1210_3225Metric_Pad1.33x2.70mm_HandSolder, F.Cu at (97.4, 79.9)
- added C27: 10uF, Capacitor_SMD:C_1210_3225Metric_Pad1.33x2.70mm_HandSolder, F.Cu at (7.43, 75.6)
- added C28: 10uF, Capacitor_SMD:C_1210_3225Metric_Pad1.33x2.70mm_HandSolder, F.Cu at (7.43, 79.9)
- added C29: 100nF, Capacitor_SMD:C_1210_3225Metric_Pad1.33x2.70mm_HandSolder, F.Cu at (7.43, 84.1)
- added C30: 100nF, Capacitor_SMD:C_1210_3225Metric_Pad1.33x2.70mm_HandSolder, F.Cu at (13.4, 71.4)
- added C31: 10uF, Capacitor_SMD:C_1210_3225Metric_Pad1.33x2.70mm_HandSolder, F.Cu at (13.4, 75.6)
- added C32: 10uF, Capacitor_SMD:C_1210_3225Metric_Pad1.33x2.70mm_HandSolder, F.Cu at (13.4, 79.9)
- added C33: 100nF, Capacitor_SMD:C_1210_3225Metric_Pad1.33x2.70mm_HandSolder, F.Cu at (13.4, 84.1)
- added C34: 10uF, Capacitor_SMD:C_1210_3225Metric_Pad1.33x2.70mm_HandSolder, F.Cu at (19.5, 71.4)
- added C35: 10uF, Capacitor_SMD:C_1210_3225Metric_Pad1.33x2.70mm_HandSolder, F.Cu at (19.5, 75.6)
- added C36: 10uF, Capacitor_SMD:C_1210_3225Metric_Pad1.33x2.70mm_HandSolder, F.Cu at (19.5, 79.9)
- added C37: 100nF, Capacitor_SMD:C_1210_3225Metric_Pad1.33x2.70mm_HandSolder, F.Cu at (19.5, 84.1)
- added C38: 100nF, Capacitor_SMD:C_1210_3225Metric_Pad1.33x2.70mm_HandSolder, F.Cu at (136.3, 69.4)
- added C39: 10uF, Capacitor_SMD:C_1210_3225Metric_Pad1.33x2.70mm_HandSolder, F.Cu at (136.3, 73.6)
- added C40: 10uF, Capacitor_SMD:C_1210_3225Metric_Pad1.33x2.70mm_HandSolder, F.Cu at (136.3, 77.9)
- added C41: 100nF, Capacitor_SMD:C_1210_3225Metric_Pad1.33x2.70mm_HandSolder, F.Cu at (136.3, 82.1)
- added C42: 100nF, Capacitor_SMD:C_1210_3225Metric_Pad1.33x2.70mm_HandSolder, F.Cu at (142.3, 69.4)
- added C43: 10uF, Capacitor_SMD:C_1210_3225Metric_Pad1.33x2.70mm_HandSolder, F.Cu at (142.3, 73.6)
- added C44: 10uF, Capacitor_SMD:C_1210_3225Metric_Pad1.33x2.70mm_HandSolder, F.Cu at (142.3, 77.9)
- added C45: 100nF, Capacitor_SMD:C_1210_3225Metric_Pad1.33x2.70mm_HandSolder, F.Cu at (142.3, 82.1)
- added C46: 10uF, Capacitor_SMD:C_1210_3225Metric_Pad1.33x2.70mm_HandSolder, F.Cu at (148.3, 69.4)
- added C47: 10uF, Capacitor_SMD:C_1210_3225Metric_Pad1.33x2.70mm_HandSolder, F.Cu at (148.3, 73.6)
- added C48: 10uF, Capacitor_SMD:C_1210_3225Metric_Pad1.33x2.70mm_HandSolder, F.Cu at (148.3, 77.9)
- added C49: 100nF, Capacitor_SMD:C_1210_3225Metric_Pad1.33x2.70mm_HandSolder, F.Cu at (148.3, 82.1)
- added C50: 100nF, Capacitor_SMD:C_1210_3225Metric_Pad1.33x2.70mm_HandSolder, F.Cu at (192.4, 71.4)
- added C51: 10uF, Capacitor_SMD:C_1210_3225Metric_Pad1.33x2.70mm_HandSolder, F.Cu at (192.4, 75.6)
- added C52: 10uF, Capacitor_SMD:C_1210_3225Metric_Pad1.33x2.70mm_HandSolder, F.Cu at (192.4, 79.9)
- added C53: 100nF, Capacitor_SMD:C_1210_3225Metric_Pad1.33x2.70mm_HandSolder, F.Cu at (192.4, 84.1)
- added C54: 100nF, Capacitor_SMD:C_1210_3225Metric_Pad1.33x2.70mm_HandSolder, F.Cu at (198.4, 71.4)
- added C55: 10uF, Capacitor_SMD:C_1210_3225Metric_Pad1.33x2.70mm_HandSolder, F.Cu at (198.4, 75.6)
- added C56: 10uF, Capacitor_SMD:C_1210_3225Metric_Pad1.33x2.70mm_HandSolder, F.Cu at (198.4, 79.9)
- added C57: 100nF, Capacitor_SMD:C_1210_3225Metric_Pad1.33x2.70mm_HandSolder, F.Cu at (198.4, 84.1)
- added C58: 10uF, Capacitor_SMD:C_1210_3225Metric_Pad1.33x2.70mm_HandSolder, F.Cu at (204.5, 71.4)
- added C59: 10uF, Capacitor_SMD:C_1210_3225Metric_Pad1.33x2.70mm_HandSolder, F.Cu at (204.5, 75.6)
- added C60: 10uF, Capacitor_SMD:C_1210_3225Metric_Pad1.33x2.70mm_HandSolder, F.Cu at (204.5, 79.9)
- added C61: 100nF, Capacitor_SMD:C_1210_3225Metric_Pad1.33x2.70mm_HandSolder, F.Cu at (204.5, 84.1)
- added C62: 100nF, Capacitor_SMD:C_1210_3225Metric_Pad1.33x2.70mm_HandSolder, F.Cu at (231.3, 73.4)
- added C63: 10uF, Capacitor_SMD:C_1210_3225Metric_Pad1.33x2.70mm_HandSolder, F.Cu at (231.3, 77.6)
- added C64: 10uF, Capacitor_SMD:C_1210_3225Metric_Pad1.33x2.70mm_HandSolder, F.Cu at (231.3, 81.9)
- added C65: 100nF, Capacitor_SMD:C_1210_3225Metric_Pad1.33x2.70mm_HandSolder, F.Cu at (231.3, 86.1)
- added C66: 100nF, Capacitor_SMD:C_1210_3225Metric_Pad1.33x2.70mm_HandSolder, F.Cu at (237.3, 73.4)
- added C67: 10uF, Capacitor_SMD:C_1210_3225Metric_Pad1.33x2.70mm_HandSolder, F.Cu at (237.3, 77.6)
- added C68: 10uF, Capacitor_SMD:C_1210_3225Metric_Pad1.33x2.70mm_HandSolder, F.Cu at (237.3, 81.9)
- added C69: 100nF, Capacitor_SMD:C_1210_3225Metric_Pad1.33x2.70mm_HandSolder, F.Cu at (237.3, 86.1)
- added C70: 10uF, Capacitor_SMD:C_1210_3225Metric_Pad1.33x2.70mm_HandSolder, F.Cu at (243.3, 73.4)
- added C71: 10uF, Capacitor_SMD:C_1210_3225Metric_Pad1.33x2.70mm_HandSolder, F.Cu at (243.3, 77.6)
- added C72: 10uF, Capacitor_SMD:C_1210_3225Metric_Pad1.33x2.70mm_HandSolder, F.Cu at (243.3, 81.9)
- added C73: 100nF, Capacitor_SMD:C_1210_3225Metric_Pad1.33x2.70mm_HandSolder, F.Cu at (243.3, 86.1)
- added D10: BAT54WS-7-F, InverterCom:SOD2513X120N, F.Cu at (162.9, 51.1)
- added D11: BAT54WS-7-F, InverterCom:SOD2513X120N, F.Cu at (162.9, 54.4)
- added D12: FM2000GP-TP, InverterCom:DIOM5226X244N, F.Cu at (155.2, 81.2)
- added D13: BAT54WS-7-F, InverterCom:SOD2513X120N, F.Cu at (219.0, 53.0)
- added D14: BAT54WS-7-F, InverterCom:SOD2513X120N, F.Cu at (219.0, 56.4)
- added D15: FM2000GP-TP, InverterCom:DIOM5226X244N, F.Cu at (211.3, 83.2)
- added D16: BAT54WS-7-F, InverterCom:SOD2513X120N, F.Cu at (257.9, 55.0)
- added D17: BAT54WS-7-F, InverterCom:SOD2513X120N, F.Cu at (257.9, 58.4)
- added D18: FM2000GP-TP, InverterCom:DIOM5226X244N, F.Cu at (250.2, 85.2)
- added D5: BAT54WS-7-F, InverterCom:SOD2513X120N, F.Cu at (124.0, 56.4)
- added D6: FM2000GP-TP, InverterCom:DIOM5226X244N, F.Cu at (116.3, 83.2)
- added D7: BAT54WS-7-F, InverterCom:SOD2513X120N, F.Cu at (34.0, 53.0)
- added D8: BAT54WS-7-F, InverterCom:SOD2513X120N, F.Cu at (34.0, 56.4)
- added D9: FM2000GP-TP, InverterCom:DIOM5226X244N, F.Cu at (26.3, 83.2)
- added H2: MountingHole, MountingHole:MountingHole_5.3mm_M5_ISO7380_Pad, F.Cu at (5.00, 40.0)
- added H6: MountingHole, MountingHole:MountingHole_5.3mm_M5_ISO7380_Pad, F.Cu at (180.0, 40.0)
- added H7: MountingHole, MountingHole:MountingHole_5.3mm_M5_ISO7380_Pad, F.Cu at (255.0, 5.00)
- added H8: MountingHole, MountingHole:MountingHole_5.3mm_M5_ISO7380_Pad, F.Cu at (255.0, 40.0)
- added IC3: NCD57100DWR2G, InverterCom:SOIC127P1030X265-16N, F.Cu at (25.0, 25.0)
- added IC4: NCD57100DWR2G, InverterCom:SOIC127P1030X265-16N, F.Cu at (147.5, 25.0)
- added IC5: NCD57100DWR2G, InverterCom:SOIC127P1030X265-16N, F.Cu at (205.0, 25.0)
- added IC6: NCD57100DWR2G, InverterCom:SOIC127P1030X265-16N, F.Cu at (236.9, 25.0)
- added J2: TBP01R2W-508-06BE, InverterCom:SHDR6W100P0X508_1X6_4064X850X1240P, F.Cu at (53.0, 5.45)
- added J3: TBP01R2W-508-06BE, InverterCom:SHDR6W100P0X508_1X6_4064X850X1240P, F.Cu at (143.0, 6.00)
- added J4: TBP01R2W-508-06BE, InverterCom:SHDR6W100P0X508_1X6_4064X850X1240P, F.Cu at (233.0, 5.45)
- added LED1: LTST-C230GKT, InverterCom:LEDC3216X120N, F.Cu at (-22.5, 57.5)
- added PS3: MGJ2D121509MPC-R7, InverterCom:MGJ2D121509MPCR7, B.Cu at (25.0, 22.1)
- added PS4: MGJ2D121509MPC-R7, InverterCom:MGJ2D121509MPCR7, B.Cu at (148.0, 22.1)
- added PS5: MGJ2D121509MPC-R7, InverterCom:MGJ2D121509MPCR7, B.Cu at (205.0, 22.1)
- added PS6: MGJ2D121509MPC-R7, InverterCom:MGJ2D121509MPCR7, B.Cu at (237.0, 22.1)
- added R15: 2.7, Resistor_SMD:R_1210_3225Metric_Pad1.30x2.65mm_HandSolder, F.Cu at (157.4, 51.5)
- added R16: 2.7, Resistor_SMD:R_1210_3225Metric_Pad1.30x2.65mm_HandSolder, F.Cu at (157.4, 55.7)
- added R18: 1k, Resistor_SMD:R_1210_3225Metric_Pad1.30x2.65mm_HandSolder, F.Cu at (157.4, 64.1)
- added R25: 1k, Resistor_SMD:R_1210_3225Metric_Pad1.30x2.65mm_HandSolder, F.Cu at (252.4, 63.9)
- added R26: 1k, Resistor_SMD:R_1210_3225Metric_Pad1.30x2.65mm_HandSolder, F.Cu at (252.4, 68.1)
- added R7: 2.7, Resistor_SMD:R_1210_3225Metric_Pad1.30x2.65mm_HandSolder, F.Cu at (118.5, 53.5)
- C1: value 100nF -> UCM1H101MCL1GS; footprint Capacitor_SMD:C_1210_3225Metric_Pad1.33x2.70mm_HandSolder -> InverterCom:CAPAE660X800N
- C11, C24, C25, R13: moved to F.Cu
- C12: value 100nF -> 10uF; moved to F.Cu
- C13, C26: value 10uF -> 100nF; moved to F.Cu
- C17, C2, C21: value 10uF -> 100nF
- C19, C22: value 100nF -> 10uF
- C3: value UCM1H101MCL1GS -> 10uF; footprint InverterCom:CAPAE660X800N -> Capacitor_SMD:C_1210_3225Metric_Pad1.33x2.70mm_HandSolder
- D2, D4: value FM2000GP-TP -> BAT54WS-7-F; footprint InverterCom:DIOM5226X244N -> InverterCom:SOD2513X120N
- D3: value BAT54WS-7-F -> FM2000GP-TP; footprint InverterCom:SOD2513X120N -> InverterCom:DIOM5226X244N
- H1, H3: footprint MountingHole:MountingHole_3.2mm_M3 -> MountingHole:MountingHole_5.3mm_M5_ISO7380_Pad
- H4, H5: value MountingHole_Pad -> MountingHole; footprint MountingHole:MountingHole_2.2mm_M2_Pad -> MountingHole:MountingHole_5.3mm_M5_ISO7380_Pad
- IC1, IC2: value ADUM4136BRWZ -> NCD57100DWR2G; footprint InverterCom:SOIC127P1032X265-16N -> InverterCom:SOIC127P1030X265-16N
- R10: value 9.1 -> 1k
- R11: value 6.8 -> 2.7; moved to F.Cu
- R12: value 1k -> 2.7
- R14: value 0 -> 1k
- R17, R5, R6: value 4.7k -> 1k; moved to F.Cu
- R19: value 0 -> 2.7; moved to F.Cu
- R2: value 4.7k -> 220
- R20: value 9.1 -> 2.7
- R21: value 6.8 -> 1k; moved to F.Cu
- R23: value 1k -> 2.7; moved to F.Cu
- R24: value 0 -> 2.7
- R3: value 4.7k -> 2.7
- R4: value 4.7k -> 2.7; moved to F.Cu
- R8: value 220 -> 2.7; moved to F.Cu
- R9: value 0 -> 1k; moved to F.Cu
- moved R23 249.5 mm to (252.4, 55.5)
- moved R24 238.4 mm to (252.4, 59.7), turned to 0 degrees
- moved R22 207.6 mm to (213.5, 66.1), turned to 0 degrees
- moved R19 204.3 mm to (213.5, 53.5)
- moved R20 195.8 mm to (213.5, 57.7), turned to 0 degrees
- moved R21 194.2 mm to (213.5, 61.9), turned to 0 degrees
- moved H5 177.6 mm to (180.0, 5.00)
- moved R17 152.2 mm to (157.4, 59.9)
- moved D4 124.0 mm to (124.0, 53.0), turned to 0 degrees
- moved C25 114.2 mm to (109.5, 84.1), turned to 0 degrees
- moved C17 98.7 mm to (97.4, 84.1), turned to 0 degrees
- moved C23 98.5 mm to (109.5, 75.6), turned to 0 degrees
- moved C24 98.1 mm to (109.5, 79.9), turned to 0 degrees
- moved LED2 95.9 mm to (-22.5, 61.2), turned to 0 degrees
- moved C22 95.0 mm to (109.5, 71.4)
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Connections:
- C1 pad 1: /GND_A -> /+12V_A
- C1 pad 2: /+3.3V_A -> /GND_A
- C12 pad 1: /SingleChannelDriver1/GND_B -> /SingleChannelDriver1/+15V_B
- C12 pad 2: Net-(IC1-DESAT) -> /SingleChannelDriver1/-9V_B
- C13 pad 1: /SingleChannelDriver1/+15V_B -> /SingleChannelDriver1/GND_B
- C13 pad 2: /SingleChannelDriver1/-9V_B -> Net-(D1-A)
- C17 pad 1: /SingleChannelDriver/GND_B -> /SingleChannelDriver2/GND_B
- C17 pad 2: /SingleChannelDriver/+15V_B -> /SingleChannelDriver2/+15V_B
- C18 pad 1: /SingleChannelDriver/GND_B -> /SingleChannelDriver2/-9V_B
- C18 pad 2: /SingleChannelDriver/+15V_B -> /SingleChannelDriver2/GND_B
- C19 pad 1: /SingleChannelDriver/-9V_B -> /SingleChannelDriver2/+15V_B
- C19 pad 2: /SingleChannelDriver/GND_B -> /SingleChannelDriver2/-9V_B
- C2 pad 1: /+3.3V_A -> /GND_A
- C2 pad 2: /GND_A -> /+3.3V_A
- C20 pad 1: /SingleChannelDriver/+15V_B -> /SingleChannelDriver2/+15V_B
- C20 pad 2: /SingleChannelDriver/-9V_B -> /SingleChannelDriver2/-9V_B
- C21 pad 1: /SingleChannelDriver/+15V_B -> /SingleChannelDriver2/-9V_B
- C21 pad 2: /SingleChannelDriver/-9V_B -> /SingleChannelDriver2/+15V_B
- C22 pad 1: /SingleChannelDriver/-9V_B -> /SingleChannelDriver2/+15V_B
- C22 pad 2: /SingleChannelDriver/+15V_B -> /SingleChannelDriver2/-9V_B
- C23 pad 1: /SingleChannelDriver/+15V_B -> /SingleChannelDriver2/+15V_B
- C23 pad 2: /SingleChannelDriver/-9V_B -> /SingleChannelDriver2/-9V_B
- C24 pad 1: /SingleChannelDriver/+15V_B -> /SingleChannelDriver2/+15V_B
- C24 pad 2: /SingleChannelDriver/-9V_B -> /SingleChannelDriver2/-9V_B
- C25 pad 1: /SingleChannelDriver/GND_B -> /SingleChannelDriver2/GND_B
- C25 pad 2: Net-(IC2-DESAT) -> Net-(D4-A)
- C26 pad 1: /SingleChannelDriver/+15V_B -> /GND_A
- C26 pad 2: /SingleChannelDriver/-9V_B -> /+3.3V_A
- C3 pad 1: /+12V_A -> /+3.3V_A
- D1 pad 1: Net-(D1-K) -> /SingleChannelDriver1/+15V_B
- D2 pad 1: /PH_L_C -> Net-(D1-A)
- D2 pad 2: Net-(D2-A) -> /SingleChannelDriver1/GND_B
- D3 pad 1: Net-(D3-K) -> /PH_U_L_C
- D4 pad 1: /PH_H_C -> /SingleChannelDriver2/+15V_B
- H4 pad 1: /PH_L_C -> (no net)
- H5 pad 1: /PH_H_C -> (no net)
- IC1 pad 1: /PH_L -> /SingleChannelDriver1/-9V_B
- IC1 pad 10: /SingleChannelDriver1/-9V_B -> /PH_U_L
- IC1 pad 11: Net-(D1-K) -> /PH_U_H
- IC1 pad 12: /SingleChannelDriver1/+15V_B -> /READY
- IC1 pad 13: /SingleChannelDriver1/+15V_B -> /FAULT
- IC1 pad 14: Net-(IC1-DESAT) -> /RESET
- IC1 pad 15: /SingleChannelDriver1/-9V_B -> /+3.3V_A
- IC1 pad 16: /SingleChannelDriver1/GND_B -> /GND_A
- IC1 pad 2: /PH_H -> Net-(D1-A)
- IC1 pad 3: /+3.3V_A -> /SingleChannelDriver1/GND_B
- IC1 pad 4: /GND_A -> Net-(IC1-OUTH)
- IC1 pad 5: /RESET -> /SingleChannelDriver1/+15V_B
- IC1 pad 6: /FAULT -> Net-(IC1-OUTL)
- IC1 pad 7: /READY -> /PH_U_L_G
- IC1 pad 8: /GND_A -> /SingleChannelDriver1/-9V_B
- IC1 pad 9: /SingleChannelDriver1/-9V_B -> /GND_A
- IC2 pad 1: /PH_H -> /SingleChannelDriver2/-9V_B
- IC2 pad 10: /SingleChannelDriver/-9V_B -> /PH_V_H
- IC2 pad 11: Net-(D3-K) -> /PH_V_L
- IC2 pad 12: /SingleChannelDriver/+15V_B -> /READY
- IC2 pad 13: /SingleChannelDriver/+15V_B -> /FAULT
- IC2 pad 14: Net-(IC2-DESAT) -> /RESET
- IC2 pad 15: /SingleChannelDriver/-9V_B -> /+3.3V_A
- IC2 pad 16: /SingleChannelDriver/GND_B -> /GND_A
- IC2 pad 2: /PH_L -> Net-(D4-A)
- IC2 pad 3: /+3.3V_A -> /SingleChannelDriver2/GND_B
- IC2 pad 4: /GND_A -> Net-(IC2-OUTH)
- IC2 pad 5: /RESET -> /SingleChannelDriver2/+15V_B
- IC2 pad 6: /FAULT -> Net-(IC2-OUTL)
- IC2 pad 7: /READY -> /PH_V_H_G
- IC2 pad 8: /GND_A -> /SingleChannelDriver2/-9V_B
- IC2 pad 9: /SingleChannelDriver/-9V_B -> /GND_A
- J1 pad 10: /PH_L -> /GND_A
- J1 pad 11: /GND_A -> /PH_W_L
- J1 pad 12: /PH_H -> /PH_W_H
- J1 pad 3: /GND_A -> /READY
- J1 pad 4: /READY -> /RESET
- J1 pad 5: /GND_A -> /PH_U_L
- J1 pad 6: /RESET -> /PH_U_H
- J1 pad 7: /GND_A -> /PH_V_L
- J1 pad 8: /GND_A -> /PH_V_H
- PS2 pad 3: /SingleChannelDriver/-9V_B -> /SingleChannelDriver2/-9V_B
- PS2 pad 4: /SingleChannelDriver/-9V_B -> /SingleChannelDriver2/-9V_B
- PS2 pad 5: /SingleChannelDriver/+15V_B -> /SingleChannelDriver2/+15V_B
- PS2 pad 6: /SingleChannelDriver/GND_B -> /SingleChannelDriver2/GND_B
- R1 pad 1: /READY -> Net-(LED1-A)
- R1 pad 2: /+3.3V_A -> /+12V_A
- R10 pad 1: Net-(FB1-Pad2) -> Net-(D6-A)
- R10 pad 2: Net-(D1-K) -> Net-(D4-A)
- R11 pad 1: Net-(FB1-Pad2) -> /PH_U_H_G
- R11 pad 2: Net-(D1-A) -> Net-(IC3-OUTL)
- R12 pad 1: /SingleChannelDriver1/+15V_B -> /PH_U_H_G
- R12 pad 2: Net-(IC1-DESAT) -> Net-(IC3-OUTH)
- R13 pad 1: Net-(D2-A) -> /SingleChannelDriver/+15V_B
- R13 pad 2: Net-(IC1-DESAT) -> Net-(D7-A)
- R14 pad 1: /PH_L_G -> Net-(D9-A)
- R14 pad 2: Net-(FB1-Pad2) -> Net-(D7-A)
- R17 pad 1: Net-(LED5-A) -> /SingleChannelDriver3/+15V_B
- R17 pad 2: /+12V_A -> Net-(D10-A)
- R19 pad 1: Net-(IC2-DESAT) -> /PH_W_H_G
- R19 pad 2: /SingleChannelDriver/GND_B -> Net-(IC5-OUTL)
- R2 pad 1: /RESET -> Net-(LED2-A)
- R20 pad 1: Net-(FB2-Pad2) -> /PH_W_H_G
- R20 pad 2: Net-(D3-K) -> Net-(IC5-OUTH)
- R21 pad 1: Net-(FB2-Pad2) -> /SingleChannelDriver4/+15V_B
- R21 pad 2: Net-(D3-A) -> Net-(D13-A)
- R22 pad 1: /SingleChannelDriver/+15V_B -> Net-(D15-A)
- R22 pad 2: Net-(IC2-DESAT) -> Net-(D13-A)
- R23 pad 1: Net-(D4-A) -> /PH_W_L_G
- R23 pad 2: Net-(IC2-DESAT) -> Net-(IC6-OUTL)
- R24 pad 1: /PH_H_G -> /PH_W_L_G
- R24 pad 2: Net-(FB2-Pad2) -> Net-(IC6-OUTH)
- R3 pad 1: /FAULT -> /PH_U_L_G
- R3 pad 2: /+3.3V_A -> Net-(IC1-OUTL)
- R4 pad 1: /GND_A -> /PH_U_L_G
- R4 pad 2: /FAULT -> Net-(IC1-OUTH)
- R5 pad 1: /GND_A -> /SingleChannelDriver1/+15V_B
- R5 pad 2: /READY -> Net-(D1-A)
- R6 pad 1: /GND_A -> Net-(D3-A)
- R6 pad 2: /RESET -> Net-(D1-A)
- R8 pad 1: Net-(LED2-A) -> /PH_V_H_G
- R8 pad 2: /+3.3V_A -> Net-(IC2-OUTH)
- R9 pad 1: Net-(IC1-DESAT) -> /SingleChannelDriver2/+15V_B
- R9 pad 2: /SingleChannelDriver1/GND_B -> Net-(D4-A)
- TP1 pad 1: /READY -> /FAULT
- TP2 pad 1: /RESET -> /READY
- TP3 pad 1: /FAULT -> /RESET
Routing:
- net /RESET: track 72.5 -> 0.00 mm, vias 5 -> 0
- net /FAULT: track 62.0 -> 0.00 mm, vias 4 -> 0
- net /READY: track 57.1 -> 0.00 mm, vias 6 -> 0
- net /PH_H: track 46.3 -> 0.00 mm, vias 5 -> 0
- net /PH_L: track 45.1 -> 0.00 mm, vias 4 -> 0
- net Net-(IC1-DESAT): track 33.5 -> 0.00 mm, vias 4 -> 0
- net Net-(IC2-DESAT): track 32.1 -> 0.00 mm, vias 2 -> 0
- net /SingleChannelDriver1/-9V_B: track 28.8 -> 0.00 mm, vias 8 -> 0
- net /SingleChannelDriver1/+15V_B: track 28.3 -> 0.00 mm, vias 9 -> 0
- net /SingleChannelDriver1/GND_B: track 27.3 -> 0.00 mm, vias 4 -> 0
- net /+3.3V_A: track 25.9 -> 0.00 mm, vias 6 -> 0
- net /SingleChannelDriver/+15V_B: track 23.3 -> 0.00 mm, vias 8 -> 0
- net /SingleChannelDriver/-9V_B: track 22.8 -> 0.00 mm, vias 8 -> 0
- net Net-(D1-K): track 18.1 -> 0.00 mm
- net Net-(D3-K): track 18.1 -> 0.00 mm
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- removed copper zone on In2.Cu, net /+12V_A
- removed copper zone on In3.Cu, net /+3.3V_A
- removed copper zone on B.Cu, net /GND_A
- removed copper zone on F.Cu, net /GND_A
- removed copper zone on In1.Cu, net /GND_A
- removed copper zone on In4.Cu, net /GND_A
- removed copper zone on In2.Cu, net /SingleChannelDriver/+15V_B
- removed copper zone on In3.Cu, net /SingleChannelDriver/-9V_B
- removed copper zone on B.Cu, net /SingleChannelDriver/GND_B
- removed copper zone on F.Cu, net /SingleChannelDriver/GND_B
- removed copper zone on In1.Cu, net /SingleChannelDriver/GND_B
- removed copper zone on In4.Cu, net /SingleChannelDriver/GND_B
- removed copper zone on In2.Cu, net /SingleChannelDriver1/+15V_B
- removed copper zone on In3.Cu, net /SingleChannelDriver1/-9V_B
- removed copper zone on B.Cu, net /SingleChannelDriver1/GND_B
- removed copper zone on F.Cu, net /SingleChannelDriver1/GND_B
- removed copper zone on In1.Cu, net /SingleChannelDriver1/GND_B
- removed copper zone on In4.Cu, net /SingleChannelDriver1/GND_B
Other:
- board size 75 x 60 mm -> 260 x 45 mm
- board text removed: "1->"
- board text removed: "62MM POWER MODULE DRIVER REV 1 1200VMAX, 800V WORKING"
- board text removed: "<- HIGH SIDE COLLECTOR DESAT PROTECTION"
- board text removed: "DANGER HIGH VOLTAGE"
- board text removed: "DESIGNED BY THOMAS LIAO"
- board text removed: "ISOLATION BARRIER DO NOT CROSS"
- board text removed: "LOW SIDE COLLECTOR -> DESAT PROTECTION"

Commit message: Finish gate driver board
Parts:
- added C74: UCM1H101MCL1GS, InverterCom:CAPAE660X800N, F.Cu at (105.5, 40.5)
- added C75: UCM1H101MCL1GS, InverterCom:CAPAE660X800N, F.Cu at (17.0, 41.0)
- added C77: UCM1H101MCL1GS, InverterCom:CAPAE660X800N, F.Cu at (95.5, 40.5)
- added C78: UCM1H101MCL1GS, InverterCom:CAPAE660X800N, F.Cu at (190.5, 41.0)
- added C80: UCM1H101MCL1GS, InverterCom:CAPAE660X800N, F.Cu at (74.5, 41.0)
- added C81: UCM1H101MCL1GS, InverterCom:CAPAE660X800N, F.Cu at (214.0, 41.0)
- added C82: UCM1H101MCL1GS, InverterCom:CAPAE660X800N, F.Cu at (224.3, 36.0)
- added U5: BTS462TATMA1, Package_TO_SOT_SMD:TO-252-4, F.Cu at (167.5, 37.3)
- C11, C13, C15, C19, C21, C23, C25, C27, C28, C3, C31, C33, C35, C37, C39, C41, C43, C47, C49, C5, C50, C55, C56, C59, C61, C63, C64, C67, C68, C7, C71, C73, R1, R2: moved to B.Cu
- moved R1 272.5 mm to (239.0, 41.0), turned to 180 degrees
- moved LED1 265.5 mm to (242.5, 41.0), turned to 180 degrees
- moved R2 265.1 mm to (231.2, 42.2)
- moved LED2 254.3 mm to (231.0, 41.0), turned to 180 degrees
- moved C1 96.7 mm to (64.5, 41.0)
- moved TP3 90.5 mm to (47.0, 37.0)
- moved TP2 84.1 mm to (41.0, 34.0)
- moved D18 77.5 mm to (243.0, 8.00), turned to -90 degrees
- moved TP1 76.9 mm to (36.0, 37.0)
- moved D15 76.7 mm to (196.0, 8.00), turned to -90 degrees
- moved D6 75.9 mm to (106.0, 8.00), turned to -90 degrees
- moved D9 75.9 mm to (16.0, 8.00), turned to -90 degrees
- moved C9 73.9 mm to (75.0, 10.0), turned to 180 degrees
- moved C45 73.7 mm to (165.0, 12.0), turned to 180 degrees
- moved D12 73.2 mm to (153.0, 8.00), turned to -90 degrees
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Connections:
- J1 pad 15: /GND_A -> /+12V_ENABLE
- J1 pad 16: /+12V_A -> /+12V_IN
- J2 pad 1: /SingleChannelDriver1/GND_B -> /PH_U_L_C
- J2 pad 2: /PH_U_L_G -> /SingleChannelDriver1/GND_B
- J2 pad 3: /PH_U_L_C -> /PH_U_L_G
- J2 pad 4: /SingleChannelDriver/GND_B -> /PH_U_H_G
- J2 pad 5: /PH_U_H_G -> /SingleChannelDriver/GND_B
- J3 pad 1: /SingleChannelDriver3/GND_B -> /PH_V_L_C
- J3 pad 2: /PH_V_L_G -> /SingleChannelDriver3/GND_B
- J3 pad 3: /PH_V_L_C -> /PH_V_L_G
- J3 pad 4: /SingleChannelDriver2/GND_B -> /PH_V_H_G
- J3 pad 5: /PH_V_H_G -> /SingleChannelDriver2/GND_B
- J4 pad 1: /SingleChannelDriver5/GND_B -> /PH_W_L_C
- J4 pad 2: /PH_W_L_G -> /SingleChannelDriver5/GND_B
- J4 pad 3: /PH_W_L_C -> /PH_W_L_G
- J4 pad 4: /SingleChannelDriver4/GND_B -> /PH_W_H_G
- J4 pad 5: /PH_W_H_G -> /SingleChannelDriver4/GND_B
Routing:
- net /READY: track 0.00 -> 286.8 mm, vias 0 -> 9
- net /FAULT: track 0.00 -> 273.3 mm, vias 0 -> 7
- net /RESET: track 0.00 -> 267.4 mm, vias 0 -> 8
- net /PH_U_L: track 0.00 -> 131.9 mm, vias 0 -> 3
- net /PH_U_H: track 0.00 -> 129.6 mm, vias 0 -> 3
- net /PH_W_L: track 0.00 -> 120.4 mm, vias 0 -> 3
- net /PH_W_H: track 0.00 -> 116.1 mm, vias 0 -> 3
- net /PH_V_L: track 0.00 -> 47.0 mm, vias 0 -> 3
- net /PH_V_H: track 0.00 -> 46.3 mm, vias 0 -> 3
- net /PH_W_H_G: track 0.00 -> 35.8 mm, vias 0 -> 2
- net /PH_V_H_G: track 0.00 -> 34.7 mm, vias 0 -> 2
- net /PH_U_H_G: track 0.00 -> 32.9 mm, vias 0 -> 2
- net /PH_U_L_G: track 0.00 -> 30.2 mm, vias 0 -> 2
- net /PH_W_L_G: track 0.00 -> 29.8 mm, vias 0 -> 2
- net /PH_V_L_G: track 0.00 -> 29.6 mm, vias 0 -> 2
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- added copper zone on In2.Cu, net /+12V_A
- added copper zone on In3.Cu, net /+3.3V_A
- added copper zone on B.Cu, net /GND_A
- added copper zone on F.Cu, net /GND_A
- added copper zone on In1.Cu, net /GND_A
- added copper zone on In4.Cu, net /GND_A
- added copper zone on In2.Cu, net /SingleChannelDriver/+15V_B
- added copper zone on In3.Cu, net /SingleChannelDriver/-9V_B
- added copper zone on B.Cu, net /SingleChannelDriver/GND_B
- added copper zone on F.Cu, net /SingleChannelDriver/GND_B
- added copper zone on In1.Cu, net /SingleChannelDriver/GND_B
- added copper zone on In4.Cu, net /SingleChannelDriver/GND_B
- added copper zone on In2.Cu, net /SingleChannelDriver1/+15V_B
- added copper zone on In3.Cu, net /SingleChannelDriver1/-9V_B
- added copper zone on B.Cu, net /SingleChannelDriver1/GND_B
- added copper zone on F.Cu, net /SingleChannelDriver1/GND_B
- added copper zone on In1.Cu, net /SingleChannelDriver1/GND_B
- added copper zone on In4.Cu, net /SingleChannelDriver1/GND_B
- added copper zone on In2.Cu, net /SingleChannelDriver2/+15V_B
- added copper zone on In3.Cu, net /SingleChannelDriver2/-9V_B
- added copper zone on B.Cu, net /SingleChannelDriver2/GND_B
- added copper zone on F.Cu, net /SingleChannelDriver2/GND_B
- added copper zone on In1.Cu, net /SingleChannelDriver2/GND_B
- added copper zone on In4.Cu, net /SingleChannelDriver2/GND_B
- added copper zone on In2.Cu, net /SingleChannelDriver3/+15V_B
- added copper zone on In3.Cu, net /SingleChannelDriver3/-9V_B
- added copper zone on B.Cu, net /SingleChannelDriver3/GND_B
- added copper zone on F.Cu, net /SingleChannelDriver3/GND_B
- added copper zone on In1.Cu, net /SingleChannelDriver3/GND_B
- added copper zone on In4.Cu, net /SingleChannelDriver3/GND_B
- added copper zone on In2.Cu, net /SingleChannelDriver4/+15V_B
- added copper zone on In3.Cu, net /SingleChannelDriver4/-9V_B
- added copper zone on B.Cu, net /SingleChannelDriver4/GND_B
- added copper zone on F.Cu, net /SingleChannelDriver4/GND_B
- added copper zone on In1.Cu, net /SingleChannelDriver4/GND_B
- added copper zone on In4.Cu, net /SingleChannelDriver4/GND_B
- added copper zone on In2.Cu, net /SingleChannelDriver5/+15V_B
- added copper zone on In3.Cu, net /SingleChannelDriver5/-9V_B
- added copper zone on B.Cu, net /SingleChannelDriver5/GND_B
- added copper zone on F.Cu, net /SingleChannelDriver5/GND_B
- added copper zone on In1.Cu, net /SingleChannelDriver5/GND_B
- added copper zone on In4.Cu, net /SingleChannelDriver5/GND_B
Other:
- board text added: "DANGER: HIGH VOLTAGE!"
- board text added: "DANGER: HIGH VOLTAGE! DO NOT TOUCH"
- board text added: "HIGH SIDE (COLLECTOR, EMITTER, GATE) | (GATE, EMITTER, COLLECTOR) LOW SIDE"
- board text added: "ISOLATED GATE DRIVER"
- board text added: "ISOLATION BARRIER DO NOT CROSS"
- board text added: "PIN 1 ->"
- board text added: "SERIAL NUMBER"
