File: Hardware/Chassis2/Boards/GateDriver/GateDriver.kicad_pcb (KiCad board)
At the start: 6 copper layers, 260 x 45 mm, 155 parts, among them IC1 NCD57100DWR2G, IC2 NCD57100DWR2G, IC3 NCD57100DWR2G, IC4 NCD57100DWR2G, IC5 NCD57100DWR2G, IC6 NCD57100DWR2G, J1 Conn_02x08_Counter_Clockwise, J2 TBP01R2W-508-06BE, J3 TBP01R2W-508-06BE, J4 TBP01R2W-508-06BE, U5 BTS462TATMA1

Commit message: Update Gate Driver Board, New Connector, New Desat Diode, 1oo2 SSO Pathway
Parts:
- removed J4: TBP01R2W-508-06BE, InverterCom:SHDR6W100P0X508_1X6_4064X850X1240P
- added C76: 100nF, Capacitor_SMD:C_1210_3225Metric_Pad1.33x2.70mm_HandSolder, B.Cu at (138.5, 43.0)
- added C79: 100nF, Capacitor_SMD:C_1210_3225Metric_Pad1.33x2.70mm_HandSolder, B.Cu at (158.2, 43.0)
- added C83: 100nF, Capacitor_SMD:C_1210_3225Metric_Pad1.33x2.70mm_HandSolder, F.Cu at (70.2, 33.8)
- added C84: 10uF, Capacitor_SMD:C_1210_3225Metric_Pad1.33x2.70mm_HandSolder, B.Cu at (73.2, 33.8)
- added C85: 100nF, Capacitor_SMD:C_1210_3225Metric_Pad1.33x2.70mm_HandSolder, F.Cu at (106.8, 33.0)
- added C86: 10uF, Capacitor_SMD:C_1210_3225Metric_Pad1.33x2.70mm_HandSolder, B.Cu at (103.5, 33.0)
- added C87: 100nF, Capacitor_SMD:C_1210_3225Metric_Pad1.33x2.70mm_HandSolder, F.Cu at (23.9, 38.2)
- added C88: 10uF, Capacitor_SMD:C_1210_3225Metric_Pad1.33x2.70mm_HandSolder, F.Cu at (23.9, 42.5)
- added C89: 100nF, Capacitor_SMD:C_1210_3225Metric_Pad1.33x2.70mm_HandSolder, F.Cu at (156.0, 33.2)
- added C90: 10uF, Capacitor_SMD:C_1210_3225Metric_Pad1.33x2.70mm_HandSolder, B.Cu at (159.2, 33.0)
- added C91: 100nF, Capacitor_SMD:C_1210_3225Metric_Pad1.33x2.70mm_HandSolder, F.Cu at (194.2, 33.2)
- added C92: 10uF, Capacitor_SMD:C_1210_3225Metric_Pad1.33x2.70mm_HandSolder, B.Cu at (191.2, 33.2)
- added C93: 100nF, Capacitor_SMD:C_1210_3225Metric_Pad1.33x2.70mm_HandSolder, F.Cu at (238.5, 37.2)
- added C94: 10uF, Capacitor_SMD:C_1210_3225Metric_Pad1.33x2.70mm_HandSolder, F.Cu at (238.5, 40.8)
- added J6: Conn_02x10_Counter_Clockwise, Connector_PinSocket_2.54mm:PinSocket_2x10_P2.54mm_Vertical, F.Cu at (94.0, 40.0)
- added R27: 1k, Resistor_SMD:R_1210_3225Metric_Pad1.30x2.65mm_HandSolder, B.Cu at (128.4, 43.0)
- added R28: 3k, Resistor_SMD:R_1210_3225Metric_Pad1.30x2.65mm_HandSolder, B.Cu at (133.4, 39.8)
- added R29: 3k, Resistor_SMD:R_1210_3225Metric_Pad1.30x2.65mm_HandSolder, B.Cu at (153.2, 39.8)
- added R30: 1k, Resistor_SMD:R_1210_3225Metric_Pad1.30x2.65mm_HandSolder, B.Cu at (148.2, 43.0)
- added R31: 120, Resistor_SMD:R_1210_3225Metric_Pad1.30x2.65mm_HandSolder, B.Cu at (133.5, 43.0)
- added R32: 120, Resistor_SMD:R_1210_3225Metric_Pad1.30x2.65mm_HandSolder, B.Cu at (153.2, 43.0)
- added TP10: TestPoint, TestPoint:TestPoint_Loop_D2.54mm_Drill1.5mm_Beaded, F.Cu at (243.0, 8.50)
- added TP11: TestPoint, TestPoint:TestPoint_Loop_D2.54mm_Drill1.5mm_Beaded, F.Cu at (50.5, 15.5)
- added TP12: TestPoint, TestPoint:TestPoint_Loop_D2.54mm_Drill1.5mm_Beaded, F.Cu at (107.5, 11.5)
- added TP13: TestPoint, TestPoint:TestPoint_Loop_D2.54mm_Drill1.5mm_Beaded, F.Cu at (21.0, 10.0)
- added TP14: TestPoint, TestPoint:TestPoint_Loop_D2.54mm_Drill1.5mm_Beaded, F.Cu at (137.0, 14.0)
- added TP15: TestPoint, TestPoint:TestPoint_Loop_D2.54mm_Drill1.5mm_Beaded, F.Cu at (194.0, 12.0)
- added TP16: TestPoint, TestPoint:TestPoint_Loop_D2.54mm_Drill1.5mm_Beaded, F.Cu at (222.5, 14.0)
- added TP5: TestPoint, TestPoint:TestPoint_Loop_D2.54mm_Drill1.5mm_Beaded, F.Cu at (71.0, 8.50)
- added TP6: TestPoint, TestPoint:TestPoint_Loop_D2.54mm_Drill1.5mm_Beaded, F.Cu at (128.0, 17.5)
- added TP7: TestPoint, TestPoint:TestPoint_Loop_D2.54mm_Drill1.5mm_Beaded, F.Cu at (42.0, 16.0)
- added TP8: TestPoint, TestPoint:TestPoint_Loop_D2.54mm_Drill1.5mm_Beaded, F.Cu at (157.5, 9.00)
- added TP9: TestPoint, TestPoint:TestPoint_Loop_D2.54mm_Drill1.5mm_Beaded, F.Cu at (214.0, 16.0)
- added U6: BTS462TATMA1, Package_TO_SOT_SMD:TO-252-4, F.Cu at (145.8, 41.0)
- added Z1: MM3Z3V0ST1G, InverterCom:SOD2512X100N, B.Cu at (128.8, 40.0)
- added Z2: MM3Z3V0ST1G, InverterCom:SOD2512X100N, B.Cu at (148.6, 40.0)
- C13, C25, C37, C49, C61, C73: value 100nF -> 220pF
- C16, C26, C44, C53, C9: moved to B.Cu
- C27, R1, R2: moved to F.Cu
- D12, D15, D18, D3, D6, D9: value FM2000GP-TP -> STTH112A; footprint InverterCom:DIOM5226X244N -> InverterCom:DIOM5126X265N; moved to B.Cu
- J1: value Conn_02x08_Counter_Clockwise -> 524265-E; footprint Connector_PinHeader_2.54mm:PinHeader_2x08_P2.54mm_Vertical -> InverterCom:524265E
- J2, J3: value TBP01R2W-508-06BE -> 524265-E; footprint InverterCom:SHDR6W100P0X508_1X6_4064X850X1240P -> InverterCom:524265E
- moved J1 87.5 mm to (46.1, 5.50), turned to 0 degrees
- moved J2 79.4 mm to (132.4, 5.50), turned to 0 degrees
- moved J3 74.7 mm to (217.7, 5.38), turned to 0 degrees
- moved C74 63.1 mm to (168.6, 40.5)
- moved C77 63.1 mm to (158.6, 40.5)
- moved TP4 63.1 mm to (76.0, 42.0)
- moved R1 44.3 mm to (194.7, 43.0)
- moved LED1 42.8 mm to (199.7, 43.0)
- moved R2 42.3 mm to (189.6, 39.8), turned to 180 degrees
- moved U5 41.7 mm to (126.0, 41.0), turned to 180 degrees
- moved LED2 37.0 mm to (194.6, 39.8)
- moved C75 34.7 mm to (51.6, 40.2)
- moved C80 32.9 mm to (41.6, 40.2)
- moved C1 32.8 mm to (31.8, 40.2)
- moved D9 27.1 mm to (43.0, 10.4)
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Connections:
- IC1 pad 14: /RESET -> /DRIVER_RESET
- IC2 pad 14: /RESET -> /DRIVER_RESET
- IC3 pad 14: /RESET -> /DRIVER_RESET
- IC4 pad 14: /RESET -> /DRIVER_RESET
- IC5 pad 14: /RESET -> /DRIVER_RESET
- IC6 pad 14: /RESET -> /DRIVER_RESET
- J1 pad 1: /GND_A -> /PH_U_H_G
- J1 pad 10: /GND_A -> unconnected-(J1-MP4-Pad10)
- J1 pad 2: /FAULT -> /SingleChannelDriver/GND_B
- J1 pad 3: /READY -> /PH_U_H_C
- J1 pad 4: /RESET -> /PH_U_L_G
- J1 pad 5: /PH_U_L -> /SingleChannelDriver1/GND_B
- J1 pad 6: /PH_U_H -> /PH_U_L_C
- J1 pad 7: /PH_V_L -> unconnected-(J1-MP1-Pad7)
- J1 pad 8: /PH_V_H -> unconnected-(J1-MP2-Pad8)
- J1 pad 9: /GND_A -> unconnected-(J1-MP3-Pad9)
- J2 pad 1: /PH_U_L_C -> /PH_V_H_G
- J2 pad 2: /SingleChannelDriver1/GND_B -> /SingleChannelDriver2/GND_B
- J2 pad 3: /PH_U_L_G -> /PH_V_H_C
- J2 pad 4: /PH_U_H_G -> /PH_V_L_G
- J2 pad 5: /SingleChannelDriver/GND_B -> /SingleChannelDriver3/GND_B
- J2 pad 6: /PH_U_H_C -> /PH_V_L_C
- J3 pad 1: /PH_V_L_C -> /PH_W_H_G
- J3 pad 2: /SingleChannelDriver3/GND_B -> /SingleChannelDriver4/GND_B
- J3 pad 3: /PH_V_L_G -> /PH_W_H_C
- J3 pad 4: /PH_V_H_G -> /PH_W_L_G
- J3 pad 5: /SingleChannelDriver2/GND_B -> /SingleChannelDriver5/GND_B
- J3 pad 6: /PH_V_H_C -> /PH_W_L_C
- TP3 pad 1: /RESET -> /DRIVER_RESET
- U5 pad 2: /+12V_ENABLE -> /GATE_DRIVE_PWR1_ENABLE
- U5 pad 5: /+12V_A -> Net-(U5-OUT)
Routing:
- net /RESET: track 267.6 -> 0.00 mm, vias 8 -> 0
- net /DRIVER_RESET: track 0.00 -> 253.2 mm, vias 0 -> 9
- net /GATE_DRIVE_PWR2_FEEDBACK: track 0.00 -> 51.6 mm, vias 0 -> 2
- net /READY: track 291.8 -> 244.6 mm, vias 11 -> 9
- net /GATE_DRIVE_PWR2_ENABLE: track 0.00 -> 44.9 mm, vias 0 -> 2
- net /PH_U_L: track 131.2 -> 87.6 mm
- net /PH_U_H: track 129.7 -> 90.0 mm
- net /GATE_DRIVE_PWR1_FEEDBACK: track 0.00 -> 35.3 mm, vias 0 -> 2
- net /+12V_ENABLE: track 26.1 -> 0.00 mm
- net /FAULT: track 275.0 -> 250.6 mm, vias 9 -> 8
- net /PH_W_H: track 113.0 -> 132.4 mm, vias 3 -> 4
- net /+12V_IN: track 27.2 -> 8.48 mm
- net /GND_A: track 6.54 -> 24.9 mm, vias 37 -> 69
- net Net-(U5-OUT): track 0.00 -> 16.5 mm, vias 0 -> 1
- net /GATE_DRIVE_PWR1_ENABLE: track 0.00 -> 15.1 mm, vias 0 -> 1
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Other:
- board text added: "1->"
- board text added: "1oo2 SSO REDUNDANT PATHWAY"
- board text added: "CONNECTOR TO CONTROL BOARD"
- board text added: "HIGH_GATE HIGH_EMTR HIGH_COL | LOW_GATE LOW_EMTR LOW_COL"
- board text added: "IMPORTANT DRIVE INFORMATION: 7A PEAK DRIVE CURRENT +15/-9V W/ ACTIVE MILLER CLAMP, DESAT PROTECTION, REDUNDANT SSO PATHWAYS"
- board text added: "INVERTER GATE DRIVE BOARD REV. B | 2026-07 | THOMAS LIAO CORZINE SMART POWER LAB, UCSC"
- board text added: "PHASE U"
- board text added: "PHASE V"
- board text added: "PHASE W"
- board text removed: "DANGER: HIGH VOLTAGE!"
- board text removed: "HIGH SIDE (COLLECTOR, EMITTER, GATE) | (GATE, EMITTER, COLLECTOR) LOW SIDE"
- board text removed: "PIN 1 ->"
