File: Hardware/Chassis2/Boards/GateDriver/GateDriver.kicad_sch (KiCad schematic)
At the start: 29 parts, among them J1 Conn_02x08_Counter_Clockwise, J2 TBP01R2W-508-06BE, J3 TBP01R2W-508-06BE, J4 TBP01R2W-508-06BE, U5 BTS462TATMA1

Commit message: update hw revision 7
Parts:
- removed J1: Conn_02x08_Counter_Clockwise, Connector_PinHeader_2.54mm:PinHeader_2x08_P2.54mm_Vertical, symbol Connector_Generic:Conn_02x08_Counter_Clockwise
- added J5: Conn_02x10_Counter_Clockwise, symbol Connector_Generic:Conn_02x10_Counter_Clockwise
- added R27, R30: 1k, Resistor_SMD:R_1210_3225Metric_Pad1.30x2.65mm_HandSolder, symbol Device:R
- added R28, R29: 3k, Resistor_SMD:R_1210_3225Metric_Pad1.30x2.65mm_HandSolder, symbol Device:R
- added U6: BTS462TATMA1, Package_TO_SOT_SMD:TO-252-4, symbol Power_Management:BTS462TATMA1
Connections:
- net +12V_A: now also J5.20 (Pin_20), R29.1, U6.5 (OUT); no longer U5.5 (OUT)
- net +3.3V_A: now also J5.18 (Pin_18)
- net FAULT: now also J5.2 (Pin_2)
- net GND_A: now also J5.1 (Pin_1), J5.12 (Pin_12), J5.14 (Pin_14), J5.17 (Pin_17), J5.9 (Pin_9), R27.2, R30.2, U6.1 (GND)
- net PH_U_H: now also J5.6 (Pin_6)
- net PH_U_L: now also J5.5 (Pin_5)
- net PH_V_H: now also J5.8 (Pin_8)
- net PH_V_L: now also J5.7 (Pin_7)
- net PH_W_H: now also J5.16 (Pin_16)
- net PH_W_L: now also J5.15 (Pin_15)
- net READY: now also J5.3 (Pin_3)
- net +12V_IN renamed GATE_DRIVE_PWR1_ENABLE
- net GATE_DRIVE_PWR1_ENABLE: now also J5.19 (Pin_19)
- net RESET renamed DRIVER_RESET
- net DRIVER_RESET: now also J5.4 (Pin_4)
- new net: R28.1, U5.5 (OUT), U6.2 (IN)
- new net GATE_DRIVE_PWR1_FB: J5.10 (Pin_10), R27.1, R28.2
- new net GATE_DRIVE_PWR2_ENABLE: J5.13 (Pin_13), U6.3 (Vbb)
- new net GATE_DRIVE_PWR2_FB: J5.11 (Pin_11), R29.2, R30.1
Other:
- note added: "CONNECTOR FROM THIS GATE DRIVER TO MAIN CONTROL BOARD ABOVE"
- note added: "Connector to control board Includes multiple redundant SSO (six-switch-off) pathways: - via gate drive reset - via gate drive power enable 1 - via gate drive power enable 2 (Gate driver power enable implemnts 1oo2, with monitoring feedback)."
- note added: "Feedback to validate power states"
- note added: "Independent gate driver power switch, reduncant 1oo2 SSO/STO"
- note added: "TODO: add zeners to this"
- note added: "TODO: replace terminal blocks potentially? (maybe not needed, as they make connecting much easier)"
- note added: "feedback pins are 0-3.3v binary (3.3v expected when +12v present)"
- note removed: "CONNECTOR FROM THIS GATE DRIVER TO MAIN CONTROL BOARD BELOW"
- company: (none) -> Corzine Lab, University of California, Santa Cruz
- title: (none) -> Open Inverter Platform - Gate Driver Board
- moved on the sheet: C77, C80, C81, C82, H1, H2, H3, H4, H5, H6, H7, H8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

Commit message: Update boards
Connections:
- net +12V_A: no longer J5.20 (Pin_20)
- net +12V_ENABLE renamed +12V_IN
- net +12V_IN: now also J5.20 (Pin_20)
- net GATE_DRIVE_PWR1_FB renamed GATE_DRIVE_PWR1_FEEDBACK
- net GATE_DRIVE_PWR2_FB renamed GATE_DRIVE_PWR2_FEEDBACK
Other:
- note added: "Feedback to validate power states Allows Main MCU and Safety coproc to independently monitor and cross-check states of switches"
- note removed: "Feedback to validate power states"
- moved on the sheet: C1, C74, C75, C77, C78, C80, C81, C82, H1, H2, H3, H4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

Commit message: eod 2026-07-08
Parts:
- removed R27, R30: 1k, Resistor_SMD:R_1210_3225Metric_Pad1.30x2.65mm_HandSolder, symbol Device:R
- removed R28, R29: 3k, Resistor_SMD:R_1210_3225Metric_Pad1.30x2.65mm_HandSolder, symbol Device:R
- removed U5, U6: BTS462TATMA1, Package_TO_SOT_SMD:TO-252-4, symbol Power_Management:BTS462TATMA1
Other:
- added sheet Redundant Monitored Power Switch (PowerSwitch.kicad_sch)
- note removed: "Feedback to validate power states Allows Main MCU and Safety coproc to independently monitor and cross-check states of switches"
- note removed: "Independent gate driver power switch, reduncant 1oo2 SSO/STO"
- note removed: "TODO: add zeners to this"
- moved on the sheet: J5

Commit message: Update Gate Driver Board, New Connector, New Desat Diode, 1oo2 SSO Pathway
Parts:
- removed J2, J3, J4: TBP01R2W-508-06BE, SHDR6W100P0X508_1X6_4064X850X1240P, symbol InverterCom:TBP01R2W-508-06BE
- removed J5: Conn_02x10_Counter_Clockwise, symbol Connector_Generic:Conn_02x10_Counter_Clockwise
- added J1, J2, J3: 524265-E, 524265E, symbol InverterCom:524265-E
- added J6: Conn_02x10_Counter_Clockwise, Connector_PinSocket_2.54mm:PinSocket_2x10_P2.54mm_Vertical, symbol Connector_Generic:Conn_02x10_Counter_Clockwise
- LED1, LED2: footprint InverterCom:LEDC3216X120N -> LEDC3216X120N
Connections:
- net +12V_IN: now also J6.20 (Pin_20)
- net +3.3V_A: now also J6.18 (Pin_18)
- net DRIVER_RESET: now also J6.4 (Pin_4)
- net FAULT: now also J6.2 (Pin_2)
- net GATE_DRIVE_PWR1_ENABLE: now also J6.19 (Pin_19)
- net GATE_DRIVE_PWR1_FEEDBACK: now also J6.10 (Pin_10)
- net GATE_DRIVE_PWR2_ENABLE: now also J6.13 (Pin_13)
- net GATE_DRIVE_PWR2_FEEDBACK: now also J6.11 (Pin_11)
- net GND_A: now also J6.1 (Pin_1), J6.12 (Pin_12), J6.14 (Pin_14), J6.17 (Pin_17), J6.9 (Pin_9)
- net PH_U_H: now also J6.6 (Pin_6)
- net PH_U_H_C: now also J1.3
- net PH_U_H_E: now also J1.2
- net PH_U_H_G: now also J1.1
- net PH_U_L: now also J6.5 (Pin_5)
- net PH_U_L_C: now also J1.6
- net PH_U_L_E: now also J1.5
- net PH_U_L_G: now also J1.4
- net PH_V_H: now also J6.8 (Pin_8)
- net PH_V_H_C: now also J2.3
- net PH_V_H_E: now also J2.2
- net PH_V_H_G: now also J2.1
- net PH_V_L: now also J6.7 (Pin_7)
- net PH_V_L_C: now also J2.6
- net PH_V_L_E: now also J2.5
- net PH_V_L_G: now also J2.4
- net PH_W_H: now also J6.16 (Pin_16)
- net PH_W_H_C: now also J3.3
- net PH_W_H_E: now also J3.2
- net PH_W_H_G: now also J3.1
- net PH_W_L: now also J6.15 (Pin_15)
- net PH_W_L_C: now also J3.6
- net PH_W_L_E: now also J3.5
- net PH_W_L_G: now also J3.4
- net READY: now also J6.3 (Pin_3)
- no-connect marks 1 -> 13
Other:
- note added: "PHASE U IGBT DRIVE CONNECTION"
- note added: "PHASE V IGBT DRIVE CONNECTION"
- note added: "PHASE W IGBT DRIVE CONNECTION"
- note removed: "TODO: replace terminal blocks potentially? (maybe not needed, as they make connecting much easier)"
- moved on the sheet: LED1, LED2, R1, R2

Commit message: Finalize Gate driver model, connectors, ss, pn
Parts:
- C1, C74, C75, C77, C78, C80, C81, C82: footprint CAPAE660X800N -> InverterCom:CAPAE660X800N
- H1, H2, H3, H4, H5, H6, H7, H8: value MountingHole -> 971150581; footprint MountingHole:MountingHole_5.3mm_M5_ISO7380_Pad -> InverterCom:971150581
- J1, J2, J3: footprint 524265E -> InverterCom:524265E
- J6: value Conn_02x10_Counter_Clockwise -> SSW-110-01-F-D
- LED1, LED2: footprint LEDC3216X120N -> InverterCom:LEDC3216X120N

Commit message: Wire harness BOMs from KiCad, board BOM re-exports, tool follows new layouts
- Four harnesses (GDVS, TSIGBT x2, CS x4, TSBCM) with per-chassis Qty
- Board BOMs move to project dirs; discovery prefers root CSV, strips
  library prefixes from footprints, reads KiCad 10 exports
- Mech list down to chassis hardware; IGBT moved to Mouser vendor
- Harness parts leave MechanicalBOM.txt (455-1135-1-ND=SXH-001T-P0.6,
  BC5011CT-ND stray cap, TSW/LA37S600/0022011042/0008500113)
Parts:
- H1, H2, H3, H4, H5, H6, H7, H8: now in the parts list
Changed lines of the file:
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@@
 	)
 	(symbol
-		(lib_id "InverterCom:Placeholder")
-		(at 113.03 20.32 0)
-		(unit 1)
-		(body_style 1)
-		(exclude_from_sim no)
-		(in_bom yes)
-		(on_board yes)
-		(in_pos_files yes)
-		(dnp no)
-		(property "Reference" "#JH1"
-			(at 112.268 20.32 0)
-			(show_name no)
-			(do_not_autoplace yes)
-			(effects
-				(font
-					(size 1.27 1.27)
-				)
-				(justify left)
-			)
-		)
-		(property "Value" "544958-E"
-			(at 123.19 20.32 0)
-			(show_name no)
-			(do_not_autoplace no)
-			(effects
-				(font
-					(size 1.27 1.27)
-				)
-			)
-		)
-		(property "Footprint" ""
-			(at 113.03 20.32 0)
-			(hide yes)
-			(show_name no)
-			(do_not_autoplace no)
-			(effects
-				(font
-					(size 1.27 1.27)
-				)
-			)
-		)
-		(property "Datasheet" ""
-			(at 113.03 20.32 0)
-			(hide yes)
-			(show_name no)
-			(do_not_autoplace no)
-			(effects
-				(font
-					(size 1.27 1.27)
-				)
-			)
-		)
-		(property "Description" ""
-			(at 113.03 20.32 0)
-			(hide yes)
-			(show_name no)
-			(do_not_autoplace no)
-			(effects
-				(font
-					(size 1.27 1.27)
-				)
-			)
-		)
-		(instances
-			(project "GateDriver"
-				(path "/d09017b7-9bb2-4a32-a451-ba266d3392f7"
-					(reference "#JH1")
-					(unit 1)
-				)
-			)
-		)
-	)
-	(symbol
 		(lib_id "InverterCom:UCM1H101MCL1GS")
 		(at 135.89 158.75 0)
@@
 	)
 	(symbol
-		(lib_id "InverterCom:Placeholder")
-		(at 172.72 19.05 0)
-		(unit 1)
-		(body_style 1)
-		(exclude_from_sim no)
-		(in_bom yes)
-		(on_board yes)
-		(in_pos_files yes)
-		(dnp no)
-		(property "Reference" "#JH2"
-			(at 171.958 19.05 0)
-			(show_name no)
-			(do_not_autoplace yes)
-			(effects
-				(font
-					(size 1.27 1.27)
-				)
-				(justify left)
-			)
-		)
-		(property "Value" "544958-E"
-			(at 182.88 19.05 0)
-			(show_name no)
-			(do_not_autoplace no)
-			(effects
-				(font
-					(size 1.27 1.27)
-				)
-			)
-		)
-		(property "Footprint" ""
-			(at 172.72 19.05 0)
-			(hide yes)
-			(show_name no)
-			(do_not_autoplace no)
-			(effects
-				(font
-					(size 1.27 1.27)
-				)
-			)
-		)
-		(property "Datasheet" ""
-			(at 172.72 19.05 0)
-			(hide yes)
-			(show_name no)
-			(do_not_autoplace no)
-			(effects
-				(font
-					(size 1.27 1.27)
-				)
-			)
-		)
-		(property "Description" ""
-			(at 172.72 19.05 0)
-			(hide yes)
-			(show_name no)
-			(do_not_autoplace no)
-			(effects
-				(font
-					(size 1.27 1.27)
-				)
-			)
-		)
-		(instances
-			(project "GateDriver"
-				(path "/d09017b7-9bb2-4a32-a451-ba266d3392f7"
-					(reference "#JH2")
-					(unit 1)
-				)
-			)
-		)
-	)
-	(symbol
 		(lib_id "InverterCom:LTST-C230CKT")
 		(at 73.66 187.96 90)
@@
 		(body_style 1)
 		(exclude_from_sim no)
-		(in_bom no)
+		(in_bom yes)
 		(on_board yes)
 		(in_pos_files yes)
@@
 		(body_style 1)
 		(exclude_from_sim no)
-		(in_bom no)
+		(in_bom yes)
 		(on_board yes)
 		(in_pos_files yes)
@@
 		(body_style 1)
 		(exclude_from_sim no)
-		(in_bom no)
+		(in_bom yes)
 		(on_board yes)
 		(in_pos_files yes)
@@
 	)
 	(symbol
-		(lib_id "InverterCom:Placeholder")
-		(at 229.87 21.59 0)
-		(unit 1)
-		(body_style 1)
-		(exclude_from_sim no)
-		(in_bom yes)
-		(on_board yes)
-		(in_pos_files yes)
-		(dnp no)
-		(property "Reference" "#JH3"
-			(at 229.108 21.59 0)
-			(show_name no)
-			(do_not_autoplace yes)
-			(effects
-				(font
-					(size 1.27 1.27)
-				)
-				(justify left)
-			)
-		)
-		(property "Value" "544958-E"
-			(at 240.03 21.59 0)
-			(show_name no)
-			(do_not_autoplace no)
-			(effects
-				(font
-					(size 1.27 1.27)
-				)
-			)
-		)
-		(property "Footprint" ""
-			(at 229.87 21.59 0)
-			(hide yes)
-			(show_name no)
-			(do_not_autoplace no)
-			(effects
-				(font
-					(size 1.27 1.27)
-				)
-			)
-		)
-		(property "Datasheet" ""
-			(at 229.87 21.59 0)
-			(hide yes)
-			(show_name no)
-			(do_not_autoplace no)
-			(effects
-				(font
-					(size 1.27 1.27)
-				)
-			)
-		)
-		(property "Description" ""
-			(at 229.87 21.59 0)
-			(hide yes)
-			(show_name no)
-			(do_not_autoplace no)
-			(effects
-				(font
-					(size 1.27 1.27)
-				)
-			)
-		)
-		(instances
-			(project "GateDriver"
-				(path "/d09017b7-9bb2-4a32-a451-ba266d3392f7"
-					(reference "#JH3")
-					(unit 1)
-				)
-			)
-		)
-	)
-	(symbol
 		(lib_id "Mechanical:MountingHole")
 		(at 205.74 167.64 90)
@@
 		(body_style 1)
 		(exclude_from_sim no)
-		(in_bom no)
+		(in_bom yes)
 		(on_board yes)
 		(in_pos_files yes)
@@
 		(body_style 1)
 		(exclude_from_sim no)
-		(in_bom no)
+		(in_bom yes)
 		(on_board yes)
 		(in_pos_files yes)
@@
 		(body_style 1)
 		(exclude_from_sim no)
-		(in_bom no)
+		(in_bom yes)
 		(on_board yes)
 		(in_pos_files yes)
@@
 		(body_style 1)
 		(exclude_from_sim no)
-		(in_bom no)
+		(in_bom yes)
 		(on_board yes)
 		(in_pos_files yes)
@@
 		(body_style 1)
 		(exclude_from_sim no)
-		(in_bom no)
+		(in_bom yes)
 		(on_board yes)
 		(in_pos_files yes)
