File: Hardware/Chassis2/Boards/ControlBoard/ADC2.kicad_sch (KiCad schematic)
At the start: 20 parts, among them IC3 MAX22530AWE+, IC4 MAX22530AWE+

Commit message: control board update progress
Parts:
- removed C13, C14, C17, C18, C19, C20: 100nF, Capacitor_SMD:C_1210_3225Metric_Pad1.33x2.70mm_HandSolder, symbol Device:C
- removed C15, C16, C21, C23: 1uF, Capacitor_SMD:C_1210_3225Metric_Pad1.33x2.70mm_HandSolder, symbol Device:C
- removed IC3, IC4: MAX22530AWE+, InverterCom:SOIC127P1032X265-16N, symbol InverterCom:MAX22530AWE+
- removed LED3, LED4: LTST-C230CKT, InverterCom:LEDC3216X120N, symbol InverterCom:LTST-C230CKT
- removed PS2, PS3: RKE-1205S_H, InverterCom:RKE1205SH, symbol InverterCom:RKE-1205S_H
- removed R6, R7: 1k, Resistor_SMD:R_1210_3225Metric_Pad1.30x2.65mm_HandSolder, symbol Device:R
- removed TP11, TP12: TestPoint, TestPoint:TestPoint_Loop_D2.54mm_Drill1.5mm_Beaded, symbol Connector:TestPoint
- added C10, C3, C9: 100nF, Capacitor_SMD:C_1210_3225Metric_Pad1.33x2.70mm_HandSolder, symbol Device:C
- added C11, C12, C4: 1uF, Capacitor_SMD:C_1210_3225Metric_Pad1.33x2.70mm_HandSolder, symbol Device:C
- added IC2: MAX22530AWE+, InverterCom:SOIC127P1032X265-16N, symbol InverterCom:MAX22530AWE+
- added TP1, TP3, TP4, TP5, TP6: TestPoint, TestPoint:TestPoint_Loop_D2.54mm_Drill1.5mm_Beaded, symbol Connector:TestPoint
Connections:
- net +3.3V_A: now also C3.2, C4.2, IC2.10 (VDDPL), IC2.11 (VDDL)
- net GND_A: now also C3.1, C4.1, IC2.9 (GNDL)
- net SPI_RX_A: now also IC2.12 (SDO)
- net SPI_SCK_A: now also IC2.14 (SCLK)
- net SPI_TX_A: now also IC2.13 (SDI)
- new net: C11.2, C9.2, IC2.7 (VDDF)
- new net: C10.1, C12.1, IC2.1 (REF)
- new net ADC1_CS_A: IC2.15 (~{CS})
- new net VSENSE_GND_B: C10.2, C11.1, C12.2, C9.1, IC2.2 (AGND), IC2.8 (GNDF), TP1.1
- new net VoltageSenseInputStage/LV_OUT: IC2.3 (AIN1), TP4.1
- new net VoltageSenseInputStage1/LV_OUT: IC2.4 (AIN2), TP6.1
- new net VoltageSenseInputStage2/LV_OUT: IC2.5 (AIN3), TP5.1
- new net VoltageSenseInputStage3/LV_OUT: IC2.6 (AIN4), TP3.1
- no-connect marks 2 -> 1
Other:
- removed sheet ADC3_5VFILTER_1
- removed sheet ADC3_5VFILTER_2
- removed sheet ADC3_5VFILTER_3
- removed sheet ADC3_5VFILTER_4
- removed sheet ADC4_5VFILTER_1
- removed sheet ADC4_5VFILTER_2
- removed sheet ADC4_5VFILTER_3
- removed sheet ADC4_5VFILTER_4
- added sheet VoltageSenseInputStage (VoltageSenseInputStage.kicad_sch)
- added sheet VoltageSenseInputStage1 (VoltageSenseInputStage.kicad_sch)
- added sheet VoltageSenseInputStage2 (VoltageSenseInputStage.kicad_sch)
- added sheet VoltageSenseInputStage3 (VoltageSenseInputStage.kicad_sch)
- note added: "ADC1: VOLTAGE SENSE (DC LINK, PHU, PHV, PHW)"
- note removed: "ADC3: MtrTemp, HallU, HallV, HallW"
- note removed: "ADC4: IGBT TEMP, THROTTLE, REGEN THROTTLE, SPARE"
- note removed: "RED LED FOR AUX +5V RAIL"
- note removed: "RED LED FOR HALL +5V RAIL"

Commit message: new stuff
Parts:
- renumbered C4 to C40, C3 to C41
Connections:
- net ADC1_INT_A: now reaches IC2.16 (~{INT})
- no-connect marks 1 -> 0
Changed lines of the file:
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@@
 		(color 0 0 0 0)
 	)
-	(no_connect
-		(at 99.06 59.69)
-	)
 	(wire
 		(pts
@@
 			)
 			(justify left)
+		)
+	)
+	(hierarchical_label "ADC1_INT_A"
+		(shape input)
+		(at 99.06 59.69 180)
+		(effects
+			(font
+				(size 1.27 1.27)
+			)
+			(justify right)
 		)
 	)
@@
 		(dnp no)
 		(fields_autoplaced yes)
-		(property "Reference" "C4"
+		(property "Reference" "C40"
 			(at 88.9 41.9099 0)
 			(effects
@@
 			(project "ControlBoard"
 				(path "/66e49eb5-2741-49e2-b48a-baf482488ca8/0caf4ddd-5aa9-47fe-b3d8-386937cdff66"
-					(reference "C4")
+					(reference "C40")
 					(unit 1)
 				)
@@
 		(on_board yes)
 		(dnp no)
-		(property "Reference" "C3"
+		(property "Reference" "C41"
 			(at 76.2 41.9099 0)
 			(effects
@@
 			(project "ControlBoard"
 				(path "/66e49eb5-2741-49e2-b48a-baf482488ca8/0caf4ddd-5aa9-47fe-b3d8-386937cdff66"
-					(reference "C3")
+					(reference "C41")
 					(unit 1)
 				)
