File: Hardware/Chassis2/Boards/ControlBoard/ADC2.kicad_sch (KiCad schematic)
At the start: 12 parts, among them IC2 MAX22530AWE+

Commit message: update hw revision 7
Connections:
- net SPI_RX_A renamed SPI_MISO_A
- net SPI_TX_A renamed SPI_MOSI_A
Other:
- company: (none) -> Corzine Lab, University of California, Santa Cruz
- title: (none) -> Open Inverter Platform - Control Board
Changed lines of the file:
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@@
 	(generator "eeschema")
 	(generator_version "10.0")
-	(paper "A4")
+	(paper "USLetter")
+	(title_block
+		(title "Open Inverter Platform - Control Board")
+		(date "2026-07-07")
+		(rev "G")
+		(company "Corzine Lab, University of California, Santa Cruz")
+		(comment 1 "Prepared by Thomas Liao")
+	)
 	(text "ADC1: VOLTAGE SENSE (DC LINK, PHU, PHV, PHW)"
 		(exclude_from_sim no)
@@
 		)
 	)
-	(hierarchical_label "SPI_TX_A"
+	(hierarchical_label "SPI_MOSI_A"
 		(shape input)
 		(at 99.06 52.07 180)
@@
 		)
 	)
-	(hierarchical_label "SPI_RX_A"
+	(hierarchical_label "SPI_MISO_A"
 		(shape input)
 		(at 99.06 49.53 180)

Commit message: Updated Gate Driver, Fixed Vsense connector on Cotnrol Board
Changed lines of the file:
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@@
-		)
-	)
-	(hierarchical_label "VSENSE_DC_LINK_B"
-		(shape input)
-		(at 200.66 71.12 0)
-		(effects
-			(font
-				(size 1.27 1.27)
-			)
-			(justify left)
 		)
 	)
@@
 		)
 	)
+	(hierarchical_label "VSENSE_PH_U_B"
+		(shape input)
+		(at 200.66 45.72 0)
+		(effects
+			(font
+				(size 1.27 1.27)
+			)
+			(justify left)
+		)
+	)
 	(hierarchical_label "VSENSE_GND_B"
 		(shape input)
 		(at 129.54 57.15 0)
+		(effects
+			(font
+				(size 1.27 1.27)
+			)
+			(justify left)
+		)
+	)
+	(hierarchical_label "VSENSE_PH_V_B"
+		(shape input)
+		(at 200.66 58.42 0)
 		(effects
 			(font
@@
 		)
 	)
+	(hierarchical_label "VSENSE_PH_W_B"
+		(shape input)
+		(at 200.66 71.12 0)
+		(effects
+			(font
+				(size 1.27 1.27)
+			)
+			(justify left)
+		)
+	)
+	(hierarchical_label "VSENSE_DC_LINK_B"
+		(shape input)
+		(at 200.66 33.02 0)
+		(effects
+			(font
+				(size 1.27 1.27)
+			)
+			(justify left)
+		)
+	)
 	(hierarchical_label "SPI_MOSI_A"
 		(shape input)
@@
 		)
 	)
-	(hierarchical_label "VSENSE_PH_U_B"
-		(shape input)
-		(at 200.66 58.42 0)
-		(effects
-			(font
-				(size 1.27 1.27)
-			)
-			(justify left)
-		)
-	)
 	(hierarchical_label "VSENSE_GND_B"
 		(shape input)
 		(at 200.66 73.66 0)
-		(effects
-			(font
-				(size 1.27 1.27)
-			)
-			(justify left)
-		)
-	)
-	(hierarchical_label "VSENSE_PH_V_B"
-		(shape input)
-		(at 200.66 45.72 0)
 		(effects
 			(font
@@
 		(effects
 			(font
-				(size 1.27 1.27)
-			)
-			(justify left)
-		)
-	)
-	(hierarchical_label "VSENSE_PH_W_B"
-		(shape input)
-		(at 200.66 33.02 0)
-		(effects
-			(font

Commit message: Labels tool, composite board views, InverterGen5 C2 branding, even render resolution
- Labels.pdf: HV warning labels, chassis ID, per-assembly labels (label cmd)
- Board sections add composite front/back views (PCB-viewer look, mirrored
  back) and layer plots now carry the drawing sheet with true plot scale
- Branding standardized to InverterGen5 C2 (cover, footer, labels)
- STEP previews render at even resolution regardless of part aspect
- Fab part titles from info.txt PartName; ALL-CAPS handling fixed
Other:
- title: Open Inverter Platform - Control Board -> InverterGen5 - Control Board
Changed lines of the file:
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@@
 	(paper "USLetter")
 	(title_block
-		(title "Open Inverter Platform - Control Board")
+		(title "InverterGen5 - Control Board")
 		(date "2026-07-07")
 		(rev "A")
