File: Hardware/Chassis2/Boards/ControlBoard/IsolatedDigitalIO.kicad_sch (KiCad schematic)
At the start: 20 parts, among them U2 ISO1212, U4 ISO1212, U5 ISO1212, U6 ISO1212

Commit message: update hw revision 7
Other:
- note added: "digital input 1-4 are mirrored to safety coprocessor allows for redundant monitoring of safety critical inputs (e-stop/kill switch, throttle/torque off limit switch, etc)"
- company: (none) -> Corzine Lab, University of California, Santa Cruz
- title: (none) -> Open Inverter Platform - Control Board
Changed lines of the file:
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@@
 	(generator "eeschema")
 	(generator_version "10.0")
-	(paper "A4")
+	(paper "USLetter")
+	(title_block
+		(title "Open Inverter Platform - Control Board")
+		(date "2026-07-07")
+		(rev "G")
+		(company "Corzine Lab, University of California, Santa Cruz")
+		(comment 1 "Prepared by Thomas Liao")
+	)
+	(text "digital input 1-4 are mirrored to safety coprocessor\nallows for redundant monitoring of safety critical inputs\n(e-stop/kill switch, throttle/torque off limit switch, etc)"
+		(exclude_from_sim no)
+		(at 119.634 67.31 0)
+		(effects
+			(font
+				(size 1.27 1.27)
+			)
+		)
+	)
 	(junction
 		(at 38.1 40.64)

Commit message: Update all repo structure, add bom tool, part cost tools, fabrication outputs, part numbering, etc, partially finished final fab files
Parts:
- U2, U4, U5, U6: value ISO1212 -> ISO1212DBQ
Changed lines of the file:
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@@
 			)
 		)
-		(property "Value" "ISO1212"
+		(property "Value" "ISO1212DBQ"
 			(at 70.7233 22.86 0)
 			(show_name no)
@@
 			)
 		)
-		(property "Value" "ISO1212"
+		(property "Value" "ISO1212DBQ"
 			(at 70.7233 120.65 0)
 			(show_name no)
@@
 			)
 		)
-		(property "Value" "ISO1212"
+		(property "Value" "ISO1212DBQ"
 			(at 146.9233 22.86 0)
 			(show_name no)
@@
 			)
 		)
-		(property "Value" "ISO1212"
+		(property "Value" "ISO1212DBQ"
 			(at 70.7233 71.12 0)
 			(show_name no)

Commit message: Labels tool, composite board views, InverterGen5 C2 branding, even render resolution
- Labels.pdf: HV warning labels, chassis ID, per-assembly labels (label cmd)
- Board sections add composite front/back views (PCB-viewer look, mirrored
  back) and layer plots now carry the drawing sheet with true plot scale
- Branding standardized to InverterGen5 C2 (cover, footer, labels)
- STEP previews render at even resolution regardless of part aspect
- Fab part titles from info.txt PartName; ALL-CAPS handling fixed
Other:
- title: Open Inverter Platform - Control Board -> InverterGen5 - Control Board
Changed lines of the file:
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@@
 	(paper "USLetter")
 	(title_block
-		(title "Open Inverter Platform - Control Board")
+		(title "InverterGen5 - Control Board")
 		(date "2026-07-07")
 		(rev "A")
