File: Hardware/Chassis2/Boards/ControlBoard/VoltageSenseInputStage.kicad_sch (KiCad schematic)
At the start: 8 parts

Commit message: control board update progress
Parts:
- renumbered C108 to C5, R75 to R23, R76 to R24, R77 to R25, R78 to R26, R79 to R27, R80 to R28, Z1 to Z4
