File: Hardware/Chassis2/Boards/ControlBoard/Control.kicad_sch (KiCad schematic)
At the start: 16 parts, among them J29 Conn_01x02_Pin

Commit message: Start new stm32h7 hardware, upgraded gate driver, etc
Parts:
- added C1: ADCM-S05R5SA224XB, ADCMS05R5SA224XB, symbol InverterCom:ADCM-S05R5SA224XB
- added C134, C136, C192: 1uF, Capacitor_SMD:C_1210_3225Metric_Pad1.33x2.70mm_HandSolder, symbol Device:C
- added C135, C137, C138, C139, C182, C183, C184, C185, C186, C187, C188, C193: 100nF, Capacitor_SMD:C_1210_3225Metric_Pad1.33x2.70mm_HandSolder, symbol Device:C
- added C189: 10uF, Capacitor_SMD:C_1210_3225Metric_Pad1.33x2.70mm_HandSolder, symbol Device:C
- added C190, C191: 2.2uF, Capacitor_SMD:C_1210_3225Metric_Pad1.33x2.70mm_HandSolder, symbol Device:C
- added JP1, JP3: Jumper_2_Small_Bridged, symbol Jumper:Jumper_2_Small_Bridged
- added JP2: Jumper_2_Small_Open, symbol Jumper:Jumper_2_Small_Open
- added R14, R15: 10k, Resistor_SMD:R_1210_3225Metric_Pad1.30x2.65mm_HandSolder, symbol Device:R
- added TP25, TP26: TestPoint, TestPoint:TestPoint_Loop_D2.54mm_Drill1.5mm_Beaded, symbol Connector:TestPoint
- added U1: STM32H723ZGTx, Package_QFP:LQFP-144_20x20mm_P0.5mm, symbol MCU_ST_STM32H7:STM32H723ZGTx
Connections:
- net +3.3V_A: now also C135.1, C136.1, C137.2, C138.2, C139.2, C182.2, C183.2, C184.2, C185.2, C186.2, C187.2, C188.2, C189.2, JP2.1 (A), JP3.2 (B), R15.2, U1.108 (VDD), U1.121 (VDD), U1.131 (VDD), U1.144 (VDD), U1.17 (VDD), U1.30 (VDD), U1.39 (VDD), U1.52 (VDD), U1.62 (VDD), U1.72 (VDD), U1.84 (VDD)
- net GND_A: now also C1.2 (-), C134.2, C137.1, C138.1, C139.1, C182.1, C183.1, C184.1, C185.1, C186.1, C187.1, C188.1, C189.1, C190.2, C191.2, C192.2, C193.2, JP1.1 (A), R14.2, U1.107 (VSS), U1.120 (VSS), U1.130 (VSS), U1.16 (VSS), U1.38 (VSS), U1.51 (VSS), U1.61 (VSS), U1.83 (VSS), U1.94 (VSS)
- new net: R14.1, TP25.1, U1.138 (BOOT0)
- new net: C1.1 (+), C134.1, JP2.2 (B), U1.6 (VBAT)
- new net: C191.1, U1.106 (VCAP)
- new net: C135.2, C136.2, U1.33 (VDDA)
- new net: R15.1, U1.143 (PDR_ON)
- new net: TP26.1, U1.25 (NRST)
- new net: C192.1, C193.1, U1.32 (VREF+)
- new net: C190.1, U1.71 (VCAP)
- new net: JP3.1 (A), U1.95 (VDD33USB)
- new net GND_ANALOG_A: JP1.2 (B), U1.31 (VSSA)
Other:
- note added: "KEEP NEAR VDDA PINS"
- note added: "PLACE NEAR VDD PINS"
- note added: "SUPERCAP FOR RTC BACKUP"
- moved on the sheet: A1, C132, C133, J29, R12, TP21, TP22, TP23, TP24, TP29, TP30, TP31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

Commit message: new stuff
Parts:
- removed A1: RaspberryPi_Pico, Module:RaspberryPi_Pico_Common_THT, symbol MCU_Module:RaspberryPi_Pico
- removed C132: 100nF, Capacitor_SMD:C_1210_3225Metric_Pad1.33x2.70mm_HandSolder, symbol Device:C
- removed C133: 10uF, Capacitor_SMD:C_1210_3225Metric_Pad1.33x2.70mm_HandSolder, symbol Device:C
- removed J29: Conn_01x02_Pin, Connector_PinHeader_2.54mm:PinHeader_1x02_P2.54mm_Vertical, symbol Connector:Conn_01x02_Pin
- removed JP3: Jumper_2_Small_Bridged, symbol Jumper:Jumper_2_Small_Bridged
- removed TP21, TP22, TP23, TP29, TP30, TP31, TP32, TP33, TP34, TP35: TestPoint, TestPoint:TestPoint_Loop_D2.54mm_Drill1.5mm_Beaded, symbol Connector:TestPoint
- added C26, C30: 22pF, Capacitor_SMD:C_1210_3225Metric_Pad1.33x2.70mm_HandSolder, symbol Device:C
- added LED1: LTST-C230CKT, LEDC3216X120N, symbol InverterCom:LTST-C230CKT
- added LED2: LTST-C230GKT, LEDC3216X120N, symbol InverterCom:LTST-C230GKT
- added R31: 4.7k, Resistor_SMD:R_1210_3225Metric_Pad1.30x2.65mm_HandSolder, symbol Device:R
- added R70: 10k, Resistor_SMD:R_1210_3225Metric_Pad1.30x2.65mm_HandSolder, symbol Device:R
- added S1, S2: TS40-66-50-R-260-SMT-TR, TS406650R260SMTTR, symbol InverterCom:TS40-66-50-R-260-SMT-TR
- added Y1: 8MHz, Crystal:Crystal_HC49-4H_Vertical, symbol Device:Crystal
- JP1: footprint (none) -> Jumper:SolderJumper-2_P1.3mm_Bridged_Pad1.0x1.5mm
- JP2: footprint (none) -> Jumper:SolderJumper-2_P1.3mm_Open_RoundedPad1.0x1.5mm
- R12: value 0 -> 4.7k
Connections:
- net +3.3V_A: now also U1.95 (VDD33USB), R70.2, S1.1 (COM_1), S1.2 (COM_2)
- net GND_A: now also C26.2, C30.2, LED1.1 (K), LED2.1 (K), S2.1 (COM_1), S2.2 (COM_2); no longer R12.2
- net BOOT_SEL: now reaches R14.1, TP25.1, U1.138 (BOOT0)
- net BOOT_SEL: now also S1.3 (NO_1), S1.4 (NO_2)
- net SPI2_SCK: now reaches U1.101 (PA9)
- net FDCAN1_RX: now reaches U1.103 (PA11)
- net FDCAN1_TX: now reaches U1.104 (PA12)
- net DEBUG_JTCK-SWDIO: now reaches U1.105 (PA13(JTMS)
- net DEBUG_JTCK-SWCLK: now reaches U1.109 (PA14(JTCK)
- net GATE_DRIVER_POWER_ENABLE: now reaches U1.111 (PC10)
- net GATE_DRIVER_FAULT: now reaches U1.112 (PC11)
- net GATE_DRIVER_FAULT: now also U1.68 (PE15)
- net GATE_DRIVER_READY: now reaches U1.113 (PC12)
- net VSENSE_ISO_ADC_INTERRUPT: now reaches U1.115 (PD1)
- net SPI1_CS: now reaches U1.116 (PD2)
- net GATE_DRIVER_RESET: now reaches U1.119 (PD5)
- net USER_DOUT_4: now reaches U1.126 (PG11)
- net USER_DOUT_3: now reaches U1.127 (PG12)
- net USER_DOUT_2: now reaches U1.128 (PG13)
- net USER_DOUT_1: now reaches U1.129 (PG14)
- net DEBUG_SWO: now reaches U1.133 (PB3(JTDO)
- net DEBUG_NJTRST: now reaches U1.134 (PB4(NJTRST))
- net FDCAN2_TX: now reaches U1.136 (PB6)
- net MOTOR_TEMP: now reaches U1.14 (PF4)
- net at U1.142 (PE1): now also R12.1
- net at U1.2 (PE3): now also R31.1
- net at U1.23 (PH0): now also C26.1, Y1.1
- net at U1.24 (PH1): now also C30.1, Y1.2
- net NRST: now reaches TP26.1, U1.25 (NRST)
- net NRST: now also R70.1, S2.3 (NO_1), S2.4 (NO_2)
- net HALL_U_ENCODER_SIN: now reaches U1.26 (PC0)
- net HALL_V_ENCODER_COS: now reaches U1.27 (PC1)
- net PHASE_W_CURRENT_SENSE_REF: now reaches U1.28 (PC2_C)
- net PHASE_W_CURRENT_SENSE_REF: now also U1.46 (PB0), U1.54 (PF14)
- net PHASE_W_CURRENT_SENSE: now reaches U1.29 (PC3_C)
- net PHASE_W_CURRENT_SENSE: now also U1.47 (PB1), U1.53 (PF13)
- net TEMP_SENSE_3: now reaches U1.34 (PA0)
- net TEMP_SENSE_2: now reaches U1.35 (PA1)
- net HALL_W: now reaches U1.36 (PA2)
- net THROTTLE_A: now reaches U1.37 (PA3)
- net THROTTLE_B: now reaches U1.40 (PA4)
- net TEMP_SENSE_1: now reaches U1.41 (PA5)
- net PHASE_V_CURRENT_SENSE: now reaches U1.42 (PA6)
- net PHASE_V_CURRENT_SENSE_REF: now reaches U1.43 (PA7)
- net PHASE_U_CURRENT_SENSE: now reaches U1.44 (PC4)
- net PHASE_U_CURRENT_SENSE_REF: now reaches U1.45 (PC5)
- net DC_LINK_CURRENT_SENSE: now reaches U1.49 (PF11)
- net DC_LINK_CURRENT_SENSE_REF: now reaches U1.50 (PF12)
- net PHASE_U_HIGH: now reaches U1.59 (PE8)
- net PHASE_U_LOW: now reaches U1.60 (PE9)
- net PHASE_V_HIGH: now reaches U1.63 (PE10)
- net PHASE_V_LOW: now reaches U1.64 (PE11)
- net PHASE_W_HIGH: now reaches U1.65 (PE12)
- net PHASE_W_LOW: now reaches U1.66 (PE13)
- net USART3_TX: now reaches U1.69 (PB10)
- net USART3_RX: now reaches U1.70 (PB11)
- net FDCAN2_RX: now reaches U1.73 (PB12)
- net SPI2_MISO: now reaches U1.75 (PB14)
- net SPI2_MOSI: now reaches U1.76 (PB15)
- net USER_DIN_6: now reaches U1.86 (PD15)
- net USER_DIN_5: now reaches U1.87 (PG2)
- net USER_DIN_4: now reaches U1.88 (PG3)
- net USER_DIN_3: now reaches U1.89 (PG4)
- net USER_DIN_2: now reaches U1.90 (PG5)
- net USER_DIN_1: now reaches U1.91 (PG6)
- net USER_DIN_7: now reaches U1.92 (PG7)
- net USER_DIN_8: now reaches U1.93 (PG8)
- net DEBUG_TRGIO: now reaches U1.97 (PC7)
- new net: LED1.2 (A), R12.2
- new net: LED2.2 (A), R31.2
- no-connect marks 5 -> 0
Other:
- note added: "bootsel switch, push for bootloader"
- note added: "reset switch, push to reset"
- note removed: "UART Debug Header"
- moved on the sheet: C192, C193, R15, TP24, TP26

Commit message: Added FRAM chip to inverter
Parts:
- added C194: 100nF, Capacitor_SMD:C_1210_3225Metric_Pad1.33x2.70mm_HandSolder, symbol Device:C
- added IC4: CY15B102Q-SXET, SOIC127P800X203-8N, symbol InverterCom:CY15B102Q-SXET
Connections:
- net +3.3V_A: now also C194.1, IC4.8 (VDD)
- net GND_A: now also C194.2, IC4.4 (VSS)
- net FRAM_SPI_SCK: now reaches U1.1 (PE2)
- net FRAM_SPI_SCK: now also IC4.6 (SCK)
- net FRAM_SPI_MISO: now reaches U1.4 (PE5)
- net FRAM_SPI_MISO: now also IC4.2 (SO)
- net FRAM_SPI_MOSI: now reaches U1.5 (PE6)
- net FRAM_SPI_MOSI: now also IC4.5 (SI)
- net FRAM_WP: now reaches U1.7 (PC13)
- net FRAM_WP: now also IC4.3 (~{WP})
- net FRAM_CS: now reaches U1.8 (PC14)
- net FRAM_CS: now also IC4.1 (~{CS})
- net FRAM_HOLD: now reaches U1.9 (PC15)
- net FRAM_HOLD: now also IC4.7 (~{HOLD})
Other:
- note added: "256KB FRAM for logs/config/hour/odo"
Changed lines of the file:
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@@
 (kicad_sch
-	(version 20250114)
+	(version 20260306)
 	(generator "eeschema")
-	(generator_version "9.0")
+	(generator_version "10.0")
 	(paper "A4")

Commit message: design changes n sruff
Connections:
- net PERIPHERAL_POWER_ENABLE: now reaches U1.12 (PF2)
- net CANBUS_12V_POWER_ENABLE: now reaches U1.98 (PC8)

Commit message: Display sorta working
Parts:
- added C27, C28: 100nF, Capacitor_SMD:C_1210_3225Metric_Pad1.33x2.70mm_HandSolder, symbol Device:C
Connections:
- net +3.3V_A: now also C135.2, C136.2, C192.1, C193.1, U1.32 (VREF+), U1.33 (VDDA); no longer C135.1, C136.1
- net BOOT_SEL: now also C27.1
- net GND_A: now also C135.1, C136.1, C27.2, C28.2
- net NRST: now also C28.1
