File: Hardware/Chassis2/Boards/ControlBoard/CurrentSensors.kicad_sch (KiCad schematic)
At the start: 4 parts, among them J3 22-04-1041, J6 22-04-1041, J8 22-04-1041, J9 22-04-1041

Commit message: design changes n sruff
Parts:
- added C140, C141: 10uF, Capacitor_SMD:C_1210_3225Metric_Pad1.33x2.70mm_HandSolder, symbol Device:C
- added C142, C143, C144, C145, C146: 100nF, Capacitor_SMD:C_1210_3225Metric_Pad1.33x2.70mm_HandSolder, symbol Device:C
- added R32, R33: 22, Resistor_SMD:R_1210_3225Metric_Pad1.30x2.65mm_HandSolder, symbol Device:R
- added R86: 499k, Resistor_SMD:R_1210_3225Metric_Pad1.30x2.65mm_HandSolder, symbol Device:R
- added U3: LT3080xQ, Package_TO_SOT_SMD:TO-263-5_TabPin3, symbol Regulator_Linear:LT3080xQ
Connections:
- net GND: now also C140.2, C141.2, C142.1, C143.2, C144.2, C145.2, C146.2, R86.1
- net +5V renamed CURRENT_SENSE_+5V_A
- net CURRENT_SENSE_+5V_A: now also C140.1, C142.2, C143.1, C144.1, C145.1, C146.1, U3.3 (OUT), U3.6 (OUT)
- new net: R32.2, R33.2, U3.5 (IN)
- new net: R86.2, U3.2 (SET)
- new net +12V_A: C141.1, R32.1, R33.1, U3.4 (V_{CONTROL})
Other:
- note added: "SERIES INPUT RESISTOR TO REDUCE LDO HEAT"
- note added: "WE USE LDO TO POWER CURRENT SENSORS AS IT HAS ~40uV NOISE"

Commit message: Display sorta working
Parts:
- added R87: 1k, Resistor_SMD:R_1210_3225Metric_Pad1.30x2.65mm_HandSolder, symbol Device:R
Connections:
- net CURRENT_SENSE_+5V_A: now also R87.2
- net GND: now also R87.1
Other:
- note added: "minimum load >1mA"
Changed lines of the file:
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@@
 	(generator_version "10.0")
 	(paper "A4")
+	(text "minimum load >1mA"
+		(exclude_from_sim no)
+		(at 140.208 103.378 0)
+		(effects
+			(font
+				(size 1.27 1.27)
+			)
+		)
+	)
 	(text "SERIES INPUT RESISTOR TO REDUCE LDO HEAT"
 		(exclude_from_sim no)
@@
 			)
 		)
+	)
+	(junction
+		(at 41.91 93.98)
+		(diameter 0)
+		(color 0 0 0 0)
+	)
+	(junction
+		(at 124.46 93.98)
+		(diameter 0)
+		(color 0 0 0 0)
+	)
+	(junction
+		(at 90.17 93.98)
+		(diameter 0)
+		(color 0 0 0 0)
+	)
+	(junction
+		(at 44.45 93.98)
+		(diameter 0)
+		(color 0 0 0 0)
 	)
 	(junction
@@
 	)
 	(junction
-		(at 41.91 93.98)
-		(diameter 0)
-		(color 0 0 0 0)
-	)
-	(junction
-		(at 90.17 93.98)
-		(diameter 0)
-		(color 0 0 0 0)
-	)
-	(junction
-		(at 44.45 93.98)
-		(diameter 0)
-		(color 0 0 0 0)
-	)
-	(junction
 		(at 31.75 93.98)
 		(diameter 0)
@@
 	(wire
 		(pts
+			(xy 124.46 93.98) (xy 130.81 93.98)
+		)
+		(stroke
+			(width 0)
+			(type default)
+		)
+	)
+	(wire
+		(pts
 			(xy 36.83 24.13) (xy 35.56 24.13)
 		)
@@
 	(wire
 		(pts
-			(xy 109.22 93.98) (xy 114.3 93.98)
+			(xy 109.22 93.98) (xy 124.46 93.98)
 		)
 		(stroke
@@
 		(pts
 			(xy 52.07 93.98) (xy 71.12 93.98)
+		)
+		(stroke
+			(width 0)
+			(type default)
+		)
+	)
+	(wire
+		(pts
+			(xy 124.46 93.98) (xy 124.46 99.06)
 		)
 		(stroke
@@
 	)
 	(label "CURRENT_SENSE_+5V_A"
-		(at 114.3 93.98 0)
+		(at 130.81 93.98 0)
 		(effects
 			(font
@@
 		(shape input)
 		(at 35.56 53.34 180)
+		(effects
+			(font
+				(size 1.27 1.27)
+			)
+			(justify right)
+		)
+	)
+	(hierarchical_label "GND"
+		(shape input)
+		(at 124.46 106.68 270)
 		(effects
 			(font
@@
 					(unit 1)
 				)
+			)
+		)
+	)
+	(symbol
+		(lib_id "Device:R")
+		(at 124.46 102.87 180)
+		(unit 1)
+		(body_style 1)
+		(exclude_from_sim no)
+		(in_bom yes)
+		(on_board yes)
+		(in_pos_files yes)
+		(dnp no)
+		(property "Reference" "R87"
+			(at 120.142 102.87 90)
+			(show_name no)
+			(do_not_autoplace no)
+			(effects
+				(font
+					(size 1.27 1.27)
+				)
+			)
+		)
+		(property "Value" "1k"
+			(at 122.682 102.87 90)
+			(show_name no)
+			(do_not_autoplace no)
+			(effects
+				(font
+					(size 1.27 1.27)
+				)
+			)
+		)
+		(property "Footprint" "Resistor_SMD:R_1210_3225Metric_Pad1.30x2.65mm_HandSolder"
+			(at 126.238 102.87 90)
+			(hide yes)
+			(show_name no)
+			(do_not_autoplace no)
+			(effects
+				(font
+					(size 1.27 1.27)
+				)
+			)
+		)
+		(property "Datasheet" ""
+			(at 124.46 102.87 0)
+			(hide yes)
+			(show_name no)
+			(do_not_autoplace no)
+			(effects
+				(font
+					(size 1.27 1.27)
+				)
+			)
+		)
+		(property "Description" "Resistor"
+			(at 124.46 102.87 0)
+			(hide yes)
+			(show_name no)
+			(do_not_autoplace no)
+			(effects
+				(font
+					(size 1.27 1.27)
+				)
+			)
+		)
+		(pin "1"
+		)
+		(pin "2"
+		)
+		(instances
+			(project "ControlBoard"
+				(path "/66e49eb5-2741-49e2-b48a-baf482488ca8/aecccc3c-ad40-4948-84a1-8bab0904bc92"
+					(reference "R87")
+					(unit 1)
+				)
