File: Hardware/Chassis2/Boards/ControlBoard/CurrentSensors.kicad_sch (KiCad schematic)
At the start: 16 parts, among them J3 22-04-1041, J6 22-04-1041, J8 22-04-1041, J9 22-04-1041, U3 LT3080xQ

Commit message: update hw revision 7
Parts:
- removed R32, R33: 22, Resistor_SMD:R_1210_3225Metric_Pad1.30x2.65mm_HandSolder, symbol Device:R
Connections:
- net +12V_A: now also U3.5 (IN)
Other:
- note added: "minimum load >1mA, load resistor ensures minimum load requirements are met"
- note removed: "SERIES INPUT RESISTOR TO REDUCE LDO HEAT"
- note removed: "minimum load >1mA"
- company: (none) -> Corzine Lab, University of California, Santa Cruz
- title: (none) -> Open Inverter Platform - Control Board
Changed lines of the file:
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@@
 	(generator "eeschema")
 	(generator_version "10.0")
-	(paper "A4")
-	(text "minimum load >1mA"
+	(paper "USLetter")
+	(title_block
+		(title "Open Inverter Platform - Control Board")
+		(date "2026-07-07")
+		(rev "G")
+		(company "Corzine Lab, University of California, Santa Cruz")
+		(comment 1 "Prepared by Thomas Liao")
+	)
+	(text "minimum load >1mA,\nload resistor ensures minimum load requirements are met"
 		(exclude_from_sim no)
-		(at 140.208 103.378 0)
-		(effects
-			(font
-				(size 1.27 1.27)
-			)
-		)
-	)
-	(text "SERIES INPUT RESISTOR TO REDUCE LDO HEAT"
-		(exclude_from_sim no)
-		(at 40.894 87.376 0)
+		(at 156.718 104.14 0)
 		(effects
 			(font
@@
 			)
 		)
-	)
-	(junction
-		(at 41.91 93.98)
-		(diameter 0)
-		(color 0 0 0 0)
 	)
 	(junction
@@
 	)
 	(junction
-		(at 90.17 93.98)
+		(at 58.42 93.98)
 		(diameter 0)
 		(color 0 0 0 0)
 	)
 	(junction
-		(at 44.45 93.98)
+		(at 90.17 93.98)
 		(diameter 0)
 		(color 0 0 0 0)
@@
 		(color 0 0 0 0)
 	)
-	(junction
-		(at 52.07 93.98)
-		(diameter 0)
-		(color 0 0 0 0)
-	)
 	(wire
 		(pts
@@
 	(wire
 		(pts
-			(xy 52.07 93.98) (xy 52.07 100.33)
-		)
-		(stroke
-			(width 0)
-			(type default)
-		)
-	)
-	(wire
-		(pts
 			(xy 25.4 93.98) (xy 31.75 93.98)
 		)
@@
 	(wire
 		(pts
-			(xy 41.91 102.87) (xy 41.91 93.98)
-		)
-		(stroke
-			(width 0)
-			(type default)
-		)
-	)
-	(wire
-		(pts
-			(xy 31.75 93.98) (xy 41.91 93.98)
+			(xy 58.42 96.52) (xy 58.42 93.98)
+		)
+		(stroke
+			(width 0)
+			(type default)
+		)
+	)
+	(wire
+		(pts
+			(xy 58.42 93.98) (xy 71.12 93.98)
+		)
+		(stroke
+			(width 0)
+			(type default)
+		)
+	)
+	(wire
+		(pts
+			(xy 31.75 93.98) (xy 58.42 93.98)
 		)
 		(stroke
@@
 	(wire
 		(pts
-			(xy 54.61 96.52) (xy 54.61 102.87)
-		)
-		(stroke
-			(width 0)
-			(type default)
-		)
-	)
-	(wire
-		(pts
 			(xy 109.22 104.14) (xy 109.22 102.87)
 		)
@@
 	(wire
 		(pts
-			(xy 44.45 93.98) (xy 44.45 100.33)
-		)
-		(stroke
-			(width 0)
-			(type default)
-		)
-	)
-	(wire
-		(pts
-			(xy 41.91 93.98) (xy 44.45 93.98)
-		)
-		(stroke
-			(width 0)
-			(type default)
-		)
-	)
-	(wire
-		(pts
 			(xy 90.17 104.14) (xy 90.17 102.87)
 		)
@@
 	(wire
 		(pts
-			(xy 54.61 102.87) (xy 41.91 102.87)
+			(xy 71.12 96.52) (xy 58.42 96.52)
 		)
 		(stroke
@@
 	(wire
 		(pts
-			(xy 52.07 93.98) (xy 71.12 93.98)
-		)
-		(stroke
-			(width 0)
-			(type default)
-		)
-	)
-	(wire
-		(pts
 			(xy 124.46 93.98) (xy 124.46 99.06)
-		)
-		(stroke
-			(width 0)
-			(type default)
-		)
-	)
-	(wire
-		(pts
-			(xy 71.12 96.52) (xy 54.61 96.52)
 		)
 		(stroke
@@
 	)
 	(symbol
-		(lib_id "Device:R")
-		(at 48.26 93.98 90)
-		(unit 1)
-		(body_style 1)
-		(exclude_from_sim no)
-		(in_bom yes)
-		(on_board yes)
-		(in_pos_files yes)
-		(dnp no)
-		(property "Reference" "R33"
-			(at 48.26 89.408 90)
-			(show_name no)
-			(do_not_autoplace no)
-			(effects
-				(font
-					(size 1.27 1.27)
-				)
-			)
-		)
-		(property "Value" "22"
-			(at 48.26 91.948 90)
-			(show_name no)
-			(do_not_autoplace no)
-			(effects
-				(font
-					(size 1.27 1.27)
-				)
-			)
-		)
-		(property "Footprint" "Resistor_SMD:R_1210_3225Metric_Pad1.30x2.65mm_HandSolder"
-			(at 48.26 95.758 90)
-			(hide yes)
-			(show_name no)
-			(do_not_autoplace no)
-			(effects
-				(font
-					(size 1.27 1.27)
-				)
-			)
-		)
-		(property "Datasheet" ""
-			(at 48.26 93.98 0)
-			(hide yes)
-			(show_name no)
-			(do_not_autoplace no)
-			(effects
-				(font
-					(size 1.27 1.27)
-				)
-			)
-		)
-		(property "Description" "Resistor"
-			(at 48.26 93.98 0)
-			(hide yes)
-			(show_name no)
-			(do_not_autoplace no)
-			(effects
-				(font
-					(size 1.27 1.27)
-				)
-			)
-		)
-		(pin "1"
-		)
-		(pin "2"
-		)
-		(instances
-			(project "ControlBoard"
-				(path "/66e49eb5-2741-49e2-b48a-baf482488ca8/aecccc3c-ad40-4948-84a1-8bab0904bc92"
-					(reference "R33")
-					(unit 1)
-				)
-			)
-		)
-	)
-	(symbol
 		(lib_id "InverterCom:22-04-1041")
 		(at 35.56 53.34 0)
@@
 					(unit 1)
 				)
-			)
-		)
-	)
-	(symbol
-		(lib_id "Device:R")
-		(at 48.26 100.33 90)
-		(unit 1)
-		(body_style 1)
-		(exclude_from_sim no)
-		(in_bom yes)
-		(on_board yes)
-		(in_pos_files yes)
-		(dnp no)
-		(property "Reference" "R32"
-			(at 48.26 96.012 90)
-			(show_name no)
-			(do_not_autoplace no)
-			(effects
-				(font
-					(size 1.27 1.27)
-				)
-			)
-		)
-		(property "Value" "22"
-			(at 48.26 98.552 90)
-			(show_name no)
-			(do_not_autoplace no)
-			(effects
-				(font
-					(size 1.27 1.27)
-				)
-			)
-		)
-		(property "Footprint" "Resistor_SMD:R_1210_3225Metric_Pad1.30x2.65mm_HandSolder"
-			(at 48.26 102.108 90)
-			(hide yes)
-			(show_name no)
-			(do_not_autoplace no)
-			(effects
-				(font
-					(size 1.27 1.27)
-				)
-			)
-		)
-		(property "Datasheet" ""
-			(at 48.26 100.33 0)
-			(hide yes)
-			(show_name no)
-			(do_not_autoplace no)
-			(effects
-				(font
-					(size 1.27 1.27)
-				)
-			)
-		)
-		(property "Description" "Resistor"
-			(at 48.26 100.33 0)
-			(hide yes)
-			(show_name no)
-			(do_not_autoplace no)
-			(effects
-				(font
-					(size 1.27 1.27)
-				)
-			)
-		)
-		(pin "1"
-		)
-		(pin "2"
-		)
-		(instances
-			(project "ControlBoard"
-				(path "/66e49eb5-2741-49e2-b48a-baf482488ca8/aecccc3c-ad40-4948-84a1-8bab0904bc92"
-					(reference "R32")
-					(unit 1)
-				)

Commit message: eod 2026-07-08
Parts:
- J3, J6, J8, J9: footprint SHDR4W64P0X250_1X4_950X580X1210P -> InverterCom:SHDR4W64P0X250_1X4_950X580X1210P
- U3: footprint Package_TO_SOT_SMD:TO-263-5_TabPin3 -> Package_TO_SOT_SMD:TO-263-5_TabPin6
Changed lines of the file:
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@@
 			)
 		)
-		(property "Footprint" "SHDR4W64P0X250_1X4_950X580X1210P"
+		(property "Footprint" "InverterCom:SHDR4W64P0X250_1X4_950X580X1210P"
 			(at 102.87 122.86 0)
 			(hide yes)
@@
 			)
 		)
-		(property "Footprint" "SHDR4W64P0X250_1X4_950X580X1210P"
+		(property "Footprint" "InverterCom:SHDR4W64P0X250_1X4_950X580X1210P"
 			(at 52.07 148.26 0)
 			(hide yes)
@@
 			)
 		)
-		(property "Footprint" "SHDR4W64P0X250_1X4_950X580X1210P"
+		(property "Footprint" "InverterCom:SHDR4W64P0X250_1X4_950X580X1210P"
 			(at 52.07 122.86 0)
 			(hide yes)
@@
 			)
 		)
-		(property "Footprint" "Package_TO_SOT_SMD:TO-263-5_TabPin3"
+		(property "Footprint" "Package_TO_SOT_SMD:TO-263-5_TabPin6"
 			(at 73.66 104.14 0)
 			(hide yes)
@@
 			)
 		)
-		(property "Footprint" "SHDR4W64P0X250_1X4_950X580X1210P"
+		(property "Footprint" "InverterCom:SHDR4W64P0X250_1X4_950X580X1210P"
 			(at 102.87 148.26 0)
 			(hide yes)

Commit message: Add Schematic / Controlboard Support for Multi-Drive Mulit-Phase, DDCP
Connections:
- net CURRENT_SENSE_+5V_A renamed +5V_ISENSE_A
Changed lines of the file:
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@@
+		)
+	)
+	(label "CURRENT_SENSE_+5V_A"
+		(at 119.38 72.39 0)
+		(effects
+			(font
+				(size 1.27 1.27)
+			)
+			(justify left bottom)
 		)
 	)
@@
 		(effects
 			(font
+				(size 1.27 1.27)
+			)
+			(justify right)
+		)
+	)
+	(hierarchical_label "+5V_ISENSE_A"
+		(shape input)
+		(at 119.38 72.39 180)
+		(effects
+			(font

Commit message: Update all repo structure, add bom tool, part cost tools, fabrication outputs, part numbering, etc, partially finished final fab files
Parts:
- U3: value LT3080xQ -> LT3080IQ#PBF
Changed lines of the file:
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@@
 			)
 		)
-		(property "Value" "LT3080xQ"
+		(property "Value" "LT3080IQ#PBF"
 			(at 78.74 88.9 0)
 			(show_name no)
