File: Hardware/Chassis2/Boards/ControlBoard/USBUARTInterface.kicad_sch (KiCad schematic)
At the start: 9 parts, among them IC1 MCP2221A-I_ST, J4 UJ20-C-H-G-MSMT-4B-P16-TR

Commit message: Added New Control Board
Parts:
- removed J4: UJ20-C-H-G-MSMT-4B-P16-TR, UJ20CHGMSMT4BP16TR, symbol InverterCom:UJ20-C-H-G-MSMT-4B-P16-TR
- removed R32, R33: 4.7k, Resistor_SMD:R_1210_3225Metric_Pad1.30x2.65mm_HandSolder, symbol Device:R
- added J15: UJ32-C-H-G-DSMT-3-P24-TR, UJ32CHGDSMT3P24TR, symbol InverterCom:UJ32-C-H-G-DSMT-3-P24-TR
- added R71, R72: 4.7k, Resistor_SMD:R_1210_3225Metric_Pad1.30x2.65mm_HandSolder, symbol Device:R
Connections:
- net +5V_A: now also J15.A4 (VBUS_1), J15.A9 (VBUS_2), J15.B4 (VBUS_3), J15.B9 (VBUS_4)
- net GND_A: now also J15.1 (MH), J15.2 (MH), J15.3 (MH1), J15.4 (MH2), J15.5 (MH3), J15.6 (MH4), J15.A1 (GND_1), J15.A12 (GND_2), J15.B1 (GND_3), J15.B12 (GND_4), R71.2, R72.2
- net USB_N: now also J15.A7 (DN1), J15.B7 (DN2)
- net USB_P: now also J15.A6 (DP1), J15.B6 (DP2)
- new net: J15.A5 (CC1), R72.1
- new net: J15.B5 (CC2), R71.1
- no-connect marks 4 -> 12

Commit message: Display sorta working
Connections:
- net +3.3V_A: now also IC1.11 (VUSB)
- net +5V_A: no longer IC1.11 (VUSB)
- net at R35.1: now also IC1.8 (GP3); no longer IC1.2 (GP0)
- net at IC1.3 (GP1): no longer R36.1
- net at IC1.7 (GP2): now also R36.1
- no-connect marks 12 -> 14
Other:
- note added: "gp0 and 1 are default to uart tx/rx indicators"
- moved on the sheet: R35, R36
Changed lines of the file:
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@@
 	(generator_version "10.0")
 	(paper "A4")
+	(text "gp0 and 1 are default\nto uart tx/rx indicators"
+		(exclude_from_sim no)
+		(at 34.036 44.958 0)
+		(effects
+			(font
+				(size 1.27 1.27)
+			)
+		)
+	)
 	(text "USB to uart interface"
 		(exclude_from_sim no)
@@
 	)
 	(no_connect
+		(at 50.8 52.07)
+	)
+	(no_connect
 		(at 78.74 59.69)
 	)
@@
 	)
 	(no_connect
+		(at 50.8 49.53)
+	)
+	(no_connect
 		(at 110.49 46.99)
 	)
@@
 	(wire
 		(pts
-			(xy 43.18 52.07) (xy 50.8 52.07)
-		)
-		(stroke
-			(width 0)
-			(type default)
-		)
-	)
-	(wire
-		(pts
 			(xy 110.49 54.61) (xy 105.41 54.61)
 		)
@@
 	(wire
 		(pts
+			(xy 50.8 68.58) (xy 50.8 62.23)
+		)
+		(stroke
+			(width 0)
+			(type default)
+		)
+	)
+	(wire
+		(pts
 			(xy 48.26 57.15) (xy 50.8 57.15)
 		)
@@
 	(wire
 		(pts
-			(xy 43.18 46.99) (xy 43.18 52.07)
-		)
-		(stroke
-			(width 0)
-			(type default)
-		)
-	)
-	(wire
-		(pts
-			(xy 45.72 49.53) (xy 45.72 39.37)
-		)
-		(stroke
-			(width 0)
-			(type default)
-		)
-	)
-	(wire
-		(pts
-			(xy 38.1 46.99) (xy 43.18 46.99)
+			(xy 78.74 69.85) (xy 78.74 62.23)
+		)
+		(stroke
+			(width 0)
+			(type default)
+		)
+	)
+	(wire
+		(pts
+			(xy 45.72 68.58) (xy 50.8 68.58)
 		)
 		(stroke
@@
 	(wire
 		(pts
-			(xy 50.8 49.53) (xy 45.72 49.53)
-		)
-		(stroke
-			(width 0)
-			(type default)
-		)
-	)
-	(wire
-		(pts
-			(xy 45.72 39.37) (xy 38.1 39.37)
+			(xy 78.74 69.85) (xy 80.01 69.85)
 		)
 		(stroke
@@
 		)
 	)
-	(label "+5V_A"
-		(at 78.74 54.61 0)
-		(effects
-			(font
-				(size 1.27 1.27)
-			)
-			(justify left bottom)
-		)
-	)
 	(label "USB_N"
 		(at 110.49 49.53 180)
@@
 	(hierarchical_label "BOOTSEL"
 		(shape input)
-		(at 30.48 39.37 180)
+		(at 87.63 69.85 0)
+		(effects
+			(font
+				(size 1.27 1.27)
+			)
+			(justify left)
+		)
+	)
+	(hierarchical_label "UART_RX"
+		(shape input)
+		(at 48.26 57.15 180)
 		(effects
 			(font
@@
 		)
 	)
-	(hierarchical_label "UART_RX"
-		(shape input)
-		(at 48.26 57.15 180)
+	(hierarchical_label "+3.3V_A"
+		(shape input)
+		(at 78.74 54.61 0)
+		(effects
+			(font
+				(size 1.27 1.27)
+			)
+			(justify left)
+		)
+	)
+	(hierarchical_label "GND_A"
+		(shape input)
+		(at 125.73 77.47 270)
 		(effects
 			(font
@@
 	(hierarchical_label "GND_A"
 		(shape input)
-		(at 125.73 77.47 270)
+		(at 143.51 64.77 0)
+		(effects
+			(font
+				(size 1.27 1.27)
+			)
+			(justify left)
+		)
+	)
+	(hierarchical_label "GND_A"
+		(shape input)
+		(at 110.49 67.31 180)
 		(effects
 			(font
@@
 	(hierarchical_label "GND_A"
 		(shape input)
-		(at 143.51 64.77 0)
+		(at 143.51 69.85 0)
 		(effects
 			(font
@@
 		)
 	)
-	(hierarchical_label "GND_A"
-		(shape input)
-		(at 110.49 67.31 180)
+	(hierarchical_label "+3.3V_A"
+		(shape input)
+		(at 35.56 54.61 180)
 		(effects
 			(font
@@
 	(hierarchical_label "GND_A"
 		(shape input)
-		(at 143.51 69.85 0)
+		(at 143.51 59.69 0)
 		(effects
 			(font
@@
 		)
 	)
-	(hierarchical_label "+3.3V_A"
-		(shape input)
-		(at 35.56 54.61 180)
-		(effects
-			(font
-				(size 1.27 1.27)
-			)
-			(justify right)
-		)
-	)
-	(hierarchical_label "GND_A"
-		(shape input)
-		(at 143.51 59.69 0)
-		(effects
-			(font
-				(size 1.27 1.27)
-			)
-			(justify left)
-		)
-	)
 	(hierarchical_label "RESET"
 		(shape input)
-		(at 30.48 46.99 180)
+		(at 38.1 68.58 180)
 		(effects
 			(font
@@
 	(symbol
 		(lib_id "Device:R")
-		(at 34.29 39.37 270)
+		(at 83.82 69.85 90)
 		(unit 1)
 		(body_style 1)
@@
 		(dnp no)
 		(property "Reference" "R35"
-			(at 35.56 33.782 0)
+			(at 82.55 75.438 0)
 			(show_name no)
 			(do_not_autoplace no)
@@
 		)
 		(property "Value" "4.7k"
-			(at 33.02 33.02 0)
+			(at 85.09 76.2 0)
 			(show_name no)
 			(do_not_autoplace no)
@@
 		)
 		(property "Footprint" "Resistor_SMD:R_1210_3225Metric_Pad1.30x2.65mm_HandSolder"
-			(at 34.29 37.592 90)
+			(at 83.82 71.628 90)
 			(hide yes)
 			(show_name no)
@@
 		)
 		(property "Datasheet" ""
-			(at 34.29 39.37 0)
+			(at 83.82 69.85 0)
 			(hide yes)
 			(show_name no)
@@
 		)
 		(property "Description" "Resistor"
-			(at 34.29 39.37 0)
+			(at 83.82 69.85 0)
 			(hide yes)
 			(show_name no)
@@
 	(symbol
 		(lib_id "Device:R")
-		(at 34.29 46.99 270)
+		(at 41.91 68.58 270)
 		(unit 1)
 		(body_style 1)
@@
 		(dnp no)
 		(property "Reference" "R36"
-			(at 35.56 41.402 0)
+			(at 43.18 62.992 0)
 			(show_name no)
 			(do_not_autoplace no)
@@
 		)
 		(property "Value" "4.7k"
-			(at 33.02 40.64 0)
+			(at 40.64 62.23 0)
 			(show_name no)
 			(do_not_autoplace no)
@@
 		)
 		(property "Footprint" "Resistor_SMD:R_1210_3225Metric_Pad1.30x2.65mm_HandSolder"
-			(at 34.29 45.212 90)
+			(at 41.91 66.802 90)
 			(hide yes)
 			(show_name no)
@@
 		)
 		(property "Datasheet" ""
-			(at 34.29 46.99 0)
+			(at 41.91 68.58 0)
 			(hide yes)
 			(show_name no)
@@
 		)
 		(property "Description" "Resistor"
-			(at 34.29 46.99 0)
-			(hide yes)
-			(show_name no)
+			(at 41.91 68.58 0)
+			(hide yes)
+			(show_name no)
