File: Hardware/Chassis2/Boards/ControlBoard/ControlBoard.kicad_pcb (KiCad board)
At the start: 6 copper layers, 260 x 45 mm, 237 parts, among them IC1 TPS389006ADJRTER, IC2 MAX22530AWE+, IC3 ISO1042BDWVR, IC4 CY15B102Q-SXET, IC5 ISO1042BDWVR, IC6 ISO1042BDWVR, IC7 ISO1042BDWVR, J1 B2B-XH-AM_LF__SN_, J10 Conn_02x03_Counter_Clockwise, J11 TBP01R2W-508-06BE, J12 Conn_02x08_Counter_Clockwise, J13 Conn_02x03_Counter_Clockwise, J14 Conn_02x10_Counter_Clockwise, J2 Conn_02x10_Counter_Clockwise, J3 22-04-1041, J4 B2B-XH-AM_LF__SN_, J5 B2B-XH-AM_LF__SN_, J6 22-04-1041, J7 Conn_02x08_Counter_Clockwise, J8 22-04-1041, J9 22-04-1041, U1 STM32H723ZGTx, U2 ISO1212, U3 LT3080xQ, U4 ISO1212, U5 ISO1212, U6 ISO1212, U7 BTS462TATMA1, U8 BTS462TATMA1, U9 STM32G474RCTx, Y1 8MHz, Y2 8MHz

Commit message: fix power monitor ic connections
Connections:
- IC1 pad 13: /Control/Power Supply Monitor/FAULT -> /DRIVER_RESET
- IC1 pad 5: /Control/Power Supply Monitor/ENABLE -> /Control/Main Processor/POWERMON_ENABLE
- IC1 pad 7: /Control/Power Supply Monitor/SLEEP -> /Control/Main Processor/POWERMON_SLEEP
- U1 pad 122: unconnected-(U1-PD6-Pad122) -> /Control/Main Processor/POWERMON_SLEEP
- U1 pad 123: unconnected-(U1-PD7-Pad123) -> /Control/Main Processor/POWERMON_ENABLE
Routing:
- net /DRIVER_RESET: track 0.00 -> 120.3 mm, vias 0 -> 8
- net /Control/Main Processor/VOLTAGE_MONITOR_I2C_SDA: track 0.00 -> 67.7 mm, vias 0 -> 2
- net /Control/Main Processor/VOLTAGE_MONITOR_I2C_SCL: track 0.00 -> 33.1 mm, vias 0 -> 2
- net /ONBOARD_12V_ENABLE_A: track 72.9 -> 103.8 mm, vias 2 -> 3
- net /GATE_DRIVE_PWR2_FEEDBACK: track 0.00 -> 30.4 mm, vias 0 -> 2
- net /Control/Main Processor/POWERMON_ENABLE: track 0.00 -> 3.12 mm, vias 0 -> 1
- net /Control/Main Processor/POWERMON_SLEEP: track 0.00 -> 3.10 mm, vias 0 -> 1
- net /GATE_DRIVE_PWR1_FEEDBACK: track 0.00 -> 2.78 mm, vias 0 -> 1
- net Net-(IC1-ADDR): track 4.98 -> 6.04 mm
- net /+3.3V_A: track 28.0 -> 29.1 mm
