File: Hardware/Chassis2/Boards/ControlBoard/CANTransciever.kicad_sch (KiCad schematic)
At the start: 10 parts, among them IC3 ISO1042BDWVR

Commit message: update hw revision 7
Parts:
- added IC5: ISO1042BDWVR, InverterCom:SOIC127P1150X280-8N, symbol InverterCom:ISO1042BDWVR
Connections:
- net +3.3V_A: now also IC5.1 (VCC1)
- net CAN_5V: now also IC5.8 (VCC2)
- net CAN_GND: now also IC5.5 (GND2)
- net GND_A: now also IC5.4 (GND1)
- net CAN_L: now reaches FL2.2, IC3.6 (CANL)
- net CAN_L: now also IC5.6 (CANL)
- net CAN_H: now reaches FL2.1, IC3.7 (CANH)
- net CAN_H: now also IC5.7 (CANH)
- net CAN_RX renamed A_CAN_RX
- net CAN_TX renamed A_CAN_TX
- new net B_CAN_RX: IC5.3 (RXD)
- new net B_CAN_TX: IC5.2 (TXD)
Other:
- note added: "two can transcievers, allows safety coproc to snoop and interact with can traffic, if needed. provides redundant path to read and cross-check motor torque commands, if using canbus for torque cmd over throttle A/B inpts"
- company: (none) -> Corzine Lab, University of California, Santa Cruz
- title: (none) -> Open Inverter Platform - Control Board
- moved on the sheet: C14, FL2, PS2

Commit message: Labels tool, composite board views, InverterGen5 C2 branding, even render resolution
- Labels.pdf: HV warning labels, chassis ID, per-assembly labels (label cmd)
- Board sections add composite front/back views (PCB-viewer look, mirrored
  back) and layer plots now carry the drawing sheet with true plot scale
- Branding standardized to InverterGen5 C2 (cover, footer, labels)
- STEP previews render at even resolution regardless of part aspect
- Fab part titles from info.txt PartName; ALL-CAPS handling fixed
Other:
- title: Open Inverter Platform - Control Board -> InverterGen5 - Control Board
Changed lines of the file:
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@@
 	(paper "USLetter")
 	(title_block
-		(title "Open Inverter Platform - Control Board")
+		(title "InverterGen5 - Control Board")
 		(date "2026-07-07")
 		(rev "A")
