File: Hardware/Chassis2/Boards/ControlBoard/HWOCP.kicad_sch (KiCad schematic)
At the start: 8 parts, among them U10 LM397, U11 LM397, U12 LM397, U13 LM397

Commit message: Labels tool, composite board views, InverterGen5 C2 branding, even render resolution
- Labels.pdf: HV warning labels, chassis ID, per-assembly labels (label cmd)
- Board sections add composite front/back views (PCB-viewer look, mirrored
  back) and layer plots now carry the drawing sheet with true plot scale
- Branding standardized to InverterGen5 C2 (cover, footer, labels)
- STEP previews render at even resolution regardless of part aspect
- Fab part titles from info.txt PartName; ALL-CAPS handling fixed
Other:
- title: Open Inverter Platform - Control Board -> InverterGen5 - Control Board
Changed lines of the file:
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@@
 	(paper "USLetter")
 	(title_block
-		(title "Open Inverter Platform - Control Board")
+		(title "InverterGen5 - Control Board")
 		(date "2026-07-07")
 		(rev "A")
