File: Hardware/Chassis2/Boards/ControlBoard/SafetyCoprocessor.kicad_sch (KiCad schematic)
At the start: 18 parts, among them U9 STM32G474RCTx, Y2 8MHz

Commit message: eod 2026-07-08
Parts:
- removed C148: 1uF, Capacitor_SMD:C_1210_3225Metric_Pad1.33x2.70mm_HandSolder, symbol Device:C
- removed C195, C196, C199: 100nF, Capacitor_SMD:C_1210_3225Metric_Pad1.33x2.70mm_HandSolder, symbol Device:C
Connections:
- net GND_A: now also R89.2

Commit message: Update all repo structure, add bom tool, part cost tools, fabrication outputs, part numbering, etc, partially finished final fab files
Parts:
- U9: value STM32G474RCTx -> STM32G474RCT3
Changed lines of the file:
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@@
 			)
 		)
-		(property "Value" "STM32G474RCTx"
+		(property "Value" "STM32G474RCT3"
 			(at 151.13 73.2946 90)
 			(show_name no)

Commit message: Labels tool, composite board views, InverterGen5 C2 branding, even render resolution
- Labels.pdf: HV warning labels, chassis ID, per-assembly labels (label cmd)
- Board sections add composite front/back views (PCB-viewer look, mirrored
  back) and layer plots now carry the drawing sheet with true plot scale
- Branding standardized to InverterGen5 C2 (cover, footer, labels)
- STEP previews render at even resolution regardless of part aspect
- Fab part titles from info.txt PartName; ALL-CAPS handling fixed
Other:
- title: Open Inverter Platform - Control Board -> InverterGen5 - Control Board
Changed lines of the file:
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@@
 	(paper "USLetter")
 	(title_block
-		(title "Open Inverter Platform - Control Board")
+		(title "InverterGen5 - Control Board")
 		(date "2026-07-07")
 		(rev "A")
