File: Hardware/Chassis2/Boards/MainBoard/MainBoard.kicad_pcb (KiCad board)
At the start: 6 copper layers, 297.5 x 60 mm, 140 parts, among them IC1 MAX22530AWE+, IC13 DRDNB21D-7, IC14 DRDNB21D-7, IC2 MAX22530AWE+, IC5 MCP2515-e_ST, IC6 ISO1042BDWVR, J1 Conn_02x08_Counter_Clockwise, J11 Conn_02x10_Counter_Clockwise, J12 Conn_02x10_Counter_Clockwise, J13 Conn_02x10_Counter_Clockwise, J14 Conn_02x10_Counter_Clockwise, J2 Conn_02x08_Counter_Clockwise, J3 Conn_02x08_Counter_Clockwise, J4 TBP01R1-508-06BE, J5 Conn_02x10_Counter_Clockwise, J6 TBP01R2-508-06BE, K1 AWHSH105D00G, K2 AWHSH105D00G, K3 AWHSH105D00G, Y1 8MHz

Commit message: Add New Mainboard
Parts:
- removed C1, C10, C25, C3, C31, C32, C34, C5, C6, C9: 100nF, Capacitor_SMD:C_1210_3225Metric_Pad1.33x2.70mm_HandSolder
- removed C108, C109, C110, C111, C112, C113, C114, C115: 10nF, Capacitor_SMD:C_1210_3225Metric_Pad1.33x2.70mm_HandSolder
- removed C11, C12, C2, C4, C7, C8: 1uF, Capacitor_SMD:C_1210_3225Metric_Pad1.33x2.70mm_HandSolder
- removed C124, C125, C134, C135, C136, C137, C138, C139, C27, C28, C29, C33: 10uF, Capacitor_SMD:C_1210_3225Metric_Pad1.33x2.70mm_HandSolder
- removed C148, C149, C150, C151, C152, C153, C154, C155, C156, C157, C158, C159: UCM1H101MCL1GS, InverterCom:CAPAE660X800N
- removed C26, C30, C35, C36, C37: 22pF, Capacitor_SMD:C_1210_3225Metric_Pad1.33x2.70mm_HandSolder
- removed FL1: ACT45B-101-2P-TL003, InverterCom:ACT45B1012PTL003
- removed G***: LOGO, InverterCom:HIGHVOLTAGE_20mm
- removed IC1, IC2: MAX22530AWE+, InverterCom:SOIC127P1032X265-16N
- removed IC13, IC14: DRDNB21D-7, InverterCom:SOT65P210X110-6N
- removed IC5: MCP2515-e_ST, InverterCom:SOP65P640X120-20N
- removed IC6: ISO1042BDWVR, InverterCom:SOIC127P1150X280-8N
- removed J11, J5: Conn_02x10_Counter_Clockwise, Connector_PinHeader_2.54mm:PinHeader_2x10_P2.54mm_Vertical
- removed J3: Conn_02x08_Counter_Clockwise, Connector_PinSocket_2.54mm:PinSocket_2x08_P2.54mm_Vertical
- removed J4: TBP01R1-508-06BE, InverterCom:TBP01R150806BE
- removed K1, K2, K3: AWHSH105D00G, InverterCom:AWHSH105D00G
- removed LED2: LTST-C230CKT, InverterCom:LEDC3216X120N
- removed PS1, PS13, PS14, PS4: RKE-1205S_H, InverterCom:RKE1205SH
- removed PS2: REC10K-2424DAW_H2, InverterCom:REC10K-AW
- removed R100, R102, R104, R106: 5k, Resistor_SMD:R_1210_3225Metric_Pad1.30x2.65mm_HandSolder
- removed R101, R103, R105, R76, R88, R94, R99: 1k, Resistor_SMD:R_1210_3225Metric_Pad1.30x2.65mm_HandSolder
- removed R75, R81, R87, R93: 2k, Resistor_SMD:R_1210_3225Metric_Pad1.30x2.65mm_HandSolder
- removed R77, R78, R79, R80, R83, R84, R85, R86, R89, R90, R91, R92, R95, R96, R97, R98: 250k, Resistor_SMD:R_1210_3225Metric_Pad1.30x2.65mm_HandSolder
- removed R8: 4.7k, Resistor_SMD:R_1210_3225Metric_Pad1.30x2.65mm_HandSolder
- removed R9: 120, Resistor_SMD:R_1210_3225Metric_Pad1.30x2.65mm_HandSolder
- removed TP1, TP10, TP2, TP3, TP4, TP5, TP6, TP7, TP8, TP9: TestPoint, TestPoint:TestPoint_Loop_D2.54mm_Drill1.5mm_Beaded
- removed Y1: 8MHz, Crystal:Crystal_HC49-4H_Vertical
- removed Z1, Z2, Z3, Z4, Z5, Z6, Z7, Z8: SZMMSZ4678T1G, InverterCom:SOD3716X135N
- added ?: , , F.Cu at (246.5, 39.7)
- added ?: , , F.Cu at (153.7, 42.0)
- added ?: , , F.Cu at (191.7, 39.7)
- added ?: , , F.Cu at (257.3, 18.7)
- added ?: , , F.Cu at (156.2, 42.0)
- added D3: S3N, InverterCom:DIOM8059X265N, F.Cu at (195.5, 128.4)
- added D4: S3N, InverterCom:DIOM8059X265N, F.Cu at (195.5, 136.2)
- added F1: MF-RHT200_32-2, InverterCom:MFRHT200322, F.Cu at (221.4, 104.2)
- added H2: MountingHole, MountingHole:MountingHole_5.3mm_M5_ISO7380_Pad, F.Cu at (5.50, 39.5)
- added H6: MountingHole, MountingHole:MountingHole_5.3mm_M5_ISO7380_Pad, F.Cu at (180.0, 39.5)
- added J10: Conn_02x03_Counter_Clockwise, Connector_PinHeader_2.54mm:PinHeader_2x03_P2.54mm_Vertical, F.Cu at (54.0, 5.50)
- added J7: Conn_02x08_Counter_Clockwise, Connector_PinHeader_2.54mm:PinHeader_2x08_P2.54mm_Vertical, F.Cu at (206.9, 39.7)
- added PS3: EC7BW-110S12, InverterCom:EC7BW110S12, F.Cu at (158.8, 96.0)
- added R1: 47k, Resistor_SMD:R_1210_3225Metric_Pad1.30x2.65mm_HandSolder, F.Cu at (182.6, 104.3)
- added R2: 10k, Resistor_SMD:R_1210_3225Metric_Pad1.30x2.65mm_HandSolder, F.Cu at (182.6, 108.5)
- added R3: 47k, Resistor_SMD:R_1210_3225Metric_Pad1.30x2.65mm_HandSolder, F.Cu at (182.6, 112.7)
- added R4: 47k, Resistor_SMD:R_1210_3225Metric_Pad1.30x2.65mm_HandSolder, F.Cu at (182.6, 116.9)
- added R6: 47k, Resistor_SMD:R_1210_3225Metric_Pad1.30x2.65mm_HandSolder, F.Cu at (182.6, 125.3)
- added R7: 10k, Resistor_SMD:R_1210_3225Metric_Pad1.30x2.65mm_HandSolder, F.Cu at (182.6, 129.5)
- H1, H7: footprint MountingHole:MountingHole_3.2mm_M3 -> MountingHole:MountingHole_5.3mm_M5_ISO7380_Pad
- H3, H4, H5, H8: footprint MountingHole:MountingHole_4.3mm_M4 -> MountingHole:MountingHole_5.3mm_M5_ISO7380_Pad
- J1: value Conn_02x08_Counter_Clockwise -> TBP01R2W-508-06BE; footprint Connector_PinSocket_2.54mm:PinSocket_2x08_P2.54mm_Vertical -> InverterCom:SHDR6W100P0X508_1X6_4064X850X1240P; moved to F.Cu
- J12: value Conn_02x10_Counter_Clockwise -> Conn_02x08_Counter_Clockwise; footprint Connector_PinHeader_2.54mm:PinHeader_2x10_P2.54mm_Vertical -> Connector_PinHeader_2.54mm:PinHeader_2x08_P2.54mm_Vertical
- J13: value Conn_02x10_Counter_Clockwise -> Conn_02x03_Counter_Clockwise; footprint Connector_PinHeader_2.54mm:PinHeader_2x10_P2.54mm_Vertical -> Connector_PinHeader_2.54mm:PinHeader_2x03_P2.54mm_Vertical
- J14: value Conn_02x10_Counter_Clockwise -> Conn_01x10; footprint Connector_PinHeader_2.54mm:PinHeader_2x10_P2.54mm_Vertical -> Connector_PinHeader_2.54mm:PinHeader_1x10_P2.54mm_Vertical
- J2: value Conn_02x08_Counter_Clockwise -> Conn_01x02; footprint Connector_PinSocket_2.54mm:PinSocket_2x08_P2.54mm_Vertical -> Connector_PinHeader_2.54mm:PinHeader_1x02_P2.54mm_Vertical; moved to F.Cu
- J6: value TBP01R2-508-06BE -> 776231-1; footprint InverterCom:TBP01R250806BE -> InverterCom:7762311; moved to F.Cu
- R5: value 1k -> 47k; moved to F.Cu
- R82: value 1k -> 47k
- moved R82 180.8 mm to (182.6, 133.7), turned to 0 degrees
- moved J12 174.0 mm to (254.7, 13.6), turned to 0 degrees
- moved J6 170.1 mm to (171.8, 72.2), turned to 0 degrees
- moved J1 147.0 mm to (187.9, 97.7), turned to 0 degrees
- moved R5 124.7 mm to (182.6, 121.1), turned to 0 degrees
- moved J2 110.3 mm to (246.5, 39.7), turned to 0 degrees
- moved J13 103.8 mm to (54.0, 43.0), turned to 90 degrees
- moved H4 85.3 mm to (85.0, 39.5)
- moved J14 59.8 mm to (148.6, 42.0), turned to 90 degrees
- moved H8 49.5 mm to (254.5, 39.5)
- moved H1 48.9 mm to (5.50, 5.50)
- moved H7 47.1 mm to (254.5, 5.50)
- moved H3 42.3 mm to (85.0, 5.50)
- moved H5 40.7 mm to (180.0, 5.50)
Connections:
- J1 pad 1: /GND_A -> /GND_Z
- J1 pad 2: /FAULT -> /GND_W
- J1 pad 3: /GND_A -> /CAN2_GND
- J1 pad 4: /READY -> /CAN2_LOW
- J1 pad 5: /GND_A -> /CAN2_HIGH
- J1 pad 6: /RESET -> /CAN2_+5V
- J12 pad 1: /+3.3V_A -> /DIN_1_W
- J12 pad 10: /SPI2_RX_A -> /GND_W
- J12 pad 11: /SPI2_TX_A -> /DIN_6_W
- J12 pad 12: /SPI2_SCK_A -> /GND_W
- J12 pad 13: /SPI2_ADC1_CS_A -> /DIN_7_W
- J12 pad 14: /SPI2_ADC2_CS_A -> /GND_W
- J12 pad 15: unconnected-(J12-Pin_15-Pad15) -> /DIN_8_W
- J12 pad 16: unconnected-(J12-Pin_16-Pad16) -> /GND_W
- J12 pad 2: /GND_A -> /GND_W
- J12 pad 3: /+12V_A -> /DIN_2_W
- J12 pad 4: /+3.3V_A -> /GND_W
- J12 pad 5: /GND_A -> /DIN_3_W
- J12 pad 6: /+12V_A -> /GND_W
- J12 pad 7: /+3.3V_A -> /DIN_4_W
- J12 pad 8: /GND_A -> /GND_W
- J12 pad 9: /+12V_A -> /DIN_5_W
- J13 pad 1: /+3.3V_A -> /CAN2_HIGH
- J13 pad 2: /+12V_A -> /CAN2_JUMPER_B
- J13 pad 3: /GND_A -> /CAN2_+5V
- J13 pad 4: /+3.3V_A -> /CAN2_GND
- J13 pad 5: /+12V_A -> /CAN2_LOW
- J13 pad 6: /GND_A -> /CAN2_HIGH
- J14 pad 1: /CAN_JUMPER_B -> /+3.3V_A
- J14 pad 10: unconnected-(J14-Pin_10-Pad10) -> /RESET
- J14 pad 2: /CAN_HIGH -> /SWDIO
- J14 pad 3: unconnected-(J14-Pin_3-Pad3) -> /GND_A
- J14 pad 4: /CAN_24V_OUT -> /SWCLK
- J14 pad 5: unconnected-(J14-Pin_5-Pad5) -> /GND_A
- J14 pad 6: /CAN_LOW -> /SWO
- J14 pad 7: /CAN_HIGH -> unconnected-(J14-Pin_7-Pad7)
- J14 pad 8: /CAN_GND -> unconnected-(J14-Pin_8-Pad8)
- J14 pad 9: unconnected-(J14-Pin_9-Pad9) -> /GND_A
- J2 pad 1: /GND_A -> /+12V_A
- J2 pad 2: /FAULT -> /GND_A
- J6 pad 1: /GND_U -> /VIN_Z
- J6 pad 2: /PH_W_VSENSE_U -> /CAN_JUMPER_A
- J6 pad 3: /PH_V_VSENSE_U -> unconnected-(J6-Pad3)
- J6 pad 4: /PH_U_VSENSE_U -> unconnected-(J6-Pad4)
- J6 pad 5: /DC_LINK_VSENSE_U -> unconnected-(J6-Pad5)
- J6 pad 6: /GND_U -> /VIN_Z
- R5 pad 2: /+5V_Y -> /VIN_Z
- R82 pad 1: /ADC_1/VoltageSenseInputStage1/LV_OUT -> /GND_Z
- R82 pad 2: /GND_U -> Net-(R1-Pad1)
Routing:
- net /FAULT: track 218.2 -> 0.00 mm, vias 5 -> 0
- net /READY: track 214.5 -> 0.00 mm, vias 5 -> 0
- net /RESET: track 213.2 -> 0.00 mm, vias 4 -> 0
- net /PH_W_L: track 117.1 -> 0.00 mm, vias 2 -> 0
- net /PH_W_H: track 116.4 -> 0.00 mm, vias 2 -> 0
- net /PH_U_L: track 96.2 -> 0.00 mm, vias 2 -> 0
- net /PH_U_H: track 93.5 -> 0.00 mm, vias 2 -> 0
- net /RELAY1_COM: track 68.6 -> 0.00 mm
- net /RELAY3_COM: track 57.8 -> 0.00 mm
- net /RELAY_3_A: track 57.8 -> 0.00 mm, vias 2 -> 0
- net /OutputRelays/+5V_A_INT_2: track 55.3 -> 0.00 mm, vias 2 -> 0
- net /SPI1_SCK_A: track 51.3 -> 0.00 mm, vias 4 -> 0
- net /SPI1_TX_A: track 48.0 -> 0.00 mm, vias 4 -> 0
- net /SPI1_CAN_INT_A: track 47.6 -> 0.00 mm, vias 4 -> 0
- net /SPI1_RX_A: track 47.4 -> 0.00 mm, vias 4 -> 0
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- removed copper zone on In2.Cu, net /+12V_A
- removed copper zone on In3.Cu, net /+3.3V_A
- removed copper zone on In2.Cu, net /+5V_Y
- removed copper zone on In3.Cu, net /CAN_5V_OUT
- removed copper zone on B.Cu, net /CAN_GND
- removed copper zone on F.Cu, net /CAN_GND
- removed copper zone on In1.Cu, net /CAN_GND
- removed copper zone on In4.Cu, net /CAN_GND
- removed copper zone on B.Cu, net /GND_A
- removed copper zone on F.Cu, net /GND_A
- removed copper zone on In1.Cu, net /GND_A
- removed copper zone on In4.Cu, net /GND_A
- removed copper zone on B.Cu, net /GND_U
- removed copper zone on F.Cu, net /GND_U
- removed copper zone on In1.Cu, net /GND_U
- removed copper zone on In2.Cu, net /GND_U
- removed copper zone on In3.Cu, net /GND_U
- removed copper zone on In4.Cu, net /GND_U
- removed copper zone on B.Cu, net /ISENSE_GND_Y
- removed copper zone on F.Cu, net /ISENSE_GND_Y
- removed copper zone on In1.Cu, net /ISENSE_GND_Y
- removed copper zone on In4.Cu, net /ISENSE_GND_Y
Other:
- board size 297.5 x 60 mm -> 260 x 45 mm
- copper layers 6 -> 2
- board text removed: "1->"
- board text removed: "<-1"
- board text removed: "AUX OUTPUT RELAYS"
- board text removed: "C2-MCB-GEN REVISION A"
- board text removed: "CONN. TO PH U GATE DRIVER"
- board text removed: "CONN. TO PH V GATE DRIVER"
- board text removed: "CONN. TO PH W GATE DRIVER"
- board text removed: "DANGER HAZARDOUS VOLTAGES PRESENT REMOVE POWER BEFORE SERVICING"
- board text removed: "DESIGNED BY THOMAS LIAO"
- board text removed: "GND +5V DC U V W"
- board text removed: "GND DC U V W GND"
- board text removed: "ISOLATED CANBUS"
- board text removed: "ISOLATED CURRENT SENSE"
- board text removed: "ISOLATED VOLTAGE SENSE"
- board text removed: "ISOLATION BARRIER DO NOT CROSS"
- board text removed: "SERIAL NUMBER"

Commit message: placement and routing
Parts:
- D3, D4, R1, R2, R3, R4, R5, R6, R7, R82: moved to B.Cu
- moved J1 136.5 mm to (73.0, 24.0), turned to 180 degrees
- moved D3 120.0 mm to (228.6, 13.0), turned to 180 degrees
- moved D4 119.9 mm to (228.6, 21.0), turned to 180 degrees
- moved PS3 114.8 mm to (238.0, 13.0), turned to -90 degrees
- moved R2 110.6 mm to (137.5, 7.50), turned to 180 degrees
- moved R82 109.9 mm to (136.6, 34.0)
- moved R1 109.7 mm to (130.9, 7.50), turned to 180 degrees
- moved R3 109.6 mm to (136.0, 13.4), turned to -90 degrees
- moved R7 105.8 mm to (129.6, 38.0), turned to 180 degrees
- moved R6 105.6 mm to (129.6, 34.0), turned to 180 degrees
- moved R5 105.4 mm to (129.6, 30.0)
- moved F1 99.2 mm to (220.0, 5.00)
- moved R4 98.3 mm to (136.6, 30.0), turned to 180 degrees
- moved J6 82.2 mm to (110.5, 17.5)
Connections:
- PS3 pad 3: /+12V_OUT_A -> /+12V_A
Routing:
- net /GND_W: track 0.00 -> 234.5 mm, vias 0 -> 5
- net /GND_Z: track 0.00 -> 206.1 mm, vias 0 -> 11
- net /GND_A: track 0.00 -> 204.5 mm, vias 0 -> 7
- net /VIN_Z: track 0.00 -> 163.4 mm, vias 0 -> 12
- net /DIN_1_W: track 0.00 -> 147.9 mm, vias 0 -> 4
- net /DIN_2_W: track 0.00 -> 145.3 mm, vias 0 -> 2
- net /+5V_A: track 0.00 -> 106.4 mm, vias 0 -> 5
- net /CAN1_+5V: track 0.00 -> 89.7 mm, vias 0 -> 6
- net /CAN1_HIGH: track 0.00 -> 89.4 mm, vias 0 -> 4
- net /CAN1_LOW: track 0.00 -> 82.3 mm, vias 0 -> 3
- net /MOTOR_TEMP_IN: track 0.00 -> 79.0 mm, vias 0 -> 4
- net Net-(R1-Pad1): track 0.00 -> 74.6 mm, vias 0 -> 2
- net /THROTTLE_A_IN: track 0.00 -> 70.1 mm, vias 0 -> 4
- net /+12V_A: track 0.00 -> 66.3 mm
- net /THROTTLE_B_IN: track 0.00 -> 58.3 mm, vias 0 -> 2
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- added copper zone on B.Cu, net /GND_A
- added copper zone on F.Cu, net /GND_A
Other:
- board text added: "CAN2_5V"
- board text added: "CAN2_GND"
- board text added: "CAN2_H"
- board text added: "CAN2_L"
- board text added: "GND_W"
- board text added: "GND_Z"

Commit message: Update Inverter design for powertrain integration
Parts:
- removed J1: TBP01R2W-508-06BE, InverterCom:SHDR6W100P0X508_1X6_4064X850X1240P
- removed R82: 47k, Resistor_SMD:R_1210_3225Metric_Pad1.30x2.65mm_HandSolder
- added IC10: DRDNB21D-7, InverterCom:SOT65P210X110-6N, B.Cu at (197.0, 32.0)
- added IC11: DRDNB21D-7, InverterCom:SOT65P210X110-6N, F.Cu at (44.5, 37.6)
- added K1: AWHSH105D00G, InverterCom:AWHSH105D00G, F.Cu at (189.8, 17.0)
- added K2: AWHSH105D00G, InverterCom:AWHSH105D00G, F.Cu at (227.3, 30.5)
- added K3: AWHSH105D00G, InverterCom:AWHSH105D00G, F.Cu at (35.7, 29.0)
- added K4: AWHSH105D00G, InverterCom:AWHSH105D00G, F.Cu at (57.7, 29.0)
- added R10: 3550150RJT, InverterCom:RESC11050X120N, B.Cu at (206.0, 7.00)
- added R8: 3550150RJT, InverterCom:RESC11050X120N, B.Cu at (222.0, 7.00)
- added R9: 3550150RJT, InverterCom:RESC11050X120N, B.Cu at (214.0, 7.00)
- D3: moved to F.Cu
- R1, R3, R4, R5, R6: value 47k -> 3550150RJT; footprint Resistor_SMD:R_1210_3225Metric_Pad1.30x2.65mm_HandSolder -> InverterCom:RESC11050X120N
- R2, R7: value 10k -> 3550150RJT; footprint Resistor_SMD:R_1210_3225Metric_Pad1.30x2.65mm_HandSolder -> InverterCom:RESC11050X120N
- moved R6 111.8 mm to (238.0, 7.00), turned to 90 degrees
- moved R5 108.8 mm to (238.0, 21.0), turned to -90 degrees
- moved R7 105.1 mm to (230.0, 7.00), turned to 90 degrees
- moved R4 93.9 mm to (230.0, 21.0), turned to -90 degrees
- moved R3 86.3 mm to (222.0, 21.0)
- moved R2 77.7 mm to (214.0, 21.0), turned to -90 degrees
- moved R1 76.3 mm to (206.0, 21.0), turned to -90 degrees
- moved PS3 39.4 mm to (199.6, 21.6), turned to 90 degrees
- moved D4 39.1 mm to (191.0, 10.0), turned to 0 degrees
- moved D3 37.7 mm to (191.0, 10.0), turned to 0 degrees
- moved F1 31.6 mm to (188.4, 3.00)
- moved J6 3.61 mm to (108.5, 14.5)
Connections:
- F1 pad 1: /VIN_Z -> /I_+VIN_Z
- J10 pad 1: /CAN1_HIGH -> /CAN1_JUMPER_A
- J12 pad 10: /GND_W -> /GND_A
- J12 pad 12: /GND_W -> /GND_A
- J12 pad 14: /GND_W -> /GND_A
- J12 pad 16: /GND_W -> /GND_A
- J12 pad 2: /GND_W -> /GND_A
- J12 pad 4: /GND_W -> /GND_A
- J12 pad 6: /GND_W -> /GND_A
- J12 pad 8: /GND_W -> /GND_A
- J13 pad 1: /CAN2_HIGH -> /CAN2_JUMPER_A
- J14 pad 1: /+3.3V_A -> unconnected-(J14-Pin_1-Pad1)
- J14 pad 10: /RESET -> unconnected-(J14-Pin_10-Pad10)
- J14 pad 2: /SWDIO -> unconnected-(J14-Pin_2-Pad2)
- J14 pad 3: /GND_A -> unconnected-(J14-Pin_3-Pad3)
- J14 pad 4: /SWCLK -> unconnected-(J14-Pin_4-Pad4)
- J14 pad 5: /GND_A -> unconnected-(J14-Pin_5-Pad5)
- J14 pad 6: /SWO -> unconnected-(J14-Pin_6-Pad6)
- J14 pad 9: /GND_A -> unconnected-(J14-Pin_9-Pad9)
- J6 pad 1: /VIN_Z -> /CAN1_GND
- J6 pad 10: unconnected-(J6-Pad10) -> /DIN_2_W
- J6 pad 12: unconnected-(J6-Pad12) -> /I_+VIN_Z
- J6 pad 13: unconnected-(J6-Pad13) -> /CAN1_JUMPER_A
- J6 pad 14: unconnected-(J6-Pad14) -> /CAN1_JUMPER_B
- J6 pad 15: /GND_A -> /CAN2_JUMPER_A
- J6 pad 16: /CAN1_HIGH -> /CAN2_JUMPER_B
- J6 pad 17: unconnected-(J6-Pad17) -> /+12V_SWITCHED_A
- J6 pad 18: /DIGITAL_IN_1 -> /+5V_A
- J6 pad 19: unconnected-(J6-Pad19) -> /I_+5V_HVIL_RETURN_A
- J6 pad 2: /CAN_JUMPER_A -> /CAN1_LOW
- J6 pad 20: unconnected-(J6-Pad20) -> /DIN_1_W
- J6 pad 21: /ENCODER_SIN -> /GND_A
- J6 pad 22: /THROTTLE_A_IN -> unconnected-(J6-Pad22)
- J6 pad 23: /THROTTLE_B_IN -> /O_PRECHARGE_DC_LINK_+_Z
- J6 pad 24: /CAN_JUMPER_B -> /CAN2_GND
- J6 pad 25: unconnected-(J6-Pad25) -> /CAN2_LOW
- J6 pad 26: /+5V_A -> /CAN2_HIGH
- J6 pad 27: /CAN1_LOW -> /CAN2_+5V
- J6 pad 28: /CAN1_+5V -> /MOTOR_TEMP_IN_A
- J6 pad 29: unconnected-(J6-Pad29) -> /HALL_W_IN_A
- J6 pad 3: unconnected-(J6-Pad3) -> /CAN1_HIGH
- J6 pad 30: /DIGITAL_IN_2 -> /HALL_V_ENCODER_COS_IN_A
- J6 pad 31: unconnected-(J6-Pad31) -> /HALL_U_ENCODER_SIN_IN_A
- J6 pad 32: unconnected-(J6-Pad32) -> /+5V_A
- J6 pad 33: /MOTOR_TEMP_IN -> unconnected-(J6-Pad33)
- J6 pad 34: unconnected-(J6-Pad34) -> /O_+VIN_SWITCHED_Z
- J6 pad 35: /ENCODER_COS -> /GND_Z
- J6 pad 4: unconnected-(J6-Pad4) -> /CAN1_+5V
- J6 pad 5: unconnected-(J6-Pad5) -> /CAN1_SWITCHED_+5V
- J6 pad 6: /VIN_Z -> /THROTTLE2_IN_A
- J6 pad 7: unconnected-(J6-Pad7) -> /THROTTLE1_IN_A
- J6 pad 8: unconnected-(J6-Pad8) -> /GND_A
- J6 pad 9: unconnected-(J6-Pad9) -> /+5V_A
- J7 pad 1: /HALL_U_ENCODER_SIN_IN -> /HALL_U_ENCODER_SIN_IN_A
- J7 pad 11: /THROTTLE_B_IN -> /THROTTLE2_IN_A
- J7 pad 13: /GND_A -> /DOUT1_A
- J7 pad 14: /GND_A -> /DOUT2_A
- J7 pad 15: /GND_A -> /DOUT3_A
- J7 pad 16: /+5V_A -> /DOUT4_A
- J7 pad 2: /GND_A -> /+5V_A
- J7 pad 3: /HALL_V_ENCODER_COS_IN -> /HALL_V_ENCODER_COS_IN_A
- J7 pad 5: /HALL_W_IN -> /HALL_W_IN_A
- J7 pad 7: /MOTOR_TEMP_IN -> /MOTOR_TEMP_IN_A
- J7 pad 9: /THROTTLE_A_IN -> /THROTTLE1_IN_A
- R1 pad 1: Net-(R1-Pad1) -> Net-(K1-COM)
- R1 pad 2: /VIN_Z -> Net-(R1-Pad2)
- R2 pad 1: /DIN_1_W -> Net-(R2-Pad1)
- R2 pad 2: Net-(R1-Pad1) -> Net-(R1-Pad2)
- R3 pad 1: Net-(R1-Pad1) -> Net-(R2-Pad1)
- R3 pad 2: /DIGITAL_IN_1 -> Net-(R3-Pad2)
- R4 pad 2: /DIGITAL_IN_2 -> Net-(R3-Pad2)
- R5 pad 2: /VIN_Z -> /O_PRECHARGE_DC_LINK_+_Z
- R6 pad 1: /GND_Z -> Net-(R6-Pad1)
- R6 pad 2: Net-(R4-Pad1) -> /O_PRECHARGE_DC_LINK_+_Z
- R7 pad 1: /DIN_2_W -> Net-(R6-Pad1)
- R7 pad 2: Net-(R4-Pad1) -> Net-(R7-Pad2)
Routing:
- net /GND_W: track 234.5 -> 0.00 mm, vias 5 -> 0
- net /GND_Z: track 206.1 -> 0.00 mm, vias 11 -> 0
- net /GND_A: track 204.5 -> 0.00 mm, vias 7 -> 0
- net /VIN_Z: track 163.4 -> 0.00 mm, vias 12 -> 0
- net /DIN_1_W: track 147.9 -> 0.00 mm, vias 4 -> 0
- net /DIN_2_W: track 145.3 -> 0.00 mm, vias 2 -> 0
- net /+5V_A: track 106.4 -> 0.00 mm, vias 5 -> 0
- net /CAN1_+5V: track 89.7 -> 0.00 mm, vias 6 -> 0
- net /CAN1_HIGH: track 89.4 -> 0.00 mm, vias 4 -> 0
- net /CAN1_LOW: track 82.3 -> 0.00 mm, vias 3 -> 0
- net /MOTOR_TEMP_IN: track 79.0 -> 0.00 mm, vias 4 -> 0
- net Net-(R1-Pad1): track 74.6 -> 0.00 mm, vias 2 -> 0
- net /THROTTLE_A_IN: track 70.1 -> 0.00 mm, vias 4 -> 0
- net /+12V_A: track 66.3 -> 0.00 mm
- net /THROTTLE_B_IN: track 58.3 -> 0.00 mm, vias 2 -> 0
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- removed copper zone on B.Cu, net /GND_A
- removed copper zone on F.Cu, net /GND_A
Other:
- copper layers 2 -> 4
- board text removed: "CAN2_5V"
- board text removed: "CAN2_GND"
- board text removed: "CAN2_H"
- board text removed: "CAN2_L"
- board text removed: "GND_W"
- board text removed: "GND_Z"

Commit message: Added FRAM chip to inverter
Parts:
- removed the ? at (153.7, 42.0)
- removed the ? at (191.7, 39.7)
- removed the ? at (156.2, 42.0)
- added C187: 100nF, Capacitor_SMD:C_1210_3225Metric_Pad1.33x2.70mm_HandSolder, B.Cu at (196.5, 32.1)
- added C188: 100nF, Capacitor_SMD:C_1210_3225Metric_Pad1.33x2.70mm_HandSolder, F.Cu at (47.5, 35.0)
- added C189: 100nF, Capacitor_SMD:C_1210_3225Metric_Pad1.33x2.70mm_HandSolder, F.Cu at (245.5, 30.6)
- IC10: moved to F.Cu
- moved F1 16.0 mm to (172.5, 3.45), turned to -90 degrees
- moved IC11 9.06 mm to (53.0, 34.5), turned to 90 degrees
- moved D3 4.37 mm to (190.0, 5.75), turned to -90 degrees
- moved D4 4.37 mm to (190.0, 5.75), turned to -90 degrees
- moved IC10 3.04 mm to (200.0, 32.5), turned to 0 degrees
- moved K1 1.75 mm to (189.8, 15.2)
- moved R1 1.57 mm to (207.5, 20.6), turned to 90 degrees
- moved R10 1.33 mm to (207.2, 6.55)
- moved R6 1.33 mm to (239.2, 6.55)
- moved R7 1.33 mm to (231.2, 6.55)
- moved R8 1.33 mm to (223.2, 6.55)
- moved R9 1.33 mm to (215.2, 6.55)
- moved R2 1.33 mm to (215.2, 20.6), turned to 90 degrees
- moved R3 1.33 mm to (223.2, 20.6), turned to 90 degrees
- moved R4 1.33 mm to (231.2, 20.6), turned to 90 degrees
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Connections:
- J6 pad 18: /+5V_A -> /CAN1_+5V
Routing:
- net /+5V_A: track 0.00 -> 271.5 mm, vias 0 -> 6
- net /DOUT3_A: track 0.00 -> 148.6 mm, vias 0 -> 4
- net /DOUT4_A: track 0.00 -> 147.6 mm, vias 0 -> 1
- net /I_+5V_HVIL_RETURN_A: track 0.00 -> 120.9 mm, vias 0 -> 2
- net /O_PRECHARGE_DC_LINK_+_Z: track 0.00 -> 115.0 mm, vias 0 -> 2
- net /CAN1_SWITCHED_+5V: track 0.00 -> 103.5 mm, vias 0 -> 2
- net /CAN1_+5V: track 0.00 -> 96.3 mm, vias 0 -> 2
- net /O_+VIN_SWITCHED_Z: track 0.00 -> 95.8 mm
- net /CAN2_JUMPER_A: track 0.00 -> 88.2 mm, vias 0 -> 5
- net /CAN2_JUMPER_B: track 0.00 -> 87.1 mm, vias 0 -> 3
- net /CAN2_+5V: track 0.00 -> 84.3 mm, vias 0 -> 2
- net /CAN1_JUMPER_B: track 0.00 -> 77.1 mm
- net /CAN2_HIGH: track 0.00 -> 71.7 mm, vias 0 -> 1
- net /CAN2_LOW: track 0.00 -> 70.4 mm, vias 0 -> 1
- net /CAN1_HIGH: track 0.00 -> 69.8 mm
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- added copper zone on In2.Cu, net /+12V_A
- added copper zone on B.Cu, net /GND_A
- added copper zone on F.Cu, net /GND_A
- added copper zone on In1.Cu, net /GND_A

Commit message: Finish New control board
Parts:
- removed the ? at (257.3, 18.7)
- added C36: UCM1H101MCL1GS, InverterCom:CAPAE660X800N, F.Cu at (39.5, 39.0)
- added C37: UCM1H101MCL1GS, InverterCom:CAPAE660X800N, F.Cu at (30.5, 39.0)
- added C38: UCM1H101MCL1GS, InverterCom:CAPAE660X800N, F.Cu at (21.5, 39.0)
- added C39: UCM1H101MCL1GS, InverterCom:CAPAE660X800N, F.Cu at (26.5, 28.4)
- added C40: UCM1H101MCL1GS, InverterCom:CAPAE660X800N, F.Cu at (17.3, 28.4)
- added C41: UCM1H101MCL1GS, InverterCom:CAPAE660X800N, F.Cu at (8.00, 28.4)
- added C42: UCM1H101MCL1GS, InverterCom:CAPAE660X800N, F.Cu at (237.5, 32.0)
- added C43: UCM1H101MCL1GS, InverterCom:CAPAE660X800N, F.Cu at (140.7, 41.0)
- added C44: UCM1H101MCL1GS, InverterCom:CAPAE660X800N, F.Cu at (109.7, 41.0)
- added C45: UCM1H101MCL1GS, InverterCom:CAPAE660X800N, F.Cu at (99.5, 41.0)
- added C46: UCM1H101MCL1GS, InverterCom:CAPAE660X800N, F.Cu at (8.00, 18.0)
- added C47: UCM1H101MCL1GS, InverterCom:CAPAE660X800N, F.Cu at (239.5, 40.5)
- added C48: UCM1H101MCL1GS, InverterCom:CAPAE660X800N, F.Cu at (130.5, 41.0)
- added C49: UCM1H101MCL1GS, InverterCom:CAPAE660X800N, F.Cu at (120.0, 41.0)
- added C50: UCM1H101MCL1GS, InverterCom:CAPAE660X800N, F.Cu at (26.5, 17.8)
- added C51: UCM1H101MCL1GS, InverterCom:CAPAE660X800N, F.Cu at (17.5, 17.8)
Routing:
- net /DIN_1_W: track 8.85 -> 150.9 mm, vias 0 -> 4
- net /DIN_2_W: track 12.3 -> 151.6 mm, vias 0 -> 4
- net /THROTTLE2_IN_A: track 12.3 -> 89.9 mm, vias 0 -> 2
- net /THROTTLE1_IN_A: track 12.8 -> 87.6 mm, vias 0 -> 2
- net /HALL_U_ENCODER_SIN_IN_A: track 12.7 -> 81.9 mm, vias 0 -> 2
- net /HALL_V_ENCODER_COS_IN_A: track 18.7 -> 85.0 mm, vias 0 -> 2
- net /HALL_W_IN_A: track 21.2 -> 85.3 mm, vias 0 -> 2
- net /MOTOR_TEMP_IN_A: track 24.3 -> 87.5 mm
- net /+5V_A: track 271.5 -> 330.2 mm
- net /GND_Z: track 49.6 -> 52.0 mm
- net /DOUT2_A: track 18.9 -> 21.3 mm
- net /O_PRECHARGE_DC_LINK_+_Z: track 115.0 -> 116.4 mm
- net /DOUT3_A: track 148.6 -> 149.4 mm
- net /DOUT1_A: track 15.2 -> 15.8 mm
- net /GND_A: track 38.4 -> 38.0 mm, vias 28 -> 54
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Other:
- board text added: "IMPORTANT"
- board text added: "NOT SEVCON COMPATIBLE"
- board text added: "NOTICE: NOT PIN COMPATIBLE WITH SEVCON. DO NOT CONNECT TO SEVCON WIRING HARNESS FAILURE TO COMPLY WILL RESULT IN DAMAGE TO BOTH INVERTER AND CONNECTED DEVICES."

Commit message: forgot
Parts:
- removed R5, R6: 3550150RJT, InverterCom:RESC11050X120N
Connections:
- R4 pad 1: Net-(R4-Pad1) -> /O_PRECHARGE_DC_LINK_+_Z
- R7 pad 1: Net-(R6-Pad1) -> /O_PRECHARGE_DC_LINK_+_Z
Routing:
- net /O_PRECHARGE_DC_LINK_+_Z: track 116.4 -> 103.5 mm
- net Net-(R6-Pad1): track 8.00 -> 0.00 mm
- net Net-(R4-Pad1): track 8.00 -> 0.00 mm

Commit message: Update for fabrication
Other:
- board text added: "<- GND"
- board text added: "<- NC"
- board text added: "<- RESET"
- board text added: "<- SWCLK"
- board text added: "<- SWDIO"
- board text added: "<- SWO"
- board text added: "MODEL: C2-CMB-LV CONNECTOR INPUT BOARD"
- board text added: "SERIAL NUMBER"
Changed lines of the file:
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@@
 		)
+	)
+	(gr_rect
+		(start 62 1.5)
+		(end 72 11.5)
+		(stroke
+			(width 0.1)
+			(type solid)
+		)
+		(fill yes)
+		(layer "F.SilkS")
 	)
 	(gr_poly
@@
 		(layer "F.SilkS")
 		(effects
+			(font
+				(size 1 1)
+				(thickness 0.25)
+				(bold yes)
+			)
+			(justify left bottom)
+		)
+	)
+	(gr_text "MODEL:\nC2-CMB-LV\nCONNECTOR INPUT BOARD"
+		(at 61.5 44 0)
+		(layer "F.SilkS")
+		(effects
+			(font
+				(size 1 1)
+				(thickness 0.25)
+				(bold yes)
+			)
+			(justify left bottom)
+		)
+	)
+	(gr_text "<- SWDIO"
+		(at 151 40 90)
+		(layer "F.SilkS")
+		(effects
+			(font
+				(size 1 1)
+				(thickness 0.25)
+				(bold yes)
+			)
+			(justify left)
+		)
+	)
+	(gr_text "<- GND"
+		(at 153.5 40 90)
+		(layer "F.SilkS")
+		(effects
+			(font
+				(size 1 1)
+				(thickness 0.25)
+				(bold yes)
+			)
+			(justify left)
+		)
+	)
+	(gr_text "<- SWCLK"
+		(at 156 40 90)
+		(layer "F.SilkS")
+		(effects
+			(font
+				(size 1 1)
+				(thickness 0.25)
+				(bold yes)
+			)
+			(justify left)
+		)
+	)
+	(gr_text "<- GND"
+		(at 158.75 40 90)
+		(layer "F.SilkS")
+		(effects
+			(font
+				(size 1 1)
+				(thickness 0.25)
+				(bold yes)
+			)
+			(justify left)
+		)
+	)
+	(gr_text "<- SWO"
+		(at 161.25 40 90)
+		(layer "F.SilkS")
+		(effects
+			(font
+				(size 1 1)
+				(thickness 0.25)
+				(bold yes)
+			)
+			(justify left)
+		)
+	)
+	(gr_text "<- NC"
+		(at 163.75 40 90)
+		(layer "F.SilkS")
+		(effects
+			(font
+				(size 1 1)
+				(thickness 0.25)
+				(bold yes)
+			)
+			(justify left)
+		)
+	)
+	(gr_text "<- NC"
+		(at 166.25 40 90)
+		(layer "F.SilkS")
+		(effects
+			(font
+				(size 1 1)
+				(thickness 0.25)
+				(bold yes)
+			)
+			(justify left)
+		)
+	)
+	(gr_text "<- GND"
+		(at 168.75 40 90)
+		(layer "F.SilkS")
+		(effects
+			(font
+				(size 1 1)
+				(thickness 0.25)
+				(bold yes)
+			)
+			(justify left)
+		)
+	)
+	(gr_text "<- RESET"
+		(at 171.25 40 90)
+		(layer "F.SilkS")
+		(effects
+			(font
+				(size 1 1)
+				(thickness 0.25)
+				(bold yes)
+			)
+			(justify left)
+		)
+	)
+	(gr_text "SERIAL NUMBER"
+		(at 74 13 90)
+		(layer "F.SilkS")
+		(effects
