File: Hardware/Chassis2/Boards/DCBusFilter/DCBusFilter.kicad_pcb (KiCad board)
At the start: 4 copper layers, 89 x 85 mm, 15 parts, among them J1 TBP01R2-508-04BE

Commit message: Powerstage intermediate rework
Parts:
- removed J1: TBP01R2-508-04BE, InverterCom:SHDR4W100P0X508_1X4_2192X850X1200P
- added C12: B58031U9254M062, InverterCom:B58031U9254M062, B.Cu at (39.0, 49.0)
- added C13: B58031U9254M062, InverterCom:B58031U9254M062, F.Cu at (50.0, 49.0)
- added C14: VY1222M47Y5UQ6TV0, InverterCom:VY1222M47Y5UQ6TV0, F.Cu at (108.0, 4.00)
- added C15: VY1222M47Y5UQ6TV0, InverterCom:VY1222M47Y5UQ6TV0, F.Cu at (82.0, 7.10)
- added C16: VY1222M47Y5UQ6TV0, InverterCom:VY1222M47Y5UQ6TV0, F.Cu at (82.0, 1.00)
- added C17: VY1222M47Y5UQ6TV0, InverterCom:VY1222M47Y5UQ6TV0, F.Cu at (172.5, 85.5)
- added C18: VY1222M47Y5UQ6TV0, InverterCom:VY1222M47Y5UQ6TV0, F.Cu at (166.4, 85.5)
- added C19: VY1222M47Y5UQ6TV0, InverterCom:VY1222M47Y5UQ6TV0, F.Cu at (204.0, 4.00)
- added C20: VY1222M47Y5UQ6TV0, InverterCom:VY1222M47Y5UQ6TV0, F.Cu at (198.0, 4.00)
- added C21: B58031U9254M062, InverterCom:B58031U9254M062, B.Cu at (129.0, 49.0)
- added C22: B58031U9254M062, InverterCom:B58031U9254M062, F.Cu at (140.0, 49.0)
- added C23: VY1222M47Y5UQ6TV0, InverterCom:VY1222M47Y5UQ6TV0, F.Cu at (172.0, 7.00)
- added C24: VY1222M47Y5UQ6TV0, InverterCom:VY1222M47Y5UQ6TV0, F.Cu at (172.0, 0.90)
- added C25: VY1222M47Y5UQ6TV0, InverterCom:VY1222M47Y5UQ6TV0, F.Cu at (262.0, 85.5)
- added C26: MKP1848S61010JY5B, InverterCom:MKP1848S61010JY5B, F.Cu at (195.0, 19.0)
- added C27: MKP1848S61010JY5B, InverterCom:MKP1848S61010JY5B, F.Cu at (244.0, 19.0)
- added C28: VY1222M47Y5UQ6TV0, InverterCom:VY1222M47Y5UQ6TV0, F.Cu at (268.0, 85.5)
- added C29: VY1222M47Y5UQ6TV0, InverterCom:VY1222M47Y5UQ6TV0, F.Cu at (280.0, 5.00)
- added C3: B58031U9254M062, InverterCom:B58031U9254M062, B.Cu at (50.0, 49.0)
- added C30: VY1222M47Y5UQ6TV0, InverterCom:VY1222M47Y5UQ6TV0, F.Cu at (274.0, 5.00)
- added C31: B58031U9254M062, InverterCom:B58031U9254M062, B.Cu at (230.0, 49.0)
- added C32: B58031U9254M062, InverterCom:B58031U9254M062, B.Cu at (241.0, 49.0)
- added C33: B58031U9254M062, InverterCom:B58031U9254M062, B.Cu at (219.0, 49.0)
- added C34: B58031U9254M062, InverterCom:B58031U9254M062, F.Cu at (230.0, 49.0)
- added C35: VY1222M47Y5UQ6TV0, InverterCom:VY1222M47Y5UQ6TV0, F.Cu at (262.0, 7.00)
- added C36: VY1222M47Y5UQ6TV0, InverterCom:VY1222M47Y5UQ6TV0, F.Cu at (262.0, 0.90)
- added C4: B58031U9254M062, InverterCom:B58031U9254M062, B.Cu at (61.0, 49.0)
- added H10: MountingHole_Pad, MountingHole:MountingHole_6.4mm_M6_ISO14580_Pad, F.Cu at (275.0, -3.00)
- added H11: MountingHole_Pad, MountingHole:MountingHole_6.4mm_M6_ISO14580_Pad, F.Cu at (230.0, 35.0)
- added H12: MountingHole_Pad, MountingHole:MountingHole_6.4mm_M6_ISO14580_Pad, F.Cu at (230.0, 63.0)
- added H13: MountingHole_Pad, MountingHole:MountingHole_6.4mm_M6_ISO14580_Pad, F.Cu at (6.00, 81.0)
- added H14: MountingHole_Pad, MountingHole:MountingHole_6.4mm_M6_ISO14580_Pad, F.Cu at (185.0, 81.0)
- added H15: MountingHole_Pad, MountingHole:MountingHole_6.4mm_M6_ISO14580_Pad, F.Cu at (285.0, 81.0)
- added H6: MountingHole_Pad, MountingHole:MountingHole_6.4mm_M6_ISO14580_Pad, F.Cu at (185.0, -3.00)
- added H7: MountingHole_Pad, MountingHole:MountingHole_6.4mm_M6_ISO14580_Pad, F.Cu at (140.0, 35.0)
- added H8: MountingHole_Pad, MountingHole:MountingHole_6.4mm_M6_ISO14580_Pad, F.Cu at (140.0, 63.0)
- added H9: MountingHole_Pad, MountingHole:MountingHole_6.4mm_M6_ISO14580_Pad, F.Cu at (230.0, 7.00)
- added J15: 524265-E, InverterCom:524265E, B.Cu at (6.85, 46.6)
- C5, C6: value VY1222M47Y5UQ6TV0 -> MKP1848S61010JY5B; footprint InverterCom:VY1222M47Y5UQ6TV0 -> InverterCom:MKP1848S61010JY5B
- C7, C8: value VY1222M47Y5UQ6TV0 -> B58031U9254M062; footprint InverterCom:VY1222M47Y5UQ6TV0 -> InverterCom:B58031U9254M062; moved to B.Cu
- H4, H5: footprint MountingHole:MountingHole_3.2mm_M3_ISO14580_Pad -> MountingHole:MountingHole_6.4mm_M6_ISO14580_Pad
- moved C8 106.6 mm to (151.0, 49.0)
- moved C6 104.2 mm to (154.0, 19.0), turned to -90 degrees
- moved C11 89.6 mm to (114.0, 4.00)
- moved C10 85.7 mm to (24.0, 85.5), turned to 90 degrees
- moved H4 81.0 mm to (95.0, -3.00)
- moved C7 64.1 mm to (140.0, 49.0), turned to -90 degrees
- moved C2 56.5 mm to (64.0, 19.0), turned to -90 degrees
- moved C1 55.7 mm to (15.0, 19.0), turned to -90 degrees
- moved H5 53.5 mm to (140.0, 7.00)
- moved C9 52.9 mm to (18.0, 85.5), turned to 90 degrees
- moved C5 35.8 mm to (105.0, 19.0)
- moved H1 28.0 mm to (50.0, 35.0)
- moved H2 28.0 mm to (50.0, 63.0)
Connections:
- C10 pad 1: /CHASSIS_GND -> /PH_U_CHASSIS_GND2
- C11 pad 1: /CHASSIS_GND -> /PH_U_CHASSIS_GND
- C11 pad 2: /PHASE_LEG -> /DC_LINK_+
- C5 pad 1: /PHASE_LEG -> /DC_LINK_+
- C5 pad 2: /DC_LINK_+ -> /DC_LINK_-
- C6 pad 1: /DC_LINK_- -> /DC_LINK_+
- C6 pad 2: /PHASE_LEG -> /DC_LINK_-
- C7 pad 1: /CHASSIS_GND_1 -> /DC_LINK_+
- C7 pad 2: /DC_LINK_+ -> /DC_LINK_-
- C8 pad 1: /DC_LINK_- -> /DC_LINK_+
- C8 pad 2: /DC_LINK_+ -> /DC_LINK_-
- C9 pad 1: /DC_LINK_- -> /PH_U_CHASSIS_GND2
- C9 pad 2: /DC_LINK_+ -> /DC_LINK_-
- H3 pad 1: /PHASE_LEG -> /PH_U
- H4 pad 1: /CHASSIS_GND -> /PH_U_CHASSIS_GND
- H5 pad 1: /CHASSIS_GND_1 -> /PH_V
Routing:
- net /PH_W: track 0.00 -> 281.8 mm, vias 0 -> 1
- net /PH_V: track 0.00 -> 174.1 mm, vias 0 -> 1
- net /PHASE_LEG: track 114.5 -> 0.00 mm
- net /PH_U: track 0.00 -> 78.7 mm, vias 0 -> 1
- net /DC_LINK_+: track 126.2 -> 50.9 mm, vias 140 -> 0
- net /DC_LINK_-: track 33.0 -> 58.6 mm, vias 140 -> 0
- net /CHASSIS_GND: track 20.1 -> 0.00 mm
- net /PH_U_CHASSIS_GND2: track 0.00 -> 19.7 mm
- net /CHASSIS_GND_1: track 13.0 -> 0.00 mm
- added copper zone on B.Cu, net /PH_U
- added copper zone on F.Cu, net /PH_U
- added copper zone on In1.Cu, net /PH_U
- added copper zone on In2.Cu, net /PH_U
- added copper zone on B.Cu, net /PH_U_CHASSIS_GND
- added copper zone on F.Cu, net /PH_U_CHASSIS_GND
- added copper zone on In1.Cu, net /PH_U_CHASSIS_GND
- added copper zone on In2.Cu, net /PH_U_CHASSIS_GND
- added copper zone on B.Cu, net /PH_U_CHASSIS_GND2
- added copper zone on F.Cu, net /PH_U_CHASSIS_GND2
- added copper zone on In1.Cu, net /PH_U_CHASSIS_GND2
- added copper zone on In2.Cu, net /PH_U_CHASSIS_GND2
- added copper zone on B.Cu, net /PH_V
- added copper zone on F.Cu, net /PH_V
- added copper zone on In1.Cu, net /PH_V
- added copper zone on In2.Cu, net /PH_V
- added copper zone on B.Cu, net /PH_V_CHASSIS_GND
- added copper zone on F.Cu, net /PH_V_CHASSIS_GND
- added copper zone on In1.Cu, net /PH_V_CHASSIS_GND
- added copper zone on In2.Cu, net /PH_V_CHASSIS_GND
- added copper zone on B.Cu, net /PH_V_CHASSIS_GND2
- added copper zone on F.Cu, net /PH_V_CHASSIS_GND2
- added copper zone on In1.Cu, net /PH_V_CHASSIS_GND2
- added copper zone on In2.Cu, net /PH_V_CHASSIS_GND2
- added copper zone on B.Cu, net /PH_W
- added copper zone on F.Cu, net /PH_W
- added copper zone on In1.Cu, net /PH_W
- added copper zone on In2.Cu, net /PH_W
- added copper zone on B.Cu, net /PH_W_CHASSIS_GND
- added copper zone on F.Cu, net /PH_W_CHASSIS_GND
- added copper zone on In1.Cu, net /PH_W_CHASSIS_GND
- added copper zone on In2.Cu, net /PH_W_CHASSIS_GND
- added copper zone on B.Cu, net /PH_W_CHASSIS_GND2
- added copper zone on F.Cu, net /PH_W_CHASSIS_GND2
- added copper zone on In1.Cu, net /PH_W_CHASSIS_GND2
- added copper zone on In2.Cu, net /PH_W_CHASSIS_GND2
- removed copper zone on B.Cu, net /PHASE_LEG
- removed copper zone on F.Cu, net /PHASE_LEG
- removed copper zone on In1.Cu, net /PHASE_LEG
- removed copper zone on In2.Cu, net /PHASE_LEG
Other:
- board size 89 x 85 mm -> 292 x 96.1 mm
- board text removed: "DANGER HIGH VOLTAGE"
- board text removed: "DANGER: HAZARDOUS VOLTAGES PRESENT"
- board text removed: "DC LINK +"
- board text removed: "DC LINK -"
- board text removed: "DCLB+, NC, PH, DCLB-"
- board text removed: "DESIGNED BY THOMAS LIAO"
- board text removed: "FOR USE WITH 62MM IGBT/SIC HALF-BRIDGE POWER MODULES"
- board text removed: "PART NUMBER: C2-SCB-800"
- board text removed: "PHASE"
- board text removed: "POWER STAGE FILTER FOR CHASSIS SIZE 2 FREQUENCY DRIVES"
- board text removed: "S/N"
- board text removed: "TRACTION INVERTER, GEN 5 POWER STAGE FILTER BOARD, REVISION 1, 800V, 800A"

Commit message: Update IO Board silkscreen, ExM pinout
Connections:
- C1 pad 1: /DC_LINK_+ -> /DC_LINK_-
- C1 pad 2: /DC_LINK_- -> /DC_LINK_+
- C1 pad 3: /DC_LINK_+ -> /DC_LINK_-
- C1 pad 4: /DC_LINK_- -> /DC_LINK_+
- C10 pad 2: /DC_LINK_- -> /DC_LINK_+
- C11 pad 2: /DC_LINK_+ -> /DC_LINK_-
- C12 pad 1: /DC_LINK_+ -> /DC_LINK_-
- C12 pad 2: /DC_LINK_- -> /DC_LINK_+
- C13 pad 1: /DC_LINK_+ -> /DC_LINK_-
- C13 pad 2: /DC_LINK_- -> /DC_LINK_+
- C14 pad 2: /DC_LINK_+ -> /DC_LINK_-
- C17 pad 2: /DC_LINK_- -> /DC_LINK_+
- C18 pad 2: /DC_LINK_- -> /DC_LINK_+
- C19 pad 2: /DC_LINK_+ -> /DC_LINK_-
- C2 pad 1: /DC_LINK_+ -> /DC_LINK_-
- C2 pad 2: /DC_LINK_- -> /DC_LINK_+
- C2 pad 3: /DC_LINK_+ -> /DC_LINK_-
- C2 pad 4: /DC_LINK_- -> /DC_LINK_+
- C20 pad 2: /DC_LINK_+ -> /DC_LINK_-
- C21 pad 1: /DC_LINK_+ -> /DC_LINK_-
- C21 pad 2: /DC_LINK_- -> /DC_LINK_+
- C22 pad 1: /DC_LINK_+ -> /DC_LINK_-
- C22 pad 2: /DC_LINK_- -> /DC_LINK_+
- C25 pad 2: /DC_LINK_- -> /DC_LINK_+
- C26 pad 1: /DC_LINK_+ -> /DC_LINK_-
- C26 pad 2: /DC_LINK_- -> /DC_LINK_+
- C26 pad 3: /DC_LINK_+ -> /DC_LINK_-
- C26 pad 4: /DC_LINK_- -> /DC_LINK_+
- C27 pad 1: /DC_LINK_+ -> /DC_LINK_-
- C27 pad 2: /DC_LINK_- -> /DC_LINK_+
- C27 pad 3: /DC_LINK_+ -> /DC_LINK_-
- C27 pad 4: /DC_LINK_- -> /DC_LINK_+
- C28 pad 2: /DC_LINK_- -> /DC_LINK_+
- C29 pad 2: /DC_LINK_+ -> /DC_LINK_-
- C3 pad 1: /DC_LINK_+ -> /DC_LINK_-
- C3 pad 2: /DC_LINK_- -> /DC_LINK_+
- C30 pad 2: /DC_LINK_+ -> /DC_LINK_-
- C31 pad 1: /DC_LINK_+ -> /DC_LINK_-
- C31 pad 2: /DC_LINK_- -> /DC_LINK_+
- C32 pad 1: /DC_LINK_+ -> /DC_LINK_-
- C32 pad 2: /DC_LINK_- -> /DC_LINK_+
- C33 pad 1: /DC_LINK_+ -> /DC_LINK_-
- C33 pad 2: /DC_LINK_- -> /DC_LINK_+
- C34 pad 1: /DC_LINK_+ -> /DC_LINK_-
- C34 pad 2: /DC_LINK_- -> /DC_LINK_+
- C4 pad 1: /DC_LINK_+ -> /DC_LINK_-
- C4 pad 2: /DC_LINK_- -> /DC_LINK_+
- C5 pad 1: /DC_LINK_+ -> /DC_LINK_-
- C5 pad 2: /DC_LINK_- -> /DC_LINK_+
- C5 pad 3: /DC_LINK_+ -> /DC_LINK_-
- C5 pad 4: /DC_LINK_- -> /DC_LINK_+
- C6 pad 1: /DC_LINK_+ -> /DC_LINK_-
- C6 pad 2: /DC_LINK_- -> /DC_LINK_+
- C6 pad 3: /DC_LINK_+ -> /DC_LINK_-
- C6 pad 4: /DC_LINK_- -> /DC_LINK_+
- C7 pad 1: /DC_LINK_+ -> /DC_LINK_-
- C7 pad 2: /DC_LINK_- -> /DC_LINK_+
- C8 pad 1: /DC_LINK_+ -> /DC_LINK_-
- C8 pad 2: /DC_LINK_- -> /DC_LINK_+
- C9 pad 2: /DC_LINK_- -> /DC_LINK_+
- H1 pad 1: /DC_LINK_+ -> /DC_LINK_-
- H11 pad 1: /DC_LINK_+ -> /DC_LINK_-
- H12 pad 1: /DC_LINK_- -> /DC_LINK_+
- H2 pad 1: /DC_LINK_- -> /DC_LINK_+
- H7 pad 1: /DC_LINK_+ -> /DC_LINK_-
- H8 pad 1: /DC_LINK_- -> /DC_LINK_+
- J15 pad 1: /DC_LINK_+ -> /DC_LINK_-
- J15 pad 5: /DC_LINK_- -> /DC_LINK_+
Routing:
- net /DC_LINK_-: track 58.6 -> 50.9 mm, vias 0 -> 3541
- net /DC_LINK_+: track 50.9 -> 58.6 mm, vias 0 -> 3483
- net /PH_W_CHASSIS_GND2: vias 0 -> 138
- net /PH_W_CHASSIS_GND: vias 0 -> 199
- net /PH_W: vias 1 -> 137
- net /PH_V_CHASSIS_GND2: vias 0 -> 94
- net /PH_V_CHASSIS_GND: vias 0 -> 247
- net /PH_V: vias 1 -> 137
- net /PH_U_CHASSIS_GND2: vias 0 -> 88
- net /PH_U_CHASSIS_GND: vias 0 -> 247
- net /PH_U: vias 1 -> 137
Other:
- board text added: "DANGER: HIGH VOLTAGE ->"
- board text added: "DC LINK + BUS BAR"
- board text added: "DC LINK - BUS BAR"
- board text added: "DC- | PHU | PHV | PHW | DC+ | GND"
- board text added: "HIGH VOLTAGE"
- board text added: "HIGH VOLTAGE CONNECTOR FOR GATE DRIVE, VOLTAGE SENSE"
- board text added: "HIGH VOLTAGE KEEP OUT"
- board text added: "SERIAL NUMBER"
- board text added: "SNUBBER CAPACITOR BOARD REV B | 2026-07 | THOMAS LIAO CORZINE SMART POWER LAB"
- board text added: "U"
- board text added: "V"
- board text added: "W"

Commit message: Update DC Bus Filter Board
Other:
- board text added: "CLASS Y CAPACITORS FOR COMMON-MODE BEARING CURRENT"
Changed lines of the file:
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@@
 		(layer "Edge.Cuts")
+	)
+	(gr_text "CLASS Y CAPACITORS\nFOR COMMON-MODE\nBEARING CURRENT"
+		(at 71 -3 0)
+		(layer "F.SilkS")
+		(effects
+			(font
+				(size 0.85 0.85)
+				(thickness 0.2125)
+				(bold yes)
+			)
+			(justify left bottom)
+		)
+	)
+	(gr_text "CLASS Y CAPACITORS\nFOR COMMON-MODE\nBEARING CURRENT"
+		(at 161 -3 0)
+		(layer "F.SilkS")
+		(effects
+			(font
+				(size 0.85 0.85)
+				(thickness 0.2125)
+				(bold yes)
+			)
+			(justify left bottom)
+		)
+	)
+	(gr_text "CLASS Y CAPACITORS\nFOR COMMON-MODE\nBEARING CURRENT"
+		(at 251 -3 0)
+		(layer "F.SilkS")
+		(effects
+			(font
+				(size 0.85 0.85)
+				(thickness 0.2125)
+				(bold yes)
+			)
+			(justify left bottom)
+		)
 	)
 	(gr_text "SERIAL NUMBER"
