File: Hardware/Chassis2/Boards/DCBusFilter/DCBusFilter.kicad_sch (KiCad schematic)
At the start: 52 parts, among them J15 524265-E

Commit message: Wire harness BOMs from KiCad, board BOM re-exports, tool follows new layouts
- Four harnesses (GDVS, TSIGBT x2, CS x4, TSBCM) with per-chassis Qty
- Board BOMs move to project dirs; discovery prefers root CSV, strips
  library prefixes from footprints, reads KiCad 10 exports
- Mech list down to chassis hardware; IGBT moved to Mouser vendor
- Harness parts leave MechanicalBOM.txt (455-1135-1-ND=SXH-001T-P0.6,
  BC5011CT-ND stray cap, TSW/LA37S600/0022011042/0008500113)
Changed lines of the file:
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@@
 	(text "high voltage connector for gate drive desat, vsense"
 		(exclude_from_sim no)
-		(at 204.216 19.05 0)
+		(at 203.962 26.924 0)
 		(effects
 			(font
@@
 					(unit 1)
 				)
-			)
-		)
-	)
-	(symbol
-		(lib_id "InverterCom:Placeholder")
-		(at 191.77 22.86 0)
-		(unit 1)
-		(body_style 1)
-		(exclude_from_sim no)
-		(in_bom yes)
-		(on_board yes)
-		(in_pos_files yes)
-		(dnp no)
-		(property "Reference" "#JH1"
-			(at 191.008 22.86 0)
-			(show_name no)
-			(do_not_autoplace yes)
-			(effects
-				(font
-					(size 1.27 1.27)
-				)
-				(justify left)
-			)
-		)
-		(property "Value" "544958-E"
-			(at 201.93 22.86 0)
-			(show_name no)
-			(do_not_autoplace no)
-			(effects
-				(font
-					(size 1.27 1.27)
-				)
-			)
-		)
-		(property "Footprint" ""
-			(at 191.77 22.86 0)
-			(hide yes)
-			(show_name no)
-			(do_not_autoplace no)
-			(effects
-				(font
-					(size 1.27 1.27)
-				)
-			)
-		)
-		(property "Datasheet" ""
-			(at 191.77 22.86 0)
-			(hide yes)
-			(show_name no)
-			(do_not_autoplace no)
-			(effects
-				(font
-					(size 1.27 1.27)
-				)
-			)
-		)
-		(property "Description" ""
-			(at 191.77 22.86 0)
-			(hide yes)
-			(show_name no)
-			(do_not_autoplace no)
-			(effects
-				(font
-					(size 1.27 1.27)
-				)
-			)
-		)
-		(instances
-			(project "DCBusFilter"
-				(path "/2365f093-f079-4cf2-9926-0ba7dd4b2726"
-					(reference "#JH1")
-					(unit 1)
-				)

Commit message: Labels tool, composite board views, InverterGen5 C2 branding, even render resolution
- Labels.pdf: HV warning labels, chassis ID, per-assembly labels (label cmd)
- Board sections add composite front/back views (PCB-viewer look, mirrored
  back) and layer plots now carry the drawing sheet with true plot scale
- Branding standardized to InverterGen5 C2 (cover, footer, labels)
- STEP previews render at even resolution regardless of part aspect
- Fab part titles from info.txt PartName; ALL-CAPS handling fixed
Other:
- title: Open Inverter Platform - Filter Board -> InverterGen5 - Filter Board
Changed lines of the file:
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@@
 	(paper "USLetter")
 	(title_block
-		(title "Open Inverter Platform - Filter Board")
+		(title "InverterGen5 - Filter Board")
 		(date "2026-07-16")
 		(rev "A")
