File: Hardware/Chassis2/Wiring/GDVSHarness/GDVSHarness.kicad_sch (KiCad schematic)
At the start: 17 parts, among them J1 524265-E, J15 524265-E, J15-2 524265-E, J2 524265-E, J3 524265-E, T1 FDFNYD1-110(5), T10 FDFNYD1-110(5), T11 FDFNYD1-110(5), T12 FDFNYD1-110(5), T2 FDFNYD1-110(5), T3 FDFNYD1-110(5), T4 FDFNYD1-110(5), T5 FDFNYD1-110(5), T6 FDFNYD1-110(5), T7 FDFNYD1-110(5), T8 FDFNYD1-110(5), T9 FDFNYD1-110(5)

Commit message: Fix internal project references after harness rename, update render
Other:
- title: Open Inverter Platform - Chassis 2 Gate Drive Wiring Harness -> Open Inverter Platform - Gate Drive Wiring Harness
Changed lines of the file:
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@@
 	(paper "USLetter")
 	(title_block
-		(title "Open Inverter Platform - Chassis 2 Gate Drive Wiring Harness")
+		(title "Open Inverter Platform - Gate Drive Wiring Harness")
 		(date "2026-07-16")
 		(rev "A")
 		(company "Corzine Lab, University of California, Santa Cruz")
 		(comment 1 "Prepared by Thomas Liao")
-		(comment 2 "HW-C2-WH-GD-A")
+		(comment 2 "HW-C2-WH-GVDS")
 	)
 	(text "BLK"
@@
 		)
 		(instances
-			(project "HW-C2-WH-GD-A"
+			(project "GDVSHarness"
 				(path "/2365f093-f079-4cf2-9926-0ba7dd4b2726"
 					(reference "J3")
@@
 		)
 		(instances
-			(project "HW-C2-WH-GD-A"
+			(project "GDVSHarness"
 				(path "/2365f093-f079-4cf2-9926-0ba7dd4b2726"
 					(reference "J2")
@@
 		)
 		(instances
-			(project "HW-C2-WH-GD-A"
+			(project "GDVSHarness"
 				(path "/2365f093-f079-4cf2-9926-0ba7dd4b2726"
 					(reference "T12")
@@
 		)
 		(instances
-			(project "HW-C2-WH-GD-A"
+			(project "GDVSHarness"
 				(path "/2365f093-f079-4cf2-9926-0ba7dd4b2726"
 					(reference "T9")
@@
 		)
 		(instances
-			(project "HW-C2-WH-GD-A"
+			(project "GDVSHarness"
 				(path "/2365f093-f079-4cf2-9926-0ba7dd4b2726"
 					(reference "T11")
@@
 		)
 		(instances
-			(project "HW-C2-WH-GD-A"
+			(project "GDVSHarness"
 				(path "/2365f093-f079-4cf2-9926-0ba7dd4b2726"
 					(reference "T7")
@@
 		)
 		(instances
-			(project "HW-C2-WH-GD-A"
+			(project "GDVSHarness"
 				(path "/2365f093-f079-4cf2-9926-0ba7dd4b2726"
 					(reference "T10")
@@
 		)
 		(instances
-			(project "HW-C2-WH-GD-A"
+			(project "GDVSHarness"
 				(path "/2365f093-f079-4cf2-9926-0ba7dd4b2726"
 					(reference "J1")
@@
 		)
 		(instances
-			(project "HW-C2-WH-GD-A"
+			(project "GDVSHarness"
 				(path "/2365f093-f079-4cf2-9926-0ba7dd4b2726"
 					(reference "T8")
@@
 		)
 		(instances
-			(project "HW-C2-WH-GD-A"
+			(project "GDVSHarness"
 				(path "/2365f093-f079-4cf2-9926-0ba7dd4b2726"
 					(reference "J15-2")
@@
 		)
 		(instances
-			(project "HW-C2-WH-GD-A"
+			(project "GDVSHarness"
 				(path "/2365f093-f079-4cf2-9926-0ba7dd4b2726"
 					(reference "J15")
@@
 		)
 		(instances
-			(project "HW-C2-WH-GD-A"
+			(project "GDVSHarness"
 				(path "/2365f093-f079-4cf2-9926-0ba7dd4b2726"
 					(reference "T4")
@@
 		)
 		(instances
-			(project "HW-C2-WH-GD-A"
+			(project "GDVSHarness"
 				(path "/2365f093-f079-4cf2-9926-0ba7dd4b2726"
 					(reference "T1")
@@
 		)
 		(instances
-			(project "HW-C2-WH-GD-A"
+			(project "GDVSHarness"
 				(path "/2365f093-f079-4cf2-9926-0ba7dd4b2726"
 					(reference "T3")
@@
 		)
 		(instances
-			(project "HW-C2-WH-GD-A"
+			(project "GDVSHarness"
 				(path "/2365f093-f079-4cf2-9926-0ba7dd4b2726"
 					(reference "T2")
@@
 		)
 		(instances
-			(project "HW-C2-WH-GD-A"
+			(project "GDVSHarness"
 				(path "/2365f093-f079-4cf2-9926-0ba7dd4b2726"
 					(reference "T6")
@@
 		)
 		(instances
-			(project "HW-C2-WH-GD-A"
+			(project "GDVSHarness"
 				(path "/2365f093-f079-4cf2-9926-0ba7dd4b2726"
 					(reference "T5")

Commit message: Wire harness BOMs from KiCad, board BOM re-exports, tool follows new layouts
- Four harnesses (GDVS, TSIGBT x2, CS x4, TSBCM) with per-chassis Qty
- Board BOMs move to project dirs; discovery prefers root CSV, strips
  library prefixes from footprints, reads KiCad 10 exports
- Mech list down to chassis hardware; IGBT moved to Mouser vendor
- Harness parts leave MechanicalBOM.txt (455-1135-1-ND=SXH-001T-P0.6,
  BC5011CT-ND stray cap, TSW/LA37S600/0022011042/0008500113)
Parts:
- added PIN1, PIN10, PIN11, PIN12, PIN13, PIN14, PIN15, PIN16, PIN17, PIN18, PIN19, PIN2, PIN20, PIN21, PIN22, PIN23, PIN24, PIN25, PIN3, PIN4, PIN5, PIN6, PIN7, PIN8, PIN9: 464762-E, symbol InverterCom:Placeholder
- J1, J15, J15-2, J2, J3: value 524265-E -> 544958-E
Other:
- note added: "PIN CRIMPS FOR CONNECTORS"

Commit message: Update GDVS and current sense harness schematics
Parts:
- J1, J15, J15-2, J2, J3: value 544958-E -> 544959-E
Changed lines of the file:
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@@
 			)
 		)
-		(property "Value" "544958-E"
+		(property "Value" "544959-E"
 			(at 184.15 86.36 0)
 			(show_name no)
@@
 			)
 		)
-		(property "Value" "544958-E"
+		(property "Value" "544959-E"
 			(at 120.65 86.36 0)
 			(show_name no)
@@
 			)
 		)
-		(property "Value" "544958-E"
+		(property "Value" "544959-E"
 			(at 57.15 86.36 0)
 			(show_name no)
@@
 			)
 		)
-		(property "Value" "544958-E"
+		(property "Value" "544959-E"
 			(at 149.86 31.7499 90)
 			(show_name no)
@@
 			)
 		)
-		(property "Value" "544958-E"
+		(property "Value" "544959-E"
 			(at 46.99 35.5599 90)
 			(show_name no)

Commit message: Rename Open Inverter Platform to InverterGen5, schematic PDF export, tidy variants
- Title blocks renamed to InverterGen5 in all harness schematics
- regen now re-exports schematic PDFs for boards and harnesses too
- Spares variants live under FabricationData/BOMs/Variants/
Other:
- title: Open Inverter Platform - Gate Drive Wiring Harness -> InverterGen5 - Gate Drive Wiring Harness
Changed lines of the file:
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@@
 	(paper "USLetter")
 	(title_block
-		(title "Open Inverter Platform - Gate Drive Wiring Harness")
+		(title "InverterGen5 - Gate Drive Wiring Harness")
 		(date "2026-07-16")
 		(rev "A")
