File: Hardware/Chassis2/Wiring/TempSenseHarness/TempSenseHarness.kicad_sch (KiCad schematic)
At the start: 4 parts, among them J1 455-2266-ND

Commit message: Rename Open Inverter Platform to InverterGen5, schematic PDF export, tidy variants
- Title blocks renamed to InverterGen5 in all harness schematics
- regen now re-exports schematic PDFs for boards and harnesses too
- Spares variants live under FabricationData/BOMs/Variants/
Other:
- title: Open Inverter Platform - IGBT Temperature Wiring Harness -> InverterGen5 - IGBT Temperature Wiring Harness
Changed lines of the file:
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@@
 	(paper "USLetter")
 	(title_block
-		(title "Open Inverter Platform - IGBT Temperature Wiring Harness")
+		(title "InverterGen5 - IGBT Temperature Wiring Harness")
 		(date "2026-07-16")
 		(rev "A")
