File: Hardware/SECC/Boards/ControlBoard/CANTransciever.kicad_sch (KiCad schematic)
At the start: 10 parts, among them IC3 ISO1042BDWVR

Commit message: esp32 stuff
Changed lines of the file:
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@@
 	(text "Close Jumper if terminating node\n"
 		(exclude_from_sim no)
-		(at 110.744 26.416 0)
+		(at 110.744 25.4 0)
 		(effects
 			(font
