File: Hardware/SECC/Boards/ControlBoard/CCSModem.kicad_sch (KiCad schematic)
At the start: 16 parts, among them T2 74941502, U6 RED-BEET-E 2.0, U7 TCMT1109

Commit message: layout
Parts:
- D1: footprint PJGBLC03CAU_R1_000A1 -> InverterCom:PJGBLC03CAU_R1_000A1
- D2: footprint PJGBLC12CAU_R1_000A1 -> InverterCom:PJGBLC03CAU_R1_000A1
- T2: footprint Transformer_SMD_Wurth:T_Wurth_WE-PLC_74941502 -> InverterCom:T_Wurth_WE-PLC_74941502
Changed lines of the file:
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@@
 			)
 		)
-		(property "Footprint" "Transformer_SMD_Wurth:T_Wurth_WE-PLC_74941502"
+		(property "Footprint" "InverterCom:T_Wurth_WE-PLC_74941502"
 			(at 114.3 92.71 0)
 			(hide yes)
@@
 			)
 		)
-		(property "Footprint" "PJGBLC03CAU_R1_000A1"
+		(property "Footprint" "InverterCom:PJGBLC03CAU_R1_000A1"
 			(at 204.14 74.93 0)
 			(hide yes)
@@
 			)
 		)
-		(property "Footprint" "PJGBLC12CAU_R1_000A1"
+		(property "Footprint" "InverterCom:PJGBLC03CAU_R1_000A1"
 			(at 169.85 74.93 0)
 			(hide yes)

Commit message: esp32 stuff
Parts:
- C51: value 2.2nF -> 2.2nF,1kV
Connections:
- net GND_A: no longer U6.9 (EPHY_VDD_2P0)
- no-connect marks 4 -> 5
Other:
- note added: "we are not using ethernet mode, so ephy data are nc'd, ephy vdd is nc"
- note removed: "we are not using ethernet mode, so ephy data are nc'd, ephy vdd is tied to gnd"
Changed lines of the file:
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@@
 		(comment 2 "HW-SECC-PCB-CTRL")
 	)
-	(text "we are not using ethernet mode, so ephy data are nc'd,\nephy vdd is tied to gnd"
+	(text "we are not using ethernet mode, so ephy data are nc'd,\nephy vdd is nc"
 		(exclude_from_sim no)
 		(at 188.722 29.21 0)
@@
 	(no_connect
 		(at 212.09 68.58)
+	)
+	(no_connect
+		(at 182.88 44.45)
 	)
 	(no_connect
@@
 			)
 			(justify right)
-		)
-	)
-	(hierarchical_label "GND_A"
-		(shape input)
-		(at 182.88 44.45 90)
-		(effects
-			(font
-				(size 1.27 1.27)
-			)
-			(justify left)
 		)
 	)
@@
 			)
 		)
-		(property "Value" "2.2nF"
+		(property "Value" "2.2nF,1kV"
 			(at 102.87 127 0)
 			(show_name no)
