File: Hardware/SECC/Boards/ControlBoard/ControlBoard.kicad_pcb (KiCad board)
At the start: 8 copper layers, 260 x 45 mm, 239 parts, among them IC1 TPS389006ADJRTER, IC2 MAX22530AWE+, IC3 ISO1042BDWVR, IC4 CY15B102Q-SXET, IC5 ISO1042BDWVR, IC6 ISO1042BDWVR, IC7 ISO1042BDWVR, J1 B2B-XH-AM_LF__SN_, J10 SSW-103-01-L-D, J12 SSW-108-01-L-D, J13 SSW-103-01-L-D, J14 SSW-110-01-F-D, J15 524265-E, J2 TSW-110-21-L-D-LL, J3 22-04-1041, J4 B2B-XH-AM_LF__SN_, J5 B2B-XH-AM_LF__SN_, J6 22-04-1041, J7 SSW-108-01-L-D, J8 22-04-1041, J9 22-04-1041, U1 STM32H723ZGT6, U14 STS41A-AWLB-R3, U2 ISO1212DBQ, U3 LT3080IQ#PBF, U4 ISO1212DBQ, U5 ISO1212DBQ, U6 ISO1212DBQ, U7 BTS462TATMA1, U8 BTS462TATMA1, U9 STM32G474RCT3, Y1 8MHz, Y2 8MHz

Commit message: layout
Parts:
- removed C13, C135, C137, C138, C139, C143, C144, C149, C182, C183, C184, C185, C186, C187, C188, C193, C194, C195, C197, C201, C202, C203, C27, C28: 100nF, Capacitor_SMD:C_1210_3225Metric_Pad1.33x2.70mm_HandSolder
- removed C134, C136, C147, C192, C200: 1uF, Capacitor_SMD:C_1210_3225Metric_Pad1.33x2.70mm_HandSolder
- removed C189, C198, C209, C210: 10uF, Capacitor_SMD:C_1210_3225Metric_Pad1.33x2.70mm_HandSolder
- removed C190, C191: 2.2uF, Capacitor_SMD:C_1210_3225Metric_Pad1.33x2.70mm_HandSolder
- removed C21, C22, C23, C24: 10nF, Capacitor_SMD:C_1210_3225Metric_Pad1.33x2.70mm_HandSolder
- removed C26, C30: 22pF, Capacitor_SMD:C_1210_3225Metric_Pad1.33x2.70mm_HandSolder
- removed H6, H7, H8: 971350581, InverterCom:971350581
- removed IC1: TPS389006ADJRTER, InverterCom:QFN50P300X300X80-17N-D
- removed IC5, IC7: ISO1042BDWVR, InverterCom:SOIC127P1150X280-8N
- removed J10, J13: SSW-103-01-L-D, InverterCom:SSW-103-01-L-D
- removed J12: SSW-108-01-L-D, InverterCom:SSW-108-01-L-D
- removed J14: SSW-110-01-F-D, InverterCom:SSW-110-01-F-D
- removed J15: 524265-E, InverterCom:524265E
- removed J4: B2B-XH-AM_LF__SN_, InverterCom:B2BXHAMLFSN
- removed LED1: LTST-C230CKT, InverterCom:LEDC3216X120N
- removed LED2: LTST-C230GKT, InverterCom:LEDC3216X120N
- removed PS1: RKE-1205S_H, InverterCom:RKE1205SH
- removed R100, R42, R44, R46, R56, R58, R60, R62, R64, R66, R72: 20k, Resistor_SMD:R_1210_3225Metric_Pad1.30x2.65mm_HandSolder
- removed R12, R31: 4.7k, Resistor_SMD:R_1210_3225Metric_Pad1.30x2.65mm_HandSolder
- removed R14, R15, R43, R45, R55, R57, R59, R61, R63, R65, R67, R70, R71, R73, R74, R75, R78, R79, R82, R83, R88, R89, R92, R94, R98, R99: 10k, Resistor_SMD:R_1210_3225Metric_Pad1.30x2.65mm_HandSolder
- removed R68, R69, R76, R77, R80, R81, R84, R85: 560, Resistor_SMD:R_1210_3225Metric_Pad1.30x2.65mm_HandSolder
- removed R93, R95: 1k, Resistor_SMD:R_1210_3225Metric_Pad1.30x2.65mm_HandSolder
- removed S1, S2: TS40-66-50-R-260-SMT-TR, InverterCom:TS406650R260SMTTR
- removed U14: STS41A-AWLB-R3, InverterCom:STS41AAWLBR3
- removed Y1, Y2: 8MHz, Crystal:Crystal_HC49-4H_Vertical
- added C52: 1uF, Capacitor_SMD:C_1210_3225Metric_Pad1.33x2.70mm_HandSolder, B.Cu at (142.9, 145.5)
- added C53: 100nF, Capacitor_SMD:C_1210_3225Metric_Pad1.33x2.70mm_HandSolder, B.Cu at (147.9, 145.5)
- added C54: 100nF, Capacitor_SMD:C_1210_3225Metric_Pad1.33x2.70mm_HandSolder, B.Cu at (152.9, 145.5)
- added C55: 1nF, Capacitor_SMD:C_1210_3225Metric_Pad1.33x2.70mm_HandSolder, B.Cu at (136.9, 145.5)
- added C56: 2.7nF, Capacitor_SMD:C_1210_3225Metric_Pad1.33x2.70mm_HandSolder, F.Cu at (48.2, 117.6)
- added C57: 2.7nF, Capacitor_SMD:C_1210_3225Metric_Pad1.33x2.70mm_HandSolder, F.Cu at (48.1, 123.0)
- added D1: PJGBLC03C-AU_R1_000A1, InverterCom:PJGBLC03CAU_R1_000A1, F.Cu at (43.7, 117.1)
- added D2: PJGBLC12C-AU_R1_000A1, InverterCom:PJGBLC03CAU_R1_000A1, F.Cu at (43.7, 125.0)
- added D9: STTH112A, InverterCom:DIOM5126X265N, B.Cu at (169.5, 132.0)
- added PS3: DPU01M-12, Samacsys:DPU01M12, F.Cu at (20.5, 107.5)
- added R32: 100k, Resistor_SMD:R_1210_3225Metric_Pad1.30x2.65mm_HandSolder, F.Cu at (59.5, 124.2)
- added R33: 24k, Resistor_SMD:R_1210_3225Metric_Pad1.30x2.65mm_HandSolder, F.Cu at (65.5, 118.7)
- added R34: 32k, Resistor_SMD:R_1210_3225Metric_Pad1.30x2.65mm_HandSolder, F.Cu at (65.5, 124.2)
- added T2: 74941502, InverterCom:T_Wurth_WE-PLC_74941502, F.Cu at (52.5, 106.0)
- C10, C18, C19, C20, C29, C35, C36, C37, C39, C9, PS6, R1, R17, R23, R49, R53, R7, R86: moved to B.Cu
- C14, C15, C17, C31, C32, C34, FL1, FL2, R11, R18, R19, R2, R21, R24, R25, R27, R3, R37, R48, R5, R52, R8, R87, R9, R91, U3, Z7: moved to F.Cu
- C33: value 22pF -> 100nF; moved to F.Cu
- C42: value 10nF -> 10uF
- C43, C45, C47: value 10nF -> 100nF
- C44, C46: value 10nF -> 10uF; moved to B.Cu
- C48: value 22pF -> 10uF
- C49: value 10nF -> 100nF; moved to F.Cu
- C50: value 10nF -> 10uF; moved to F.Cu
- C51: value 10nF -> 2.2nF
- IC4: value CY15B102Q-SXET -> NCV57100DWR2G; footprint InverterCom:SOIC127P800X203-8N -> InverterCom:SOIC127P1030X265-16N
- J1: value B2B-XH-AM_LF__SN_ -> TBP02R2W-381-08BE; footprint InverterCom:B2BXHAMLFSN -> InverterCom:TBP02R2W38108BE
- J2: value TSW-110-21-L-D-LL -> TBP02R2W-381-06BE; footprint InverterCom:PinHeader_2x10_P2.54mm_Vertical-31mm -> InverterCom:TBP02R2W38106BE
- J5: value B2B-XH-AM_LF__SN_ -> TBP02R2W-381-06BE; footprint InverterCom:B2BXHAMLFSN -> InverterCom:TBP02R2W38106BE
- J7: value SSW-108-01-L-D -> TBP02R2W-381-06BE; footprint InverterCom:SSW-108-01-L-D -> InverterCom:TBP02R2W38106BE
- J8: value 22-04-1041 -> TBP01R2-508-06BE; footprint InverterCom:SHDR4W64P0X250_1X4_950X580X1210P -> InverterCom:TBP01R250806BE
- J9: value 22-04-1041 -> TBP01R2-508-04BE; footprint InverterCom:SHDR4W64P0X250_1X4_950X580X1210P -> InverterCom:SHDR4W100P0X508_1X4_2192X850X1200P
- R29: value 3k -> 0
- R39: value 10k -> 820k
- R40: value 20k -> 39k
- R41: value 10k -> 100; moved to B.Cu
- U1: value STM32H723ZGT6 -> NUCLEO144-H723ZGx; footprint Package_QFP:LQFP-144_20x20mm_P0.5mm -> Module:ST_Morpho_Connector_144_STLink
- U2, U4, U5: value ISO1212DBQ -> BTS462TATMA1; footprint Package_SO:SSOP-16_3.9x4.9mm_P0.635mm -> Package_TO_SOT_SMD:TO-252-4; moved to B.Cu
- U6: value ISO1212DBQ -> RED-BEET-E 2.0; footprint Package_SO:SSOP-16_3.9x4.9mm_P0.635mm -> InverterCom:RED-BEET-E 2.0
- U7: value BTS462TATMA1 -> TCMT1109; footprint Package_TO_SOT_SMD:TO-252-4 -> Package_SO:SOP-4_4.4x2.6mm_P1.27mm
- U8: value BTS462TATMA1 -> IRM-60-12; footprint Package_TO_SOT_SMD:TO-252-4 -> Converter_ACDC:Converter_ACDC_MeanWell_IRM-60-xx_THT; moved to B.Cu
- U9: value STM32G474RCT3 -> IRM-60-24; footprint Package_QFP:LQFP-64_10x10mm_P0.5mm -> Converter_ACDC:Converter_ACDC_MeanWell_IRM-60-xx_THT; moved to B.Cu
- Z5, Z6: value MM3Z3V0ST1G -> SZMMSZ4678T1G; footprint InverterCom:SOD2512X100N -> InverterCom:SOD3716X135N; moved to F.Cu
- moved U5 220.2 mm to (48.0, 134.0), turned to 90 degrees
- moved U4 219.5 mm to (56.6, 133.0), turned to 90 degrees
- moved C46 213.1 mm to (17.0, 121.5)
- moved C47 209.8 mm to (21.5, 127.5), turned to 0 degrees
- moved C43 209.3 mm to (11.0, 115.9)
- moved U2 208.9 mm to (65.5, 134.0), turned to 90 degrees
- moved C45 205.1 mm to (13.5, 121.5), turned to -90 degrees
- moved C44 201.7 mm to (17.0, 116.0), turned to -90 degrees
- moved C42 193.5 mm to (26.5, 106.5), turned to 180 degrees
- moved J8 188.2 mm to (18.8, 6.50)
- moved C49 188.0 mm to (9.00, 108.0), turned to 90 degrees
- moved H2 187.3 mm to (190.0, 7.50)
- moved C50 186.3 mm to (13.0, 108.0), turned to -90 degrees
- moved U6 185.9 mm to (60.0, 82.5), turned to 90 degrees
- moved Z7 182.1 mm to (41.5, 132.0)
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Connections:
- C208 pad 1: /HS_TMP_1 -> /CABLE_THERMISTOR
- C25 pad 1: /Control/SN_CUR_SENSE_PH_W_REF -> /Main Processor/CURSENS_A_SIG
- C29 pad 1: /Control/SN_CUR_SENSE_PH_W_SIG -> /Main Processor/CURSENS_A_REF
- C33 pad 1: Net-(U9-PF0) -> /GND_A
- C33 pad 2: /GND_A -> /+3.3V_A
- C38 pad 1: /Control/SN_CUR_SENSE_PH_V_REF -> /Main Processor/CURSENS_B_SIG
- C39 pad 1: /Control/SN_CUR_SENSE_PH_V_SIG -> /Main Processor/CURSENS_B_REF
- C42 pad 1: /Control/SN_HALL_W -> /+3.3V_A
- C43 pad 1: /Control/SN_MOTOR_TEMP -> /GND_A
- C43 pad 2: /GND_A -> /Control Pilot Driver/-12V_B
- C44 pad 1: /Control/SN_THROTTLE_A -> /Control Pilot Driver/-12V_B
- C45 pad 1: /Control/SN_THROTTLE_B -> /GND_A
- C45 pad 2: /GND_A -> /Control Pilot Driver/+12V_B
- C46 pad 1: /Control/SN_HALL_U_ENCODER_SIN -> /Control Pilot Driver/+12V_B
- C47 pad 1: /Control/SN_HALL_V_ENCODER_COS -> /Control Pilot Driver/+12V_B
- C47 pad 2: /GND_A -> /Control Pilot Driver/-12V_B
- C48 pad 1: Net-(U9-PF1) -> /Control Pilot Driver/-12V_B
- C48 pad 2: /GND_A -> /Control Pilot Driver/+12V_B
- C49 pad 1: Net-(IC1-MON2) -> /GND_A
- C49 pad 2: /GND_A -> /+12V_A
- C50 pad 1: Net-(IC1-MON5) -> /+12V_A
- C51 pad 1: Net-(IC1-MON4) -> Net-(C51-Pad1)
- C51 pad 2: /GND_A -> Net-(D9-K)
- IC4 pad 1: /Control/Main Processor/FRAM_CS -> /Control Pilot Driver/-12V_B
- IC4 pad 2: /Control/Main Processor/FRAM_SPI_MISO -> /Control Pilot Driver/-12V_B
- IC4 pad 3: /Control/Main Processor/FRAM_WP -> /Control Pilot Driver/-12V_B
- IC4 pad 4: /GND_A -> Net-(IC4-OUTH)
- IC4 pad 5: /Control/Main Processor/FRAM_SPI_MOSI -> /Control Pilot Driver/+12V_B
- IC4 pad 6: /Control/Main Processor/FRAM_SPI_SCK -> Net-(IC4-OUTH)
- IC4 pad 7: /Control/Main Processor/FRAM_HOLD -> Net-(IC4-CLAMP)
- IC4 pad 8: /+3.3V_A -> /Control Pilot Driver/-12V_B
- J1 pad 1: /GND_A -> /CP_PIN
- J1 pad 2: Net-(Z5-K) -> /GND_A
- J2 pad 2: /FAULT -> /+PWM_VBUS
- J2 pad 3: /READY -> /GND_A
- J2 pad 4: /DRIVER_RESET -> /+12V_A
- J2 pad 5: /PH_U_L -> /+CONTACTOR_VBUS
- J2 pad 6: /PH_U_H -> /+24V_A
- J3 pad 1: /Current Sensors/PH_U_CURSENS_REF -> /Current Sensors/CURSENSE_A_REF
- J3 pad 2: /Current Sensors/PH_U_CURSENS -> /Current Sensors/CURSENSE_A
- J5 pad 1: /GND_A -> /CAN2_LOW
- J5 pad 2: Net-(Z7-K) -> /CAN2_HIGH
- J6 pad 1: /Current Sensors/PH_V_CURSENS_REF -> /Current Sensors/CURSENSE_B_REF
- J6 pad 2: /Current Sensors/PH_V_CURSENS -> /Current Sensors/CURSENSE_B
- J7 pad 1: /HALL_U_ENCODER_SIN_IN -> /CAN1_LOW
- J7 pad 2: /+5V_A -> /CAN1_HIGH
- J7 pad 3: /HALL_V_ENCODER_COS_IN -> /CAN1_GND
- J7 pad 4: /GND_A -> /CAN1_+5V
- J7 pad 5: /HALL_W_IN -> /CAN1_HIGH
- J7 pad 6: /GND_A -> /CAN1_JUMPER_B
- J8 pad 1: /Current Sensors/PH_W_CURSENS_REF -> /VS_DC_LINK_Y
- J8 pad 2: /Current Sensors/PH_W_CURSENS -> /VS_PH_U_Y
- J8 pad 3: /GND_A -> /VS_PH_V_Y
- J8 pad 4: /+5V_ISENSE_A -> /VS_PH_W_Y
- J9 pad 1: /Current Sensors/DC_LINK_CURSENS_REF -> /AC_EARTH
- J9 pad 2: /Current Sensors/DC_LINK_CURSENS -> unconnected-(J9-Pad2)
- J9 pad 3: /GND_A -> /AC_LINE2
- J9 pad 4: /+5V_ISENSE_A -> /AC_LINE1
- R29 pad 1: /+12V_A -> Net-(IC4-CLAMP)
- R29 pad 2: Net-(IC1-MON4) -> Net-(IC4-OUTH)
- R30 pad 1: Net-(IC1-MON4) -> Net-(IC4-OUTH)
- R30 pad 2: /GND_A -> /CP_PIN
- R39 pad 1: /Control/SN_CUR_SENSE_PH_U_REF -> /AC_LINE1
- R39 pad 2: /Current Sensors/PH_U_CURSENS_REF -> Net-(C51-Pad1)
- R40 pad 1: /GND_A -> Net-(C53-Pad2)
- R40 pad 2: /Control/SN_CUR_SENSE_PH_U_REF -> Net-(C52-Pad1)
- R41 pad 1: /Control/SN_CUR_SENSE_PH_U_SIG -> Net-(C52-Pad1)
- R41 pad 2: /Current Sensors/PH_U_CURSENS -> /+3.3V_A
- R47 pad 1: /Control/SN_CUR_SENSE_PH_W_REF -> /Main Processor/CURSENS_A_SIG
- R47 pad 2: /Current Sensors/PH_W_CURSENS_REF -> /Current Sensors/CURSENSE_A
- R48 pad 2: /Control/SN_CUR_SENSE_PH_W_REF -> /Main Processor/CURSENS_A_SIG
- R49 pad 1: /Control/SN_CUR_SENSE_PH_W_SIG -> /Main Processor/CURSENS_A_REF
- R49 pad 2: /Current Sensors/PH_W_CURSENS -> /Current Sensors/CURSENSE_A_REF
- R50 pad 2: /Control/SN_CUR_SENSE_PH_W_SIG -> /Main Processor/CURSENS_A_REF
- R51 pad 1: /Control/SN_CUR_SENSE_PH_V_REF -> /Main Processor/CURSENS_B_SIG
- R51 pad 2: /Current Sensors/PH_V_CURSENS_REF -> /Current Sensors/CURSENSE_B
- R52 pad 2: /Control/SN_CUR_SENSE_PH_V_REF -> /Main Processor/CURSENS_B_SIG
- R53 pad 1: /Control/SN_CUR_SENSE_PH_V_SIG -> /Main Processor/CURSENS_B_REF
- R53 pad 2: /Current Sensors/PH_V_CURSENS -> /Current Sensors/CURSENSE_B_REF
- R54 pad 2: /Control/SN_CUR_SENSE_PH_V_SIG -> /Main Processor/CURSENS_B_REF
- R90 pad 1: Net-(Z5-K) -> /CableIO/TEMP_LOGIC_A
- R91 pad 1: /HS_TMP_1 -> /CABLE_THERMISTOR
- R91 pad 2: Net-(Z5-K) -> /CableIO/TEMP_LOGIC_A
- U1 pad 1: /Control/Main Processor/FRAM_SPI_SCK -> unconnected-(U1-PC10-Pad1)
- U1 pad 10: /Control/OBTS_I2C_SDA -> unconnected-(U1-NC-Pad10)
- U1 pad 101: /ADC/SPI_SCK_A -> unconnected-(U1-PB5-Pad101)
- U1 pad 102: unconnected-(U1-PA10-Pad102) -> /CAN Transciever1/A_CAN_TX
- U1 pad 103: /CAN Transciever/A_CAN_RX -> unconnected-(U1-SWO/PB3-Pad103)
- U1 pad 104: /CAN Transciever/A_CAN_TX -> /GND_A
- U1 pad 105: /MP_SWDIO -> unconnected-(U1-USB_ID/PA10-Pad105)
- U1 pad 106: Net-(C191-Pad1) -> unconnected-(U1-ETH_RXD0/PC4-Pad106)
- U1 pad 107: /GND_A -> unconnected-(U1-ETH_MDIO/PA2-Pad107)
- U1 pad 108: /+3.3V_A -> unconnected-(U1-PF5-Pad108)
- U1 pad 109: /MP_SWCLK -> unconnected-(U1-PA3-Pad109)
- U1 pad 11: /Control/OBTS_I2C_SCL -> /CAN Transciever/A_CAN_TX
- U1 pad 111: /GATE_DRIVE_PWR1_ENABLE -> /GND_A
- U1 pad 112: /FAULT -> /Control Pilot Driver/INPUT_-
- U1 pad 113: /READY -> unconnected-(U1-PD13-Pad113)
- U1 pad 114: /MD_FIBER_RX -> unconnected-(U1-PF10-Pad114)
- U1 pad 115: /ADC/ADC1_INT_A -> unconnected-(U1-PD12-Pad115)
- U1 pad 116: /ADC/ADC1_CS_A -> unconnected-(U1-PE7-Pad116)
- U1 pad 117: /GATE_DRIVE_PWR2_FEEDBACK -> unconnected-(U1-PD11-Pad117)
- U1 pad 118: /GATE_DRIVE_PWR1_FEEDBACK -> unconnected-(U1-PD14-Pad118)
- U1 pad 119: /DRIVER_RESET -> unconnected-(U1-PE10-Pad119)
- U1 pad 12: /ONBOARD_12V_ENABLE_A -> unconnected-(U1-IOREF-Pad12)
- U1 pad 120: /GND_A -> unconnected-(U1-PD15-Pad120)
- U1 pad 121: /+3.3V_A -> unconnected-(U1-PE12-Pad121)
- U1 pad 122: /Control/Main Processor/POWERMON_SLEEP -> unconnected-(U1-PF14-Pad122)
- U1 pad 123: /Control/Main Processor/POWERMON_ENABLE -> unconnected-(U1-PE14-Pad123)
- U1 pad 124: unconnected-(U1-PG9-Pad124) -> /Control Pilot Driver/INPUT_+
- U1 pad 125: unconnected-(U1-PG10-Pad125) -> /Main Processor/GATE_DRIVER_FAULT
- U1 pad 126: /DOUT4_A -> /GND_A
- U1 pad 127: /DOUT3_A -> unconnected-(U1-PE13-Pad127)
- U1 pad 128: /DOUT2_A -> unconnected-(U1-PE11-Pad128)
- U1 pad 129: /DOUT1_A -> unconnected-(U1-PF13-Pad129)
- U1 pad 130: /GND_A -> unconnected-(U1-PF3-Pad130)
- U1 pad 131: /+3.3V_A -> /Main Processor/CURSENS_B_REF
- U1 pad 133: /MP_SWO -> unconnected-(U1-PG14-Pad133)
- U1 pad 134: /Control/MP_DEBUG_NJTRST -> /Main Processor/CURSENS_A_SIG
- U1 pad 135: unconnected-(U1-PB5-Pad135) -> /GND_A
- U1 pad 136: /CAN Transciever1/A_CAN_TX -> unconnected-(U1-PE0-Pad136)
- U1 pad 138: /MP_BOOTSEL -> unconnected-(U1-PG8-Pad138)
- U1 pad 14: /Control/SN_MOTOR_TEMP -> unconnected-(U1-~{RST}-Pad14)
- U1 pad 140: /MD_FIBER_TX -> unconnected-(U1-PG5-Pad140)
- U1 pad 142: Net-(U1-PE1) -> unconnected-(U1-PG6/USB_GPIO_OUT-Pad142)
- U1 pad 143: Net-(U1-PDR_ON) -> /GND_A
- U1 pad 144: /+3.3V_A -> /GND_A
- U1 pad 16: /GND_A -> /+3.3V_A
- U1 pad 17: /+3.3V_A -> unconnected-(U1-PA15-Pad17)
- U1 pad 18: /Control/SN_THROTTLE_B -> unconnected-(U1-+5V-Pad18)
- U1 pad 19: unconnected-(U1-PF7-Pad19) -> /GND_A
- U1 pad 2: Net-(U1-PE3) -> unconnected-(U1-PC11-Pad2)
- U1 pad 20: /HS_TMP_1 -> /GND_A
- U1 pad 22: unconnected-(U1-PF10-Pad22) -> /GND_A
- U1 pad 23: Net-(U1-PH0) -> /CableIO/MAIN_CONT_LOGIC_A
- U1 pad 24: Net-(U1-PH1) -> unconnected-(U1-VIN-Pad24)
- U1 pad 25: /MP_RESET -> unconnected-(U1-RTC_CRYSTAL/PC14-Pad25)
- U1 pad 26: /Control/SN_HALL_U_ENCODER_SIN -> unconnected-(U1-NC-Pad26)
- U1 pad 27: /Control/SN_HALL_V_ENCODER_COS -> unconnected-(U1-RTC_CRYSTAL/PC15-Pad27)
- U1 pad 28: /Control/SN_CUR_SENSE_PH_W_REF -> /CableIO/PUMP_PWM_LOGIC_A
- U1 pad 29: /Control/SN_CUR_SENSE_PH_W_SIG -> unconnected-(U1-PH0-Pad29)
- U1 pad 30: /+3.3V_A -> unconnected-(U1-ETH_REF_CLK/PA1-Pad30)
- U1 pad 31: /GND_A -> unconnected-(U1-PH1-Pad31)
- U1 pad 32: /+3.3V_A -> unconnected-(U1-PA4-Pad32)
- U1 pad 34: /HS_TMP_3 -> /CableIO/TEMP_LOGIC_A
- U1 pad 35: /HS_TMP_2 -> /ADC/SPI_MISO_A
- U1 pad 36: /Control/SN_HALL_W -> unconnected-(U1-ETH_MDC/PC1-Pad36)
- U1 pad 37: /Control/SN_THROTTLE_A -> /ADC/SPI_MOSI_A
- U1 pad 38: /GND_A -> unconnected-(U1-PC0-Pad38)
- U1 pad 39: /+3.3V_A -> /CCS Greenphy Modem/RED_BEET_GPIO_2
- U1 pad 4: /Control/Main Processor/FRAM_SPI_MISO -> /CCS Greenphy Modem/RED_BEET_GPIO_0
- U1 pad 40: /Control/PHASE_CURSENSE_COMP_N -> /CCS Greenphy Modem/RED_BEET_GPIO_1
- U1 pad 41: /Control/DC_LINK_CURSENSE_COMP_N -> /CCS Greenphy Modem/RED_BEET_GPIO_3
- U1 pad 42: /Control/SN_CUR_SENSE_PH_V_SIG -> unconnected-(U1-PG2-Pad42)
- U1 pad 43: /Control/SN_CUR_SENSE_PH_V_REF -> unconnected-(U1-PD6-Pad43)
- U1 pad 44: /Control/SN_CUR_SENSE_PH_U_SIG -> unconnected-(U1-PG3-Pad44)
- U1 pad 45: /Control/SN_CUR_SENSE_PH_U_REF -> /CCS Greenphy Modem/SPI_MOSI_A
- U1 pad 46: /Control/SN_CUR_SENSE_PH_W_REF -> /Control Pilot Driver/READY
- U1 pad 47: /Control/SN_CUR_SENSE_PH_W_SIG -> /Control Pilot Driver/RESET
- U1 pad 48: unconnected-(U1-PB2-Pad48) -> /Control Pilot Driver/CP_FEEDBACK
- U1 pad 49: /Control/SN_CUR_SENSE_DC_LINK_SIG -> /GND_A
- U1 pad 5: /Control/Main Processor/FRAM_SPI_MOSI -> /+3.3V_A
- U1 pad 50: /Control/SN_CUR_SENSE_DC_LINK_REF -> /ADC/ADC1_INT_A
- U1 pad 51: /GND_A -> /CableIO/PRECHARGE_CONT_LOGIC_A
- U1 pad 52: /+3.3V_A -> /ADC/ADC1_CS_A
- U1 pad 53: /Control/SN_CUR_SENSE_PH_W_SIG -> /CCS Greenphy Modem/SPI_CS_A
- U1 pad 54: /Control/SN_CUR_SENSE_PH_W_REF -> unconnected-(U1-PF8-Pad54)
- U1 pad 55: /Control/Main Processor/VOLTAGE_MONITOR_I2C_SDA -> /CCS Greenphy Modem/SPI_INT_A
- U1 pad 57: unconnected-(U1-PG1-Pad57) -> /CCS Greenphy Modem/RESET_A
- U1 pad 58: /MD_FIBER_SYNC -> unconnected-(U1-PG1-Pad58)
- U1 pad 59: /PH_U_H -> unconnected-(U1-PG0-Pad59)
- U1 pad 6: /+3.3V_A -> unconnected-(U1-E5V-Pad6)
- U1 pad 60: /PH_U_L -> /GND_A
- U1 pad 61: /GND_A -> unconnected-(U1-PE1-Pad61)
- U1 pad 62: /+3.3V_A -> unconnected-(U1-PE6-Pad62)
- U1 pad 63: /PH_V_H -> /CCS Greenphy Modem/SPI_MISO_A
- U1 pad 64: /PH_V_L -> unconnected-(U1-PG15-Pad64)
- U1 pad 65: /PH_W_H -> unconnected-(U1-PG12-Pad65)
- U1 pad 66: /PH_W_L -> unconnected-(U1-PG10-Pad66)
- U1 pad 68: /FAULT -> unconnected-(U1-PG13/ETH_TXD0-Pad68)
- U1 pad 69: /Control/Main Processor/USART3_TX -> unconnected-(U1-STLINK_RX/PD9-Pad69)
- U1 pad 7: /Control/Main Processor/FRAM_WP -> unconnected-(U1-~{BOOT0}-Pad7)
- U1 pad 70: /Control/Main Processor/USART3_RX -> unconnected-(U1-PG11/ETH_TX_EN-Pad70)
- U1 pad 71: Net-(C190-Pad1) -> /GND_A
- U1 pad 72: /+3.3V_A -> /GND_A
- U1 pad 73: /CAN Transciever1/A_CAN_RX -> unconnected-(U1-PC9-Pad73)
- U1 pad 75: /ADC/SPI_MISO_A -> unconnected-(U1-PB8-Pad75)
- U1 pad 76: /ADC/SPI_MOSI_A -> unconnected-(U1-PC6-Pad76)
- U1 pad 77: /Control/Main Processor/COPROCESSOR_SYNC -> unconnected-(U1-PB9-Pad77)
- U1 pad 78: /Control/Main Processor/COPROCESSOR_WAKEUP -> unconnected-(U1-ETH_RXD1/PC5-Pad78)
- U1 pad 79: /CP_RESET -> /+3.3V_A
- U1 pad 8: /Control/Main Processor/FRAM_CS -> /GND_A
- U1 pad 80: /CP_BOOTSEL -> unconnected-(U1-U5V-Pad80)
- U1 pad 81: /Control/Main Processor/VOLTAGE_MONITOR_I2C_SCL -> /GND_A
- U1 pad 83: /GND_A -> /CCS Greenphy Modem/SPI_SCK_A
- U1 pad 84: /+3.3V_A -> unconnected-(U1-USB_DP/PA12-Pad84)
- U1 pad 85: unconnected-(U1-PD14-Pad85) -> /Main Processor/CURSENS_A_REF
- U1 pad 86: /Control/MP_USER_DIN_6 -> unconnected-(U1-USB_DM/PA11-Pad86)
- U1 pad 87: /Control/MP_USER_DIN_5 -> unconnected-(U1-ETH_CRS_DV/PA7-Pad87)
- U1 pad 88: /Control/SN_USER_DIN_4 -> /CAN Transciever1/A_CAN_RX
- U1 pad 89: /Control/SN_USER_DIN_3 -> unconnected-(U1-PB6-Pad89)
- U1 pad 9: /Control/Main Processor/FRAM_HOLD -> /CAN Transciever/A_CAN_RX
- U1 pad 90: /Control/SN_USER_DIN_2 -> unconnected-(U1-PB11-Pad90)
- U1 pad 91: /Control/SN_USER_DIN_1 -> unconnected-(U1-PC7-Pad91)
- U1 pad 92: /Control/MP_USER_DIN_7 -> /GND_A
- U1 pad 93: /Control/MP_USER_DIN_8 -> /ADC/SPI_SCK_A
- U1 pad 94: /GND_A -> unconnected-(U1-PB2-Pad94)
- U1 pad 95: /+3.3V_A -> unconnected-(U1-USB_SOF/PA8-Pad95)
- U1 pad 96: /Control/Main Processor/COPROCESSOR_TIMER_SYNC_OUT -> /Main Processor/CURSENS_B_SIG
- U1 pad 97: /Control/MP_DEBUG_TRGIO -> unconnected-(U1-PB10-Pad97)
- U1 pad 98: /CANBUS_ENABLE_12V_A -> unconnected-(U1-PB15-Pad98)
- U2 pad 2: /+3.3V_A -> /CableIO/MAIN_CONT_LOGIC_A
- U2 pad 3: /+3.3V_A -> /+CONTACTOR_VBUS
- U2 pad 4: /Control/SN_USER_DIN_3 -> unconnected-(U2-NC-Pad4)
- U2 pad 5: /Control/SN_USER_DIN_4 -> /MAIN_CONTACTOR_OUT
- U4 pad 2: /+3.3V_A -> /CableIO/PRECHARGE_CONT_LOGIC_A
- U4 pad 3: /+3.3V_A -> /+CONTACTOR_VBUS
- U4 pad 4: /Control/SN_USER_DIN_1 -> unconnected-(U4-NC-Pad4)
- U4 pad 5: /Control/SN_USER_DIN_2 -> /PRECHARGE_CONTACTOR_OUT
- U5 pad 2: /+3.3V_A -> /CableIO/PUMP_PWM_LOGIC_A
- U5 pad 3: /+3.3V_A -> /+PWM_VBUS
- U5 pad 4: /Control/MP_USER_DIN_5 -> unconnected-(U5-NC-Pad4)
- U5 pad 5: /Control/MP_USER_DIN_6 -> /PUMP_PWM_OUT
- U6 pad 10: Net-(U6-IN2) -> /GND_A
- U6 pad 11: Net-(U6-SENSE2) -> unconnected-(U6-EPHY_TX_N-Pad11)
- U6 pad 14: /GND_W -> unconnected-(U6-EPHY_RX_P-Pad14)
- U6 pad 15: Net-(U6-IN1) -> /GND_A
- U6 pad 16: Net-(U6-SENSE1) -> /CCS Greenphy Modem/RED_BEET_GPIO_0
- U6 pad 2: /+3.3V_A -> /GND_A
- U6 pad 3: /+3.3V_A -> /GND_A
- U6 pad 4: /Control/MP_USER_DIN_7 -> /CCS Greenphy Modem/ZC_IN
- U6 pad 5: /Control/MP_USER_DIN_8 -> /GND_A
- U6 pad 6: unconnected-(U6-NC-Pad6) -> /GND_A
- U6 pad 7: unconnected-(U6-NC-Pad7) -> /GND_A
- U6 pad 8: /GND_A -> /+3.3V_A
- U6 pad 9: /GND_W -> /GND_A
- U7 pad 1: /GND_A -> Net-(D9-K)
- U7 pad 2: /ONBOARD_12V_ENABLE_A -> /AC_LINE2
- U7 pad 3: /+12V_A -> /GND_A
- U7 pad 4: unconnected-(U7-NC-Pad4) -> Net-(C53-Pad2)
- U8 pad 1: /GND_A -> /AC_LINE1
- U8 pad 2: /CANBUS_ENABLE_12V_A -> /AC_LINE2
- U8 pad 4: unconnected-(U8-NC-Pad4) -> /GND_A
- U9 pad 1: /+3.3V_A -> /AC_LINE1
- U9 pad 2: /Control/Main Processor/COPROCESSOR_WAKEUP -> /AC_LINE2
- U9 pad 3: /GATE_DRIVE_PWR1_FEEDBACK -> /+24V_A
- U9 pad 4: /GATE_DRIVE_PWR2_FEEDBACK -> /GND_A
- Z5 pad 1: Net-(Z5-K) -> /Control Pilot Driver/CP_FEEDBACK
- Z5 pad 2: /GND_A -> Net-(Z5-A)
- Z6 pad 1: Net-(Z6-K) -> Net-(Z5-A)
- Z7 pad 1: Net-(Z7-K) -> /CableIO/TEMP_LOGIC_A
Routing:
- net /GND_A: track 224.3 -> 0.00 mm, vias 127 -> 0
- net /AC_LINE1: track 0.00 -> 174.3 mm
- net /DRIVER_RESET: track 171.2 -> 0.00 mm, vias 7 -> 0
- net /AC_LINE2: track 0.00 -> 163.4 mm, vias 0 -> 1
- net /GATE_DRIVE_PWR1_FEEDBACK: track 161.4 -> 0.00 mm, vias 8 -> 0
- net /GATE_DRIVE_PWR2_FEEDBACK: track 159.5 -> 0.00 mm, vias 10 -> 0
- net /Control/SN_CUR_SENSE_PH_W_REF: track 151.2 -> 0.00 mm, vias 10 -> 0
- net /Control/SN_CUR_SENSE_PH_U_REF: track 149.6 -> 0.00 mm, vias 8 -> 0
- net /Control/SN_CUR_SENSE_PH_U_SIG: track 148.3 -> 0.00 mm, vias 7 -> 0
- net /Control/SN_CUR_SENSE_PH_W_SIG: track 147.4 -> 0.00 mm, vias 10 -> 0
- net /Control/SN_CUR_SENSE_PH_V_SIG: track 138.7 -> 0.00 mm, vias 7 -> 0
- net /ONBOARD_12V_ENABLE_A: track 134.1 -> 0.00 mm, vias 3 -> 0
- net /Control/SN_CUR_SENSE_PH_V_REF: track 133.0 -> 0.00 mm, vias 6 -> 0
- net /Control/SN_HALL_U_ENCODER_SIN: track 132.4 -> 0.00 mm, vias 6 -> 0
- net /Control/SN_USER_DIN_3: track 129.1 -> 0.00 mm, vias 6 -> 0
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- removed copper zone on In4.Cu, net /+12V_A
- removed copper zone on In4.Cu, net /+12V_CANBUS_A
- removed copper zone on In4.Cu, net /+12V_SWITCHED_A
- removed copper zone on In3.Cu, net /+3.3V_A
- removed copper zone on In4.Cu, net /+5V_ISENSE_A
- removed copper zone on In2.Cu, net /CAN1_+5V
- removed copper zone on B.Cu, net /CAN1_GND
- removed copper zone on F.Cu, net /CAN1_GND
- removed copper zone on In1.Cu, net /CAN1_GND
- removed copper zone on In3.Cu, net /CAN1_GND
- removed copper zone on In4.Cu, net /CAN1_GND
- removed copper zone on In2.Cu, net /CAN2_+5V
- removed copper zone on B.Cu, net /CAN2_GND
- removed copper zone on F.Cu, net /CAN2_GND
- removed copper zone on In1.Cu, net /CAN2_GND
- removed copper zone on In3.Cu, net /CAN2_GND
- removed copper zone on In4.Cu, net /CAN2_GND
- removed copper zone on B.Cu, net /GND_A
- removed copper zone on F.Cu, net /GND_A
- removed copper zone on In1.Cu, net /GND_A
- removed copper zone on In2.Cu, net /GND_A
- removed copper zone on In4.Cu, net /GND_A
- removed copper zone on In5.Cu, net /GND_A
- removed copper zone on In6.Cu, net /GND_A
- removed copper zone on B.Cu, net /GND_W
- removed copper zone on F.Cu, net /GND_W
- removed copper zone on In1.Cu, net /GND_W
- removed copper zone on In2.Cu, net /GND_W
- removed copper zone on In3.Cu, net /GND_W
- removed copper zone on In4.Cu, net /GND_W
- removed copper zone on In5.Cu, net /GND_W
- removed copper zone on In6.Cu, net /GND_W
- removed copper zone on B.Cu, net /VS_GND_Y
- removed copper zone on F.Cu, net /VS_GND_Y
- removed copper zone on In1.Cu, net /VS_GND_Y
- removed copper zone on In2.Cu, net /VS_GND_Y
- removed copper zone on In3.Cu, net /VS_GND_Y
- removed copper zone on In4.Cu, net /VS_GND_Y
Other:
- board size 260 x 45 mm -> 197.5 x 150 mm
- copper layers 8 -> 6
- board text removed: "1->"
- board text removed: "256KB FRAM ->"
- board text removed: "<-1"
- board text removed: "BOOTSEL"
- board text removed: "CAUTION! MAX VOLTAGE: 1200V"
- board text removed: "CURRENT SENSOR CONNECTORS"
- board text removed: "DC LINK"
- board text removed: "DEBUG/FIBER MULTIDRIVE/USB"
- board text removed: "GATE DRIVE/GD POWER CONTROL"
- board text removed: "INVERTER CONTROL BOARD REV. A | 2026-07 | THOMAS LIAO CORZINE SMART POWER LAB, UCSC"
- board text removed: "ISOLATED CAN1 <-"
- board text removed: "ISOLATED CAN2 <-"
- board text removed: "ISOLATED USER DIGITAL INPUTS"
- board text removed: "ISOLATED VOLTAGE SENSE"
- board text removed: "MAIN PROCESSOR"
- board text removed: "NOTE: WILL RESET BOTH PROCESSORS"
- board text removed: "ONBOARD TEMP SENSE"
- board text removed: "P/N: HW-C2-PCB-CTRL-A"
- board text removed: "PH U"
- board text removed: "PH V"
- board text removed: "PH W"
- board text removed: "PHASE U"
- board text removed: "PHASE V"
- board text removed: "PHASE W"
- board text removed: "POWER RAIL MONITORING"
- board text removed: "RESET"
- board text removed: "SAFETY COPROCESSOR"
- board text removed: "SERIAL NUMBER"
- board text removed: "SWITCHING ELEMENT TEMPERATURE SENSORS"
- board text removed: "TEMP 1"
- board text removed: "TEMP 2"
- board text removed: "TEMP 3"
- board text removed: "USER ANALOG INPUTS"
- board text removed: "VOLTAGE SENSE CONNECTOR GND | GND | W | V | U | DC LINK"
- board text removed: "VSENSE CIRCUIT MUST BE CONFORMAL COATED"

Commit message: esp32 stuff
Parts:
- added C58: 10nF, Capacitor_SMD:C_1210_3225Metric_Pad1.33x2.70mm_HandSolder, F.Cu at (67.9, 105.0)
- moved TP6 15.1 mm to (40.0, 29.5)
- moved TP3 10.0 mm to (12.5, 30.0)
- moved TP5 6.95 mm to (12.5, 40.0)
- moved TP4 3.61 mm to (40.0, 34.5)
- moved C32 3.50 mm to (65.0, 38.0), turned to 180 degrees
- moved C15 2.98 mm to (39.5, 75.8), turned to 0 degrees
- moved C31 2.66 mm to (75.0, 43.2)
- moved TP1 1.58 mm to (12.5, 35.0)
Connections:
- C14 pad 1: /+12V_CANBUS_A -> /+12V_A
- C14 pad 2: /GND_A -> /AC_EARTH
- C140 pad 2: /GND_A -> /AC_EARTH
- C141 pad 1: /+12V_SWITCHED_A -> /+12V_A
- C141 pad 2: /GND_A -> /AC_EARTH
- C142 pad 1: /GND_A -> /AC_EARTH
- C145 pad 2: /GND_A -> /AC_EARTH
- C146 pad 2: /GND_A -> /AC_EARTH
- C15 pad 2: /GND_A -> /AC_EARTH
- C208 pad 2: /GND_A -> /AC_EARTH
- C25 pad 2: /GND_A -> /AC_EARTH
- C29 pad 2: /GND_A -> /AC_EARTH
- C31 pad 1: /+12V_CANBUS_A -> /+12V_A
- C31 pad 2: /GND_A -> /AC_EARTH
- C32 pad 2: /GND_A -> /AC_EARTH
- C33 pad 1: /GND_A -> /AC_EARTH
- C38 pad 2: /GND_A -> /AC_EARTH
- C39 pad 2: /GND_A -> /AC_EARTH
- C40 pad 1: /GND_A -> /AC_EARTH
- C41 pad 1: /GND_A -> /AC_EARTH
- C42 pad 2: /GND_A -> /AC_EARTH
- C43 pad 1: /GND_A -> /AC_EARTH
- C44 pad 2: /GND_A -> /AC_EARTH
- C45 pad 1: /GND_A -> /AC_EARTH
- C46 pad 2: /GND_A -> /AC_EARTH
- C49 pad 1: /GND_A -> /AC_EARTH
- C50 pad 2: /GND_A -> /AC_EARTH
- C52 pad 2: /GND_A -> /AC_EARTH
- C53 pad 1: /GND_A -> /AC_EARTH
- C54 pad 1: /GND_A -> /AC_EARTH
- D1 pad 1: /GND_A -> /AC_EARTH
- D2 pad 1: /GND_A -> /AC_EARTH
- IC2 pad 9: /GND_A -> /AC_EARTH
- IC3 pad 4: /GND_A -> /AC_EARTH
- IC4 pad 16: /GND_A -> /AC_EARTH
- IC4 pad 9: /GND_A -> /AC_EARTH
- IC6 pad 4: /GND_A -> /AC_EARTH
- J1 pad 2: /GND_A -> /AC_EARTH
- J1 pad 4: /GND_A -> /AC_EARTH
- J1 pad 8: /GND_A -> /AC_EARTH
- J2 pad 1: /GND_A -> /AC_EARTH
- J2 pad 3: /GND_A -> /AC_EARTH
- J3 pad 3: /GND_A -> /AC_EARTH
- J6 pad 3: /GND_A -> /AC_EARTH
- PS2 pad 1: /+12V_CANBUS_A -> /+12V_A
- PS2 pad 2: /GND_A -> /AC_EARTH
- PS3 pad 2: /GND_A -> /AC_EARTH
- PS3 pad 5: /GND_A -> /AC_EARTH
- PS4 pad 1: /+12V_CANBUS_A -> /+12V_A
- PS4 pad 2: /GND_A -> /AC_EARTH
- PS6 pad 1: /GND_A -> /AC_EARTH
- PS6 pad 7: /GND_A -> /AC_EARTH
- R32 pad 2: unconnected-(R32-Pad2) -> /CP_PIN
- R34 pad 1: /GND_A -> /AC_EARTH
- R48 pad 1: /GND_A -> /AC_EARTH
- R50 pad 1: /GND_A -> /AC_EARTH
- R52 pad 1: /GND_A -> /AC_EARTH
- R54 pad 1: /GND_A -> /AC_EARTH
- R86 pad 1: /GND_A -> /AC_EARTH
- R87 pad 1: /GND_A -> /AC_EARTH
- T2 pad 8: /GND_A -> /AC_EARTH
- U1 pad 104: /GND_A -> /AC_EARTH
- U1 pad 111: /GND_A -> /AC_EARTH
- U1 pad 125: /Main Processor/GATE_DRIVER_FAULT -> /Control Pilot Driver/FAULT
- U1 pad 126: /GND_A -> /AC_EARTH
- U1 pad 129: unconnected-(U1-PF13-Pad129) -> /Control Pilot Driver/CP_FEEDBACK
- U1 pad 135: /GND_A -> /AC_EARTH
- U1 pad 143: /GND_A -> /AC_EARTH
- U1 pad 144: /GND_A -> /AC_EARTH
- U1 pad 19: /GND_A -> /AC_EARTH
- U1 pad 20: /GND_A -> /AC_EARTH
- U1 pad 22: /GND_A -> /AC_EARTH
- U1 pad 48: /Control Pilot Driver/CP_FEEDBACK -> unconnected-(U1-PE4-Pad48)
- U1 pad 49: /GND_A -> /AC_EARTH
- U1 pad 60: /GND_A -> /AC_EARTH
- U1 pad 71: /GND_A -> /AC_EARTH
- U1 pad 72: /GND_A -> /AC_EARTH
- U1 pad 8: /GND_A -> /AC_EARTH
- U1 pad 81: /GND_A -> /AC_EARTH
- U1 pad 84: unconnected-(U1-USB_DP/PA12-Pad84) -> /Main Processor/FDCAN1_TX
- U1 pad 86: unconnected-(U1-USB_DM/PA11-Pad86) -> /Main Processor/FDCAN1_RX
- U1 pad 92: /GND_A -> /AC_EARTH
- U2 pad 1: /GND_A -> /AC_EARTH
- U3 pad 4: /+12V_SWITCHED_A -> /+12V_A
- U3 pad 5: /+12V_SWITCHED_A -> /+12V_A
- U4 pad 1: /GND_A -> /AC_EARTH
- U5 pad 1: /GND_A -> /AC_EARTH
- U6 pad 1: /GND_A -> /AC_EARTH
- U6 pad 10: /GND_A -> /AC_EARTH
- U6 pad 15: /GND_A -> /AC_EARTH
- U6 pad 2: /GND_A -> /AC_EARTH
- U6 pad 21: /GND_A -> /AC_EARTH
- U6 pad 22: /GND_A -> /AC_EARTH
- U6 pad 28: /GND_A -> /AC_EARTH
- U6 pad 29: /GND_A -> /AC_EARTH
- U6 pad 3: /GND_A -> /AC_EARTH
- U6 pad 30: /GND_A -> /AC_EARTH
- U6 pad 31: /GND_A -> /AC_EARTH
- U6 pad 32: /GND_A -> /AC_EARTH
- U6 pad 35: /GND_A -> /AC_EARTH
- U6 pad 38: /GND_A -> /AC_EARTH
- U6 pad 39: /GND_A -> /AC_EARTH
- U6 pad 40: /GND_A -> /AC_EARTH
- U6 pad 5: /GND_A -> /AC_EARTH
- U6 pad 6: /GND_A -> /AC_EARTH
- U6 pad 7: /GND_A -> /AC_EARTH
- U6 pad 9: /GND_A -> unconnected-(U6-EPHY_VDD_2P0-Pad9)
- U7 pad 3: /GND_A -> /AC_EARTH
- U8 pad 4: /GND_A -> /AC_EARTH
- U9 pad 4: /GND_A -> /AC_EARTH
- Z6 pad 2: /GND_A -> /AC_EARTH
- Z7 pad 2: /GND_A -> /AC_EARTH
Routing:
- net /Control Pilot Driver/INPUT_-: track 0.00 -> 135.6 mm, vias 0 -> 4
- net /Control Pilot Driver/FAULT: track 0.00 -> 134.4 mm, vias 0 -> 4
- net /CAN Transciever1/A_CAN_TX: track 0.00 -> 134.1 mm, vias 0 -> 4
- net /CCS Greenphy Modem/SPI_SCK_A: track 0.00 -> 132.9 mm, vias 0 -> 4
- net /Main Processor/CURSENS_A_SIG: track 0.00 -> 130.2 mm, vias 0 -> 3
- net /Control Pilot Driver/INPUT_+: track 0.00 -> 129.0 mm, vias 0 -> 4
- net /Main Processor/CURSENS_B_REF: track 0.00 -> 126.7 mm, vias 0 -> 3
- net /ADC/SPI_SCK_A: track 0.00 -> 125.5 mm
- net /Control Pilot Driver/CP_FEEDBACK: track 0.00 -> 122.6 mm, vias 0 -> 2
- net /CAN Transciever1/A_CAN_RX: track 0.00 -> 122.2 mm, vias 0 -> 2
- net /CableIO/PUMP_PWM_LOGIC_A: track 0.00 -> 110.6 mm, vias 0 -> 3
- net /CableIO/TEMP_LOGIC_A: track 3.50 -> 112.6 mm, vias 1 -> 4
- net /ADC/ADC1_CS_A: track 0.00 -> 107.2 mm, vias 0 -> 4
- net /Main Processor/CURSENS_B_SIG: track 0.00 -> 105.3 mm, vias 0 -> 3
- net /ADC/ADC1_INT_A: track 0.00 -> 102.7 mm, vias 0 -> 4
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- added copper zone on In2.Cu, net /+12V_A
- added copper zone on In3.Cu, net /+3.3V_A
- added copper zone on B.Cu, net /AC_EARTH
- added copper zone on F.Cu, net /AC_EARTH
- added copper zone on In1.Cu, net /AC_EARTH
- added copper zone on In4.Cu, net /AC_EARTH
- added copper zone on In3.Cu, net /CAN1_+5V
- added copper zone on B.Cu, net /CAN1_GND
- added copper zone on F.Cu, net /CAN1_GND
- added copper zone on In1.Cu, net /CAN1_GND
- added copper zone on In2.Cu, net /CAN1_GND
- added copper zone on In4.Cu, net /CAN1_GND
- added copper zone on F.Cu, net /CAN2_+5V
- added copper zone on In3.Cu, net /CAN2_+5V
- added copper zone on B.Cu, net /CAN2_GND
- added copper zone on F.Cu, net /CAN2_GND
- added copper zone on In1.Cu, net /CAN2_GND
- added copper zone on In2.Cu, net /CAN2_GND
- added copper zone on In4.Cu, net /CAN2_GND
- added copper zone on B.Cu, net /VS_GND_Y
- added copper zone on F.Cu, net /VS_GND_Y
- added copper zone on In1.Cu, net /VS_GND_Y
- added copper zone on In2.Cu, net /VS_GND_Y
- added copper zone on In3.Cu, net /VS_GND_Y
- added copper zone on In4.Cu, net /VS_GND_Y
Other:
- board text added: "+12V"
- board text added: "+24V"
- board text added: "+5V"
- board text added: "-CP"
- board text added: "-PE"
- board text added: "AC MAINS INPUT 120/208/240V"
- board text added: "CANBUS 1"
- board text added: "CANBUS 2"
- board text added: "CAN_H"
- board text added: "CAN_L"
- board text added: "CONNECTOR TO J1772/CCS/NACS CABLE, CONTACTORS --->"
- board text added: "CONTACTOR VBUS"
- board text added: "CONTACTOR VOLTAGE SELECTION"
- board text added: "DC-"
- board text added: "EARTH"
- board text added: "GND"
- board text added: "JMP1"
- board text added: "JMP2"
- board text added: "L1"
- board text added: "L2/N"
- board text added: "MAIN"
- board text added: "NC"
- board text added: "OpenVVVF DC FAST CHARGER SECC"
- board text added: "PRE"
- board text added: "PWM"
- board text added: "PWM VBUS"
- board text added: "TMP"
- board text added: "VOLTAGE SENSE"
- board text added: "VS0"
- board text added: "VS1"
- board text added: "VS2"
- board text added: "VS3"
