File: Hardware/SECC/Boards/ControlBoard/ESP32_COPROC.kicad_sch (KiCad schematic)
At the start: 6 parts, among them U10 ESP32-C3-WROOM-02

Commit message: esp32 progress
Parts:
- added R14, R15: 10k,1%, symbol Device:R
Connections:
- net GND: now also C7.1; no longer C7.2
- net VCC_3.3V: now also R14.1, R15.1
- net ESP_EN: now reaches R12.2, U10.2 (EN)
- net ESP_EN: now also C7.2; no longer C7.1
- net ESP_SPI_CS: now reaches U10.10 (IO10)
- net ESP_SPI_CS: now also R15.2
- net ESP_UART_RX: now reaches U10.11 (IO20/RXD)
- net ESP_UART_TX: now reaches U10.12 (IO21/TXD)
- net ESP_USB_DM: now reaches U10.13 (IO18)
- net ESP_USB_DP: now reaches U10.14 (IO19)
- net ESP_SPI_MISO: now reaches U10.16 (IO2)
- net ESP_SPI_MISO: now also R14.2
- net ESP_SPI_SCK: now reaches U10.5 (IO6)
- net ESP_SPI_MOSI: now reaches U10.6 (IO7)
- net ESP_BOOT: now reaches U10.8 (IO9)
- no-connect marks 0 -> 3
Other:
- note added: "3V3 rail must supply >=500 mA peaks (Wi-Fi TX). Place C6 closer to pin 1 than C1. SPI is ESP32-C3 SPI2 in slave mode, up to 60 MHz. Keep traces short, length-matched. GPIO11-17 not available (in-package flash)."
- note added: "Cross to H7 UART: ESP_UART_TX -> H7_RX, ESP_UART_RX -> H7_TX. H7 idles its TX (ESP_UART_RX) high. Enter download mode: ESP_BOOT low + pulse ESP_EN low."
- note added: "H7 drives open-drain or push-pull-LOW only. EN is shared with the R12/C7 power-on-reset RC, so the H7 must never source current into it (a push-pull high would override the RC delay and fight any pull-down on the net)."
- note added: "Reserved for future USB connector (native USB-Serial/JTAG flashing/debug)."
